File: Boards/LCD_Screen/LCD_Screen.sch (KiCad schematic (older format))
At the start: 27 parts, among them J1 Ultrafit_4_RA, U1 MCP25625-x-SS, U101 TPS560430YF, U2 Raspberry_Pi_Zero, Y1 Crystal_SMD

Commit message: lcd board with new buck
Parts:
- removed C101, C103: C_0.1uF, footprints:C_0805_OEM, symbol formula:C_0.1uF
- removed C102: C_2.2uF, footprints:C_0603_1608Metric, symbol formula:C_2.2uF
- removed COUT101: C_22uF, footprints:C_1206_OEM, symbol formula:C_22uF
- removed COUT102: C_33uF, footprints:Fuse_1812, symbol formula:C_33uF
- removed COUT103: C_47uF, footprints:C_0805_OEM, symbol formula:C_47uF
- removed D101: D_Zener_18V, footprints:DO-214AA, symbol formula:D_Zener_18V
- removed D102, D103: LED_0805, footprints:LED_0805_OEM, symbol formula:LED_0805
- removed F101: F_500mA_16V, footprints:Fuse_1210, symbol formula:F_500mA_16V
- removed J1: Ultrafit_4_RA, footprints:Ultrafit_4_RA, symbol formula:Ultrafit_4_RA
- removed L101: L_100uH, footprints:L_100uH, symbol formula:L_100uH
- removed R101, R105: R_200, footprints:R_0805_OEM, symbol formula:R_200
- removed R102: R_25K, footprints:R_0805_OEM, symbol formula:R_25K
- removed R103: R_100K, footprints:R_0805_OEM, symbol formula:R_100K
- removed R104: R_0_2512, footprints:R_2512_OEM, symbol formula:R_0_2512
- removed R2: R_100, footprints:R_0805_OEM, symbol formula:R_200
- removed U101: TPS560430YF, footprints:SOT-23-6_OEM, symbol formula:TPS560430YF
- added C10: C_10uF, footprints:C_0805_OEM, symbol LCD_Screen-rescue:C_10uF-footprints-Buck_HighCurrent-rescue
- added C11: C_22uF, footprints:C_1206_OEM, symbol LCD_Screen-rescue:C_22uF-footprints-Buck_HighCurrent-rescue
- added C12: C_33uF, Capacitor_SMD:C_1812_4532Metric, symbol LCD_Screen-rescue:C_33uF-footprints-Buck_HighCurrent-rescue
- added C5: C_0.1uF, footprints:C_0603_1608Metric, symbol LCD_Screen-rescue:C_0.1uF_0603-footprints-Buck_HighCurrent-rescue
- added C6, C7: C_10uF_25V, footprints:C_0805_OEM, symbol LCD_Screen-rescue:C_10uF_25V-footprints-Buck_HighCurrent-rescue
- added C8: C_0.1uF_0603, footprints:C_0603_1608Metric, symbol LCD_Screen-rescue:C_0.1uF_0603-footprints-Buck_HighCurrent-rescue
- added C9: C_100nF, footprints:C_0603_1608Metric, symbol LCD_Screen-rescue:C_100nF-footprints-Buck_HighCurrent-rescue
- added D1: D_Zener_18V, footprints:DO-214AA, symbol LCD_Screen-rescue:D_Zener_18V-footprints-Buck_HighCurrent-rescue
- added D2, D3: LED_0805, footprints:LED_0805_OEM, symbol LCD_Screen-rescue:LED_0805-footprints-Buck_HighCurrent-rescue
- added F1: F_2.6A_16V, Fuse:Fuse_1812_4532Metric, symbol LCD_Screen-rescue:F_2.6A_16V-footprints-Buck_HighCurrent-rescue
- added J1: MicroFit_VT_4, footprints:MicroFit_VT_4, symbol formula:MicroFit_VT_4
- added L1: L_4.7uH_3.2A, footprints:IHLP2020BZER4R7M11, symbol LCD_Screen-rescue:IHLP2020BZER4R7M11-footprints-Buck_HighCurrent-rescue
- added R1: R_1K, footprints:R_0805_OEM, symbol LCD_Screen-rescue:R_200-footprints-Buck_HighCurrent-rescue
- added R2: R_120_DNP, footprints:R_0805_OEM, symbol formula:R_120_DNP
- added R4: R_10K, footprints:R_0805_OEM, symbol LCD_Screen-rescue:R_10K-footprints-Buck_HighCurrent-rescue
- added R5: R_51.1K, footprints:R_0805_OEM, symbol LCD_Screen-rescue:R_51.1K-footprints-Buck_HighCurrent-rescue
- added R6: R_22K, footprints:R_0805_OEM, symbol LCD_Screen-rescue:R_22K-footprints-Buck_HighCurrent-rescue
- added R7: R_1, footprints:R_0603_1608Metric, symbol LCD_Screen-rescue:R_1-footprints-Buck_HighCurrent-rescue
- added R8: R_0_2512, footprints:R_2512_OEM, symbol LCD_Screen-rescue:R_0_2512-footprints-Buck_HighCurrent-rescue
- added R9: R_200, footprints:R_0805_OEM, symbol LCD_Screen-rescue:R_200-footprints-Buck_HighCurrent-rescue
- added U3: TPS563231, footprints:SOT-563, symbol LCD_Screen-rescue:TPS563231-footprints-Buck_HighCurrent-rescue
- U2: footprint (none) -> footprints:PinHeader_2x20_P2.54mm_Vertical
Connections:
- net labels removed: CAN_HI, CAN_LO
- wire segments 84 -> 115
Other:
- note added: "MICROFIT"
- note removed: "12V Indicator"
- note removed: "5V"
- note removed: "5V Indicator"
- note removed: "Bootstrap Capacitor\n"
- note removed: "Feedback Divider\n"
- note removed: "Inductor\n"
- note removed: "Input Capacitors\n\n"
- note removed: "Output Capacitors\n"
- note removed: "Protection\n"
- note removed: "This buck converter will eventually change. Adi is currently coming up with a new one\n"
- note removed: "ULTRAFIT\n"
- note removed: "VCC Jumper\n"
- moved on the sheet: C1, C2, C3, C4, R3, U1, U2, Y1
