File: Boards/BMS_Data_Acquisition/DA_Board_1/DA_Board_1.kicad_pcb (KiCad board)
At the start: 2 copper layers, 340.1 x 44.9 mm, 75 parts, among them J1 MM_M_VT_10, J2 MM_M_VT_12, J3 MM_M_VT_12, J4 MM_M_VT_12, J5 MM_M_VT_16, J6 MM_M_VT_12, J7 MM_M_VT_12, J8 MM_M_VT_10, J9 MM_M_VT_12, Q10 BSS308PE, Q12 BSS308PE, Q14 BSS308PE, Q16 BSS308PE, Q2 BSS308PE, Q4 BSS308PE, Q6 BSS308PE, Q8 BSS308PE, T0 Tab_connect_BMS, T10 Tab_connect_BMS, T12 Tab_connect_BMS, T14 Tab_connect_BMS, T16 Tab_connect_BMS, T2 Tab_connect_BMS, T4 Tab_connect_BMS, T6 Tab_connect_BMS, T8 Tab_connect_BMS

Commit message: Working on layout
Parts:
- moved J5 8.20 mm to (154.5, 145.5), turned to 270 degrees
- moved J9 3.96 mm to (351.0, 138.4)
- moved J6 3.96 mm to (364.0, 138.8)
- moved J7 3.96 mm to (357.9, 138.7)
- moved J8 3.96 mm to (369.8, 139.0)
Changed lines of the file:
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@@
   )
   (setup
-    (last_trace_width 0.254)
+    (last_trace_width 0.25)
     (user_trace_width 0.254)
     (user_trace_width 0.381)
@@
   )
   (module footprints:micromatch_female_vert_16 (layer F.Cu)
-    (at 146.3294 144.3736)
-    (fp_text reference J5 (at 5.08 5.08) (layer F.SilkS)
-      (effects (font (size 1 1) (thickness 0.15)))
-    )
-    (fp_text value MM_M_VT_16 (at 6.35 0 90) (layer F.Fab) hide
-      (effects (font (size 1 1) (thickness 0.15)))
-    )
-    (fp_text user 16 (at 2.54 17.78) (layer F.SilkS)
-      (effects (font (size 1 1) (thickness 0.15)))
-    )
-    (fp_text user 1 (at 0 -8.89) (layer F.SilkS)
+    (at 154.4574 145.4658 270)
+    (fp_text reference J5 (at 5.08 5.08 270) (layer F.SilkS)
+      (effects (font (size 1 1) (thickness 0.15)))
+    )
+    (fp_text value MM_M_VT_16 (at 6.35 0) (layer F.Fab) hide
+      (effects (font (size 1 1) (thickness 0.15)))
+    )
+    (fp_text user 16 (at 2.54 17.78 270) (layer F.SilkS)
+      (effects (font (size 1 1) (thickness 0.15)))
+    )
+    (fp_text user 1 (at 0 -8.89 270) (layer F.SilkS)
       (effects (font (size 1 1) (thickness 0.15)))
     )
@@
     (fp_line (start -1.38 16.91) (end -1.38 -8.02) (layer F.SilkS) (width 0.15))
     (fp_line (start 3.92 16.91) (end 3.92 -8.02) (layer F.SilkS) (width 0.15))
-    (pad 5 thru_hole circle (at 0 0) (size 1.3 1.3) (drill 0.8) (layers *.Cu *.Mask)
+    (pad 5 thru_hole circle (at 0 0 270) (size 1.3 1.3) (drill 0.8) (layers *.Cu *.Mask)
       (net 62 /Q12))
-    (pad 3 thru_hole circle (at 0 -2.54) (size 1.3 1.3) (drill 0.8) (layers *.Cu *.Mask)
+    (pad 3 thru_hole circle (at 0 -2.54 270) (size 1.3 1.3) (drill 0.8) (layers *.Cu *.Mask)
       (net 63 /Q14))
-    (pad 1 thru_hole circle (at 0 -5.08) (size 1.3 1.3) (drill 0.8) (layers *.Cu *.Mask)
+    (pad 1 thru_hole circle (at 0 -5.08 270) (size 1.3 1.3) (drill 0.8) (layers *.Cu *.Mask)
       (net 64 /Q16))
-    (pad 7 thru_hole circle (at 0 2.54) (size 1.3 1.3) (drill 0.8) (layers *.Cu *.Mask)
+    (pad 7 thru_hole circle (at 0 2.54 270) (size 1.3 1.3) (drill 0.8) (layers *.Cu *.Mask)
       (net 65 /Q10))
-    (pad 2 thru_hole circle (at 2.54 -3.81) (size 1.3 1.3) (drill 0.8) (layers *.Cu *.Mask)
+    (pad 2 thru_hole circle (at 2.54 -3.81 270) (size 1.3 1.3) (drill 0.8) (layers *.Cu *.Mask)
       (net 66 /Q15))
-    (pad 4 thru_hole circle (at 2.54 -1.27) (size 1.3 1.3) (drill 0.8) (layers *.Cu *.Mask)
+    (pad 4 thru_hole circle (at 2.54 -1.27 270) (size 1.3 1.3) (drill 0.8) (layers *.Cu *.Mask)
       (net 67 /Q13))
-    (pad 6 thru_hole circle (at 2.54 1.27) (size 1.3 1.3) (drill 0.8) (layers *.Cu *.Mask)
+    (pad 6 thru_hole circle (at 2.54 1.27 270) (size 1.3 1.3) (drill 0.8) (layers *.Cu *.Mask)
       (net 68 /Q11))
-    (pad 8 thru_hole circle (at 2.54 3.81) (size 1.3 1.3) (drill 0.8) (layers *.Cu *.Mask)
+    (pad 8 thru_hole circle (at 2.54 3.81 270) (size 1.3 1.3) (drill 0.8) (layers *.Cu *.Mask)
       (net 69 /Q9))
-    (pad 9 thru_hole circle (at 0 5.08) (size 1.3 1.3) (drill 0.8) (layers *.Cu *.Mask)
+    (pad 9 thru_hole circle (at 0 5.08 270) (size 1.3 1.3) (drill 0.8) (layers *.Cu *.Mask)
       (net 70 /Q8))
-    (pad 10 thru_hole circle (at 2.54 6.35) (size 1.3 1.3) (drill 0.8) (layers *.Cu *.Mask)
+    (pad 10 thru_hole circle (at 2.54 6.35 270) (size 1.3 1.3) (drill 0.8) (layers *.Cu *.Mask)
       (net 71 /Q7))
-    (pad 11 thru_hole circle (at 0 7.62) (size 1.3 1.3) (drill 0.8) (layers *.Cu *.Mask)
+    (pad 11 thru_hole circle (at 0 7.62 270) (size 1.3 1.3) (drill 0.8) (layers *.Cu *.Mask)
       (net 72 /Q6))
-    (pad 12 thru_hole circle (at 2.54 8.89) (size 1.3 1.3) (drill 0.8) (layers *.Cu *.Mask)
+    (pad 12 thru_hole circle (at 2.54 8.89 270) (size 1.3 1.3) (drill 0.8) (layers *.Cu *.Mask)
       (net 73 /Q5))
-    (pad 13 thru_hole circle (at 0 10.16) (size 1.3 1.3) (drill 0.8) (layers *.Cu *.Mask)
+    (pad 13 thru_hole circle (at 0 10.16 270) (size 1.3 1.3) (drill 0.8) (layers *.Cu *.Mask)
       (net 74 /Q4))
-    (pad 14 thru_hole circle (at 2.54 11.43) (size 1.3 1.3) (drill 0.8) (layers *.Cu *.Mask)
+    (pad 14 thru_hole circle (at 2.54 11.43 270) (size 1.3 1.3) (drill 0.8) (layers *.Cu *.Mask)
       (net 75 /Q3))
-    (pad 15 thru_hole circle (at 0 12.7) (size 1.3 1.3) (drill 0.8) (layers *.Cu *.Mask)
+    (pad 15 thru_hole circle (at 0 12.7 270) (size 1.3 1.3) (drill 0.8) (layers *.Cu *.Mask)
       (net 76 /Q2))
-    (pad 16 thru_hole circle (at 2.54 13.97) (size 1.3 1.3) (drill 0.8) (layers *.Cu *.Mask)
+    (pad 16 thru_hole circle (at 2.54 13.97 270) (size 1.3 1.3) (drill 0.8) (layers *.Cu *.Mask)
       (net 77 /Q1))
-    (pad 17 thru_hole circle (at 1.8 -6.48) (size 2 2) (drill 1.5) (layers *.Cu *.Mask))
+    (pad 17 thru_hole circle (at 1.8 -6.48 270) (size 2 2) (drill 1.5) (layers *.Cu *.Mask))
     (model ${LOCAL_DIR}/OEM_Preferred_Parts/3DModels/micromatch_female_vert_16/c-1-338068-6-f-3d.stp
       (offset (xyz 1.3 -4.5 3.6))
@@
   )
   (module footprints:micromatch_female_vert_12 (layer F.Cu)
-    (at 367.1062 136.3726)
+    (at 363.982 138.811)
     (fp_text reference J6 (at 5.08 5.08) (layer F.SilkS)
       (effects (font (size 1 1) (thickness 0.15)))
@@
   )
   (module footprints:micromatch_female_vert_12 (layer F.Cu)
-    (at 360.981001 136.238001)
+    (at 357.856801 138.676401)
     (fp_text reference J7 (at 5.08 5.08) (layer F.SilkS)
       (effects (font (size 1 1) (thickness 0.15)))
@@
   )
   (module footprints:micromatch_female_vert_10 (layer F.Cu)
-    (at 372.9736 136.525)
+    (at 369.8494 138.9634)
     (fp_text reference J8 (at 5.08 5.08) (layer F.SilkS)
       (effects (font (size 1 1) (thickness 0.15)))
@@
   )
   (module footprints:micromatch_female_vert_12 (layer F.Cu)
-    (at 354.1268 135.9662)
+    (at 351.0026 138.4046)
     (fp_text reference J9 (at 5.08 5.08) (layer F.SilkS)
       (effects (font (size 1 1) (thickness 0.15)))

Commit message: More DA board layout
Parts:
- T0, T10, T12, T14, T16, T2, T4, T6, T8: value Tab_connect_BMS -> Tab_Connect_BMS; footprint footprints:Tab_connect_BMS -> footprints:Tab_Connect_BMS_2
- moved J2 145.1 mm to (44.1, 139.1)
- moved J1 145.0 mm to (44.1, 160.2)
- moved J3 142.9 mm to (184.9, 163.9)
- moved J4 142.8 mm to (184.7, 143.5)
- moved J7 40.2 mm to (320.0, 152.2)
- moved J9 40.1 mm to (315.1, 156.2), turned to 180 degrees
- moved R34 15.9 mm to (126.1, 174.0), turned to 90 degrees
- moved R32 15.9 mm to (84.3, 173.7), turned to 90 degrees
- moved R36 15.5 mm to (171.6, 173.6), turned to 90 degrees
- moved R40 14.7 mm to (260.5, 173.8), turned to 90 degrees
- moved R42 13.0 mm to (303.0, 174.0), turned to 90 degrees
- moved R44 13.0 mm to (341.8, 173.8), turned to 90 degrees
- moved R46 12.6 mm to (360.1, 174.0), turned to 90 degrees
- moved R38 12.2 mm to (216.2, 174.0), turned to 90 degrees
- moved D4 11.4 mm to (124.0, 173.9), turned to 90 degrees
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Connections:
- T0 pad 1: (no net) -> /PWR1
- T10 pad 1: (no net) -> /PWR11
- T12 pad 1: (no net) -> /PWR13
- T14 pad 1: (no net) -> /PWR15
- T16 pad 1: (no net) -> Net-(F+2-Pad1)
- T2 pad 1: (no net) -> /PWR3
- T4 pad 1: (no net) -> /PWR5
- T6 pad 1: (no net) -> /PWR7
- T8 pad 1: (no net) -> /PWR9
Routing:
- net /C3: track 0.00 -> 331.4 mm
- net /C5: track 0.00 -> 330.9 mm
- net /Q1: track 0.00 -> 275.5 mm
- net /Q3: track 0.00 -> 274.5 mm
- net /Q5: track 0.00 -> 267.6 mm
- net /Q7: track 0.00 -> 264.0 mm
- net /Q9: track 0.00 -> 254.8 mm
- net /Q11: track 0.00 -> 249.7 mm
- net /Q13: track 0.00 -> 239.5 mm
- net /Q15: track 0.00 -> 232.7 mm
- net /PWR6: track 217.9 -> 5.35 mm
- net /C7: track 0.00 -> 204.8 mm, vias 0 -> 1
- net /C9: track 0.00 -> 203.6 mm, vias 0 -> 1
- net /C13_T2: track 0.00 -> 200.5 mm
- net /C13_T1: track 0.00 -> 199.7 mm
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- added copper zone on F.Cu, net Net-(R10-PadEP)
- added copper zone on F.Cu, net Net-(R12-PadEP)
- added copper zone on F.Cu, net Net-(R14-PadEP)
- added copper zone on F.Cu, net Net-(R16-PadEP)
- added copper zone on F.Cu, net Net-(R2-PadEP)
- added copper zone on F.Cu, net Net-(R4-PadEP)
- added copper zone on F.Cu, net Net-(R6-PadEP)
- added copper zone on F.Cu, net Net-(R8-PadEP)

Commit message: Copied connectors from peripheral to DA board 1
Parts:
- added J1: MM_F_VT_12, footprints:micromatch_female_vert_12, B.Cu at (573.5, 356.7)
- added J2: MM_F_VT_10, footprints:micromatch_female_vert_10, B.Cu at (588.8, 358.6)
- added J3: MM_F_VT_16, footprints:micromatch_female_vert_16, B.Cu at (579.6, 273.8)
- added J4: MM_F_VT_12, footprints:micromatch_female_vert_12, B.Cu at (569.0, 95.0)
- added J5: MM_M_VT_12, footprints:micromatch_female_vert_12, B.Cu at (592.8, 95.0)
- moved J6 5.45 mm to (353.0, 140.8)
- moved J8 3.97 mm to (364.4, 140.5)
Routing:
- net /C9: track 203.6 -> 162.9 mm
- net /C7: track 204.8 -> 166.8 mm
- net /C13: track 199.6 -> 178.3 mm
- net /C11: track 194.8 -> 176.9 mm
- net /C5: track 330.9 -> 317.1 mm
- net /C3: track 331.4 -> 321.5 mm
- net /C15: track 194.1 -> 188.8 mm
Other:
- board size 340.1 x 44.9 mm -> 568.5 x 287 mm

Commit message: DA board work
Parts:
- removed the J1 at (573.5, 356.7)
- removed the J1 at (44.1, 160.2)
- removed the J2 at (588.8, 358.6)
- removed the J2 at (44.1, 139.1)
- removed the J3 at (579.6, 273.8)
- removed the J4 at (569.0, 95.0)
- removed the J5 at (592.8, 95.0)
- added J1: MM_M_VT_10, footprints:micromatch_female_vert_10, F.Cu at (319.1, 144.5)
- added J2: MM_M_VT_12, footprints:micromatch_female_vert_12, F.Cu at (56.1, 165.6)
- moved J3 132.9 mm to (317.8, 161.0), turned to 90 degrees
- moved J4 128.7 mm to (56.1, 141.7), turned to 90 degrees
- moved J5 85.6 mm to (234.9, 154.9), turned to 90 degrees
- moved J9 25.6 mm to (338.1, 144.9)
- moved J7 24.8 mm to (342.0, 140.9)
Routing:
- net /Q13: track 239.5 -> 0.00 mm
- net (no net): track 0.00 -> 239.5 mm
Other:
- board size 568.5 x 287 mm -> 340.1 x 60.8 mm

Commit message: Changes to DA_Board_1 Layout
Parts:
- J6: value MM_M_VT_12 -> MM_M_VT_10; footprint footprints:micromatch_female_vert_12 -> footprints:micromatch_female_vert_10
- J8: value MM_M_VT_10 -> MM_M_VT_12; footprint footprints:micromatch_female_vert_10 -> footprints:micromatch_female_vert_12
- moved J6 17.9 mm to (370.9, 141.0)
- moved J7 8.99 mm to (350.6, 138.4)
- moved J9 6.79 mm to (339.9, 138.3), turned to 0 degrees
- moved J8 4.09 mm to (360.9, 138.4)
Connections:
- J6 pad 1: /C15 -> /Q13
- J6 pad 10: /C15_T2 -> /PWR15
- J6 pad 11: /C15_T1 -> (no net)
- J6 pad 2: /C13 -> /PWR14
- J6 pad 3: /C11 -> /C15_T3
- J6 pad 4: /C9 -> /C15_T2
- J6 pad 5: /C7 -> /C15_T1
- J6 pad 6: /C5 -> /GND1
- J6 pad 7: /C3 -> /PWR16
- J6 pad 8: /C1 -> /C15
- J6 pad 9: /C15_T3 -> /Q15
- J7 pad 1: /C11_T2 -> Net-(J7-Pad1)
- J7 pad 10: /PWR15 -> /Q7
- J7 pad 11: /PWR14 -> /PWR8
- J7 pad 12: /PWR13 -> /C9
- J7 pad 2: /C11_T1 -> /PWR5
- J7 pad 3: /C7_T3 -> /Q5
- J7 pad 4: /C7_T2 -> /PWR6
- J7 pad 5: /C7_T1 -> /C7_T3
- J7 pad 6: /C3_T3 -> /C7_T2
- J7 pad 7: /C3_T2 -> /C7_T1
- J7 pad 8: /C3_T1 -> /C7
- J7 pad 9: /PWR16 -> /PWR7
- J8 pad 1: /Q15 -> /PWR9
- J8 pad 10: Net-(J8-Pad10) -> /PWR12
- J8 pad 11: (no net) -> /C13
- J8 pad 2: /Q13 -> /Q9
- J8 pad 3: /Q11 -> /PWR10
- J8 pad 4: /Q9 -> /C11_T3
- J8 pad 5: /Q7 -> /C11_T2
- J8 pad 6: /Q5 -> /C11_T1
- J8 pad 7: /Q3 -> /C11
- J8 pad 8: /Q1 -> /PWR11
- J8 pad 9: /GND1 -> /Q11
- J9 pad 1: /PWR12 -> /C1
- J9 pad 10: /PWR3 -> /Q3
- J9 pad 11: /PWR2 -> /PWR4
- J9 pad 12: /PWR1 -> /C5
- J9 pad 2: /PWR11 -> /PWR1
- J9 pad 3: /PWR10 -> /Q1
- J9 pad 4: /PWR9 -> /PWR2
- J9 pad 5: /PWR8 -> /C3_T3
- J9 pad 6: /PWR7 -> /C3_T2
- J9 pad 7: /PWR6 -> /C3_T1
- J9 pad 8: /PWR5 -> /C3
- J9 pad 9: /PWR4 -> /PWR3
Routing:
- net /C16: track 0.00 -> 369.2 mm, vias 0 -> 1
- net /PWR1: track 14.3 -> 382.1 mm, vias 0 -> 2
- net /C15_T1: track 0.00 -> 349.9 mm, vias 0 -> 1
- net /C15_T2: track 0.00 -> 338.4 mm
- net /C15_T3: track 0.00 -> 331.5 mm
- net /V+2: track 0.00 -> 327.2 mm, vias 0 -> 1
- net /C7_T2: track 0.00 -> 323.5 mm
- net /C7_T1: track 0.00 -> 318.5 mm
- net /C3_T3: track 0.00 -> 300.0 mm, vias 0 -> 1
- net /C3_T2: track 0.00 -> 299.0 mm
- net /PWR3: track 18.5 -> 317.3 mm, vias 0 -> 2
- net /C3_T1: track 0.00 -> 297.5 mm, vias 0 -> 1
- net /C3: track 321.5 -> 25.9 mm
- net /C1_T1: track 0.00 -> 291.6 mm, vias 0 -> 1
- net /C1_T3: track 0.00 -> 290.5 mm, vias 0 -> 1
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
Commit message: DA board layout rev 1.0
Parts:
- T0, T10, T12, T14, T16, T2, T4, T6, T8: footprint footprints:Tab_Connect_BMS_2 -> footprints:Tab_connect_BMS
- moved D16 15.2 mm to (371.8, 167.4)
- moved Q16 15.2 mm to (367.8, 167.3)
- moved R46 15.2 mm to (373.9, 167.5)
- moved D14 11.4 mm to (350.1, 168.7), turned to 270 degrees
- moved F16 11.1 mm to (362.0, 170.1), turned to 180 degrees
- moved D6 8.77 mm to (176.2, 168.3), turned to 270 degrees
- moved R44 7.96 mm to (348.1, 168.9)
- moved T10 7.20 mm to (250.6, 181.9)
- moved D2 6.63 mm to (86.2, 168.5), turned to 270 degrees
- moved D4 6.58 mm to (128.5, 169.2), turned to 270 degrees
- moved T12 6.40 mm to (294.3, 181.9)
- moved T4 6.10 mm to (119.7, 182.2)
- moved T6 6.07 mm to (163.2, 181.8)
- moved T14 5.95 mm to (338.0, 182.0)
- moved D12 5.95 mm to (303.7, 168.7), turned to 270 degrees
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Routing:
- net /GND1: track 14.5 -> 413.3 mm, vias 1 -> 7
- net /C14: track 0.00 -> 345.6 mm, vias 0 -> 2
- net /C11_T1: track 0.00 -> 331.8 mm
- net /C11_T3: track 0.00 -> 328.8 mm
- net /C11_T2: track 0.00 -> 325.0 mm
- net /C7_T3: track 0.00 -> 307.3 mm, vias 0 -> 2
- net /C12: track 0.00 -> 288.0 mm, vias 0 -> 2
- net /PWR2: track 5.51 -> 288.7 mm, vias 0 -> 1
- net /PWR5: track 18.2 -> 278.5 mm, vias 0 -> 1
- net /C10: track 0.00 -> 248.4 mm, vias 0 -> 2
- net /PWR4: track 5.30 -> 242.5 mm, vias 0 -> 2
- net /Q2: track 0.00 -> 232.2 mm, vias 0 -> 2
- net /PWR7: track 19.4 -> 230.5 mm, vias 0 -> 1
- net /PWR6: track 5.35 -> 212.3 mm, vias 0 -> 1
- net /Q16: track 0.00 -> 190.5 mm, vias 0 -> 2
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Other:
- outline, holes or cut-outs redrawn
- board text added: "BMS Data Acquisition #1 Rev 1.0 Olin Electric Motorsports Vienna Scheyer '21"

Commit message: gerbers for DA baords
Other:
- outline, holes or cut-outs redrawn

Commit message: Transferred Peripheral edge cuts and connectors over for reference
Parts:
- added D10: LED_0805, footprints:LED_0805_OEM, F.Cu at (263.5, 225.9)
- added D12: LED_0805, footprints:LED_0805_OEM, F.Cu at (305.4, 225.4)
- added D14: LED_0805, footprints:LED_0805_OEM, F.Cu at (351.8, 225.5)
- added D16: LED_0805, footprints:LED_0805_OEM, F.Cu at (373.5, 224.1)
- added D2: LED_0805, footprints:LED_0805_OEM, F.Cu at (87.9, 225.2)
- added D4: LED_0805, footprints:LED_0805_OEM, F.Cu at (130.2, 225.9)
- added D6: LED_0805, footprints:LED_0805_OEM, F.Cu at (177.9, 225.0)
- added D8: LED_0805, footprints:LED_0805_OEM, F.Cu at (218.4, 226.2)
- added F+1: 200mA_Fuse, footprints:Fuse_1812, F.Cu at (195.8, 230.8)
- added F+2: 200mA_Fuse, footprints:Fuse_1812, F.Cu at (363.7, 232.2)
- added F-1: 200mA_Fuse, footprints:Fuse_1812, F.Cu at (42.1, 231.1)
- added F-2: 200mA_Fuse, footprints:Fuse_1812, F.Cu at (201.2, 230.8)
- added F0: 200mA_Fuse, footprints:Fuse_1812, F.Cu at (48.1, 231.1)
- added F10: 200mA_Fuse, footprints:Fuse_1812, F.Cu at (262.5, 235.3)
- added F12: 200mA_Fuse, footprints:Fuse_1812, F.Cu at (303.8, 234.9)
- added F14: 200mA_Fuse, footprints:Fuse_1812, F.Cu at (346.8, 235.1)
- added F16: 200mA_Fuse, footprints:Fuse_1812, F.Cu at (363.7, 226.8)
- added F2: 200mA_Fuse, footprints:Fuse_1812, F.Cu at (86.6, 234.8)
- added F4: 200mA_Fuse, footprints:Fuse_1812, F.Cu at (128.5, 235.6)
- added F6: 200mA_Fuse, footprints:Fuse_1812, F.Cu at (177.1, 235.9)
- added F8: 200mA_Fuse, footprints:Fuse_1812, F.Cu at (216.7, 235.7)
- added J11: MM_F_VT_12, footprints:micromatch_female_vt_12, B.Cu at (162.4, 209.4)
- added J12: MM_F_VT_10, footprints:micromatch_female_vert_10, B.Cu at (186.9, 206.5)
- added J13: MM_F_VT_16, footprints:micromatch_female_vert_16, B.Cu at (220.8, 212.3)
- added J14: MM_F_VT_12, footprints:micromatch_female_vt_12, B.Cu at (245.0, 225.5)
- added J15: MM_M_VT_12, footprints:micromatch_female_vt_12, B.Cu at (269.9, 225.8)
- added Q10: BSS308PE, footprints:SOT-23-3_OEM, F.Cu at (256.6, 231.8)
- added Q12: BSS308PE, footprints:SOT-23-3_OEM, F.Cu at (297.7, 229.9)
- added Q14: BSS308PE, footprints:SOT-23-3_OEM, F.Cu at (340.6, 230.0)
- added Q16: BSS308PE, footprints:SOT-23-3_OEM, F.Cu at (369.5, 224.0)
- added Q2: BSS308PE, footprints:SOT-23-3_OEM, F.Cu at (80.7, 229.8)
- added Q4: BSS308PE, footprints:SOT-23-3_OEM, F.Cu at (122.2, 230.5)
- added Q6: BSS308PE, footprints:SOT-23-3_OEM, F.Cu at (170.1, 229.6)
- added Q8: BSS308PE, footprints:SOT-23-3_OEM, F.Cu at (210.7, 230.5)
- added R10: R_3.3_25W_TO163, footprints:PWR163, F.Cu at (255.3, 219.3)
- added R12: R_3.3_25W_TO163, footprints:PWR163, F.Cu at (297.4, 217.1)
- added R14: R_3.3_25W_TO163, footprints:PWR163, F.Cu at (337.6, 221.8)
- added R16: R_3.3_25W_TO163, footprints:PWR163, F.Cu at (361.6, 216.8)
- added R2: R_3.3_25W_TO163, footprints:PWR163, F.Cu at (79.8, 217.0)
- added R32: R_475, footprints:R_0805_OEM, F.Cu at (85.9, 225.6)
- added R34: R_475, footprints:R_0805_OEM, F.Cu at (128.2, 226.3)
- added R36: R_475, footprints:R_0805_OEM, F.Cu at (175.9, 225.4)
- added R38: R_475, footprints:R_0805_OEM, F.Cu at (216.4, 226.6)
- added R4: R_3.3_25W_TO163, footprints:PWR163, F.Cu at (122.3, 217.7)
- added R40: R_475, footprints:R_0805_OEM, F.Cu at (261.4, 226.3)
- added R42: R_475, footprints:R_0805_OEM, F.Cu at (303.4, 225.8)
- added R44: R_475, footprints:R_0805_OEM, F.Cu at (349.8, 225.6)
- added R46: R_475, footprints:R_0805_OEM, F.Cu at (375.6, 224.2)
- added R6: R_3.3_25W_TO163, footprints:PWR163, F.Cu at (170.1, 216.6)
- added R8: R_3.3_25W_TO163, footprints:PWR163, F.Cu at (210.5, 217.9)
- added RT11: Thermistor, footprints:Thermistor, F.Cu at (55.5, 232.2)
- added RT12: Thermistor, footprints:Thermistor, F.Cu at (61.4, 232.3)
- added RT13: Thermistor, footprints:Thermistor, F.Cu at (67.3, 232.4)
- added RT131: Thermistor, footprints:Thermistor, F.Cu at (316.5, 232.1)
- added RT132: Thermistor, footprints:Thermistor, F.Cu at (322.6, 232.1)
- added RT133: Thermistor, footprints:Thermistor, F.Cu at (328.4, 232.2)
- added RT51: Thermistor, footprints:Thermistor, F.Cu at (141.5, 232.3)
- added RT52: Thermistor, footprints:Thermistor, F.Cu at (147.6, 232.3)
- added RT53: Thermistor, footprints:Thermistor, F.Cu at (153.6, 232.3)
- added RT91: Thermistor, footprints:Thermistor, F.Cu at (229.5, 232.1)
- added RT92: Thermistor, footprints:Thermistor, F.Cu at (235.3, 232.0)
- added RT93: Thermistor, footprints:Thermistor, F.Cu at (241.3, 232.0)
- added T0: Tab_Connect_BMS, footprints:Tab_connect_BMS, F.Cu at (41.6, 238.8)
- added T10: Tab_Connect_BMS, footprints:Tab_connect_BMS, F.Cu at (252.3, 238.7)
- added T12: Tab_Connect_BMS, footprints:Tab_connect_BMS, F.Cu at (296.0, 238.6)
- added T14: Tab_Connect_BMS, footprints:Tab_connect_BMS, F.Cu at (339.7, 238.7)
- added T16: Tab_Connect_BMS, footprints:Tab_connect_BMS, F.Cu at (372.6, 232.2)
- added T2: Tab_Connect_BMS, footprints:Tab_connect_BMS, F.Cu at (77.8, 238.9)
- added T4: Tab_Connect_BMS, footprints:Tab_connect_BMS, F.Cu at (121.4, 238.9)
- added T6: Tab_Connect_BMS, footprints:Tab_connect_BMS, F.Cu at (164.9, 238.6)
- added T8: Tab_Connect_BMS, footprints:Tab_connect_BMS, F.Cu at (208.6, 238.7)
- moved D10 85.5 mm to (266.2, 83.8)
- moved D12 85.5 mm to (308.2, 83.3)
- moved D6 85.5 mm to (180.7, 82.9)
- moved F-1 85.5 mm to (44.9, 89.0)
- moved F10 85.5 mm to (265.3, 93.2)
- moved F12 85.5 mm to (306.6, 92.8)
- moved F16 85.5 mm to (366.5, 84.8)
- moved F2 85.5 mm to (89.3, 92.8)
- moved F4 85.5 mm to (131.3, 93.5)
- moved J2 85.5 mm to (60.5, 80.2)
- moved J3 85.5 mm to (322.3, 75.7)
- moved J4 85.5 mm to (60.6, 56.4)
- moved J5 85.5 mm to (239.4, 69.6)
- moved J7 85.5 mm to (354.7, 56.9)
- moved Q10 85.5 mm to (259.3, 89.7)
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Routing:
- net /GND1: track 413.3 -> 647.3 mm, vias 7 -> 11
- net /PWR9: track 230.4 -> 278.4 mm
- net Net-(F+2-Pad1): track 27.7 -> 55.5 mm
- net /PWR7: track 230.5 -> 258.0 mm
- net /PWR3: track 300.5 -> 322.5 mm
- net /PWR1: track 346.2 -> 366.1 mm
- net /PWR13: track 100.3 -> 119.5 mm
- net /PWR15: track 62.6 -> 80.8 mm
- net /PWR11: track 148.1 -> 165.9 mm
- net /PWR5: track 278.5 -> 296.1 mm
- net Net-(D14-Pad2): track 16.5 -> 33.0 mm
- net /Q4: track 181.5 -> 197.8 mm
- net Net-(D10-Pad2): track 14.9 -> 29.9 mm
- net Net-(D6-Pad2): track 14.3 -> 28.7 mm
- net Net-(D12-Pad2): track 14.3 -> 28.6 mm
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Other:
- board size 340.1 x 60.8 mm -> 342.9 x 202.9 mm
- board text added: "TOP"
