File: Boards/wheel_speed/_autosave-wheel_speed.sch (KiCad schematic (older format))
At the start: 41 parts, among them J1 CONN_02X03, J2 MM_F_RA_08, U1 MCP2561-E_SN, U101 TPS560430YF, U2 ATMEGA16M1, Y1 Crystal_SMD

Commit message: v0 checklist edits, generate gerbers
Parts:
- L101: footprint formula:L_100uH -> footprints:L_100uH
Changed lines of the file:
@@
 F 0 "L101" H 4250 6300 50  0000 C CNN
 F 1 "L_100uH" H 4250 6150 50  0000 C CNN
-F 2 "formula:L_100uH" H 4150 6000 50  0001 C CNN
+F 2 "footprints:L_100uH" H 4150 6000 50  0001 C CNN
 F 3 "https://product.tdk.com/info/en/catalog/datasheets/inductor_commercial_decoupling_nlfv32-ef_en.pdf" H 4150 6050 50  0001 C CNN
 F 4 "Digikey" H 4350 6000 50  0001 C CNN "MFN"
