File: Boards/328_Hacker/328_Hacker.sch (KiCad schematic (older format))
At the start: 17 parts, among them J1 Conn_01x11, J2 Conn_01x11, J3 CONN_02X03, J4 CONN_02X03, J5 Conn_02x02, U1 ATmega328P-AU, Y1 Crystal_SMD

Commit message: Addressed review comments
Connections:
- net 1L: now also R4.1
Changed lines of the file:
@@
 Text Notes 3250 3950 0    50   ~ 0
 5V Indication Light\n
-Text Label 3450 4200 0    50   ~ 0
+Text Label 3500 4200 0    50   ~ 0
 1L
 Text Label 2800 4200 0    50   ~ 0
