File: Boards/DUX_Interface/interface/interface.kicad_pcb (KiCad board)
At the start: 2 copper layers, 151.1 x 42.1 mm, 15 parts, among them J1 MM_F_VT_20, J2 MM_F_VT_20, J3 MM_F_VT_04, J4 MM_F_VT_10, J5 MM_F_VT_04, J6 NF_F_RA_2x02, J7 Ampseal_35_VT, J8 MicroFit_RA_V_2, U1 Nanofit_12, U2 Nanofit_4, U3 Nanofit_4, U4 Nanofit_10, U5 RJ45_VT, U6 RJ45_VT

Commit message: Finalized all Rev1 traces; added name; generated GERBERS and drill files
Other:
- board text added: "Dashboard Interface Alex Wenstrup REV1 - 11/25/19"
Changed lines of the file:
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@@
   (general
     (thickness 1.6)
-    (drawings 9)
-    (tracks 536)
+    (drawings 10)
+    (tracks 537)
     (zones 0)
     (modules 15)
@@
   )
   (setup
-    (last_trace_width 0.1524)
+    (last_trace_width 0.254)
     (user_trace_width 0.1524)
     (user_trace_width 0.254)
@@
     )
   )
+  (gr_text "Dashboard Interface\nAlex Wenstrup\nREV1 - 11/25/19" (at 83.8454 73.8378) (layer F.SilkS)
+    (effects (font (size 0.762 0.762) (thickness 0.1905)))
+  )
   (gr_text "SS_INERTIA\n" (at 80.4164 86.6902 90) (layer F.SilkS)
     (effects (font (size 0.762 0.762) (thickness 0.1524)))
@@
   (segment (start 210.202811 80.468471) (end 210.202811 82.447992) (width 0.254) (layer F.Cu) (net 2))
   (segment (start 210.0434 80.30906) (end 210.202811 80.468471) (width 0.254) (layer F.Cu) (net 2))
-  (segment (start 137.795 91.9226) (end 137.6788 91.8064) (width 0.1524) (layer B.Cu) (net 3))
   (segment (start 137.0076 90.6526) (end 139.5076 90.6526) (width 0.254) (layer F.Cu) (net 3))
   (segment (start 163.957 90.3986) (end 166.457 90.3986) (width 0.254) (layer F.Cu) (net 3))
@@
   (segment (start 204.9634 82.037178) (end 203.952979 83.047599) (width 0.1524) (layer F.Cu) (net 4))
   (segment (start 193.410599 83.047599) (end 192.7606 82.3976) (width 0.1524) (layer F.Cu) (net 4))
-  (segment (start 111.2012 89.0016) (end 110.360199 89.842601) (width 0.762) (layer B.Cu) (net 5))
-  (segment (start 110.360199 89.842601) (end 110.360199 92.430481) (width 0.762) (layer B.Cu) (net 5))
-  (segment (start 189.570601 89.397599) (end 190.2206 88.7476) (width 0.762) (layer B.Cu) (net 5))
   (segment (start 167.2836 79.8242) (end 168.783599 81.324199) (width 0.762) (layer F.Cu) (net 5))
   (segment (start 189.570601 88.097601) (end 190.2206 88.7476) (width 0.762) (layer F.Cu) (net 5))
@@
   (segment (start 163.2836 79.8242) (end 167.2836 79.8242) (width 0.762) (layer F.Cu) (net 5))
   (segment (start 133.2836 83.8242) (end 132.401074 83.8242) (width 0.8128) (layer B.Cu) (net 5))
-  (segment (start 110.360199 92.430481) (end 112.789119 94.859401) (width 0.762) (layer B.Cu) (net 5))
-  (segment (start 112.789119 94.859401) (end 184.108799 94.859401) (width 0.762) (layer B.Cu) (net 5))
-  (segment (start 184.108799 94.859401) (end 189.570601 89.397599) (width 0.762) (layer B.Cu) (net 5))
   (segment (start 129.8448 89.0016) (end 111.2012 89.0016) (width 0.762) (layer F.Cu) (net 5))
   (segment (start 131.191 89.0016) (end 129.8448 89.0016) (width 0.762) (layer F.Cu) (net 5))
   (segment (start 133.2836 83.8242) (end 133.2836 86.909) (width 0.762) (layer F.Cu) (net 5))
   (segment (start 133.2836 86.909) (end 131.191 89.0016) (width 0.762) (layer F.Cu) (net 5))
+  (segment (start 183.7182 95.25) (end 189.570601 89.397599) (width 0.762) (layer B.Cu) (net 5))
+  (segment (start 189.570601 89.397599) (end 190.2206 88.7476) (width 0.762) (layer B.Cu) (net 5))
+  (segment (start 113.179718 95.25) (end 183.7182 95.25) (width 0.762) (layer B.Cu) (net 5))
+  (segment (start 111.2012 89.0016) (end 110.360199 89.842601) (width 0.762) (layer B.Cu) (net 5))
+  (segment (start 110.360199 92.430481) (end 113.179718 95.25) (width 0.762) (layer B.Cu) (net 5))
+  (segment (start 110.360199 89.842601) (end 110.360199 92.430481) (width 0.762) (layer B.Cu) (net 5))
   (segment (start 204.404154 84.104829) (end 194.964149 84.104829) (width 0.1524) (layer F.Cu) (net 6))
   (segment (start 207.5034 79.2484) (end 207.752178 79.2484) (width 0.1524) (layer F.Cu) (net 6))
@@
   (segment (start 137.0076 88.1526) (end 135.83059 89.32961) (width 0.254) (layer F.Cu) (net 36))
   (segment (start 135.83059 89.32961) (end 135.83059 91.491608) (width 0.254) (layer F.Cu) (net 36))
-  (segment (start 148.4122 94.2594) (end 149.7584 94.2594) (width 0.254) (layer F.Cu) (net 36))
-  (via (at 150.241 93.7768) (size 0.8) (drill 0.4) (layers F.Cu B.Cu) (net 36))
-  (segment (start 149.7584 94.2594) (end 150.241 93.7768) (width 0.254) (layer F.Cu) (net 36))
+  (via (at 150.2918 93.9038) (size 0.8) (drill 0.4) (layers F.Cu B.Cu) (net 36))
   (segment (start 148.4122 94.2594) (end 148.5646 94.2594) (width 0.254) (layer F.Cu) (net 36))
   (segment (start 138.598382 94.2594) (end 148.4122 94.2594) (width 0.254) (layer F.Cu) (net 36))
   (via (at 152.7556 93.7768) (size 0.8) (drill 0.4) (layers F.Cu B.Cu) (net 36))
-  (segment (start 150.241 93.7768) (end 152.7556 93.7768) (width 0.254) (layer B.Cu) (net 36))
   (segment (start 153.155599 94.176799) (end 152.7556 93.7768) (width 0.254) (layer F.Cu) (net 36))
   (segment (start 165.801782 94.2594) (end 153.2382 94.2594) (width 0.254) (layer F.Cu) (net 36))
   (segment (start 153.2382 94.2594) (end 153.155599 94.176799) (width 0.254) (layer F.Cu) (net 36))
+  (segment (start 152.6286 93.9038) (end 152.7556 93.7768) (width 0.254) (layer B.Cu) (net 36))
+  (segment (start 150.2918 93.9038) (end 152.6286 93.9038) (width 0.254) (layer B.Cu) (net 36))
+  (segment (start 150.114 93.9038) (end 150.2918 93.9038) (width 0.254) (layer F.Cu) (net 36))
+  (segment (start 148.4122 94.2594) (end 149.7584 94.2594) (width 0.254) (layer F.Cu) (net 36))
+  (segment (start 149.7584 94.2594) (end 150.114 93.9038) (width 0.254) (layer F.Cu) (net 36))
   (via (at 163.6522 93.4212) (size 0.8) (drill 0.4) (layers F.Cu B.Cu) (net 37))
   (via (at 166.8018 93.3704) (size 0.8) (drill 0.4) (layers F.Cu B.Cu) (net 37))
@@
   (segment (start 155.524178 93.4212) (end 153.709577 91.606599) (width 0.1524) (layer F.Cu) (net 37))
   (via (at 149.4028 93.2688) (size 0.8) (drill 0.4) (layers F.Cu B.Cu) (net 37))
-  (segment (start 151.669801 92.868801) (end 151.8412 93.0402) (width 0.1524) (layer B.Cu) (net 37))
-  (segment (start 149.802799 92.868801) (end 151.669801 92.868801) (width 0.1524) (layer B.Cu) (net 37))
-  (segment (start 149.4028 93.2688) (end 149.802799 92.868801) (width 0.1524) (layer B.Cu) (net 37))
   (segment (start 152.709116 91.606599) (end 153.0604 91.606599) (width 0.1524) (layer F.Cu) (net 37))
   (segment (start 151.8412 92.474515) (end 152.709116 91.606599) (width 0.1524) (layer F.Cu) (net 37))
@@
   (segment (start 139.5076 88.1526) (end 144.6238 93.2688) (width 0.1524) (layer F.Cu) (net 37))
   (segment (start 144.708494 93.2688) (end 144.78 93.2688) (width 0.1524) (layer F.Cu) (net 37))
+  (segment (start 151.669801 92.868801) (end 151.8412 93.0402) (width 0.1524) (layer B.Cu) (net 37))
+  (segment (start 149.802799 92.868801) (end 151.669801 92.868801) (width 0.1524) (layer B.Cu) (net 37))
   (segment (start 144.78 93.2688) (end 149.4028 93.2688) (width 0.1524) (layer F.Cu) (net 37))
+  (segment (start 149.4028 93.2688) (end 149.802799 92.868801) (width 0.1524) (layer B.Cu) (net 37))
   (segment (start 172.0558 93.4974) (end 195.3768 93.4974) (width 0.1524) (layer F.Cu) (net 38))
   (segment (start 200.035401 89.164401) (end 200.6854 89.8144) (width 0.1524) (layer F.Cu) (net 38))
