File: Boards/TSAL_AIL/TSAL-AIL/TSAL-AIL.sch (KiCad schematic (older format))
At the start: 29 parts

Commit message: hopefully one of the last schematic pushes
Parts:
- C1: renamed from C?; symbol Formula:C_10uF -> TSAL-AIL-rescue:C_10uF-Formula
- C2: renamed from C?; symbol Formula:C_0.1uF -> TSAL-AIL-rescue:C_0.1uF-Formula
- C3, C4: renamed from C?; symbol Formula:C_1uF -> TSAL-AIL-rescue:C_1uF-Formula
- D1: renamed from D?; symbol Formula:LED_0805 -> TSAL-AIL-rescue:LED_0805-Formula
- F1: renamed from F?; symbol Formula:F_21mA_420V -> TSAL-AIL-rescue:F_21mA_420V-Formula
- J1: renamed from J?; symbol Formula:Ultrafit_4_RA -> TSAL-AIL-rescue:Ultrafit_4_RA-Formula
- J2: renamed from J?; symbol Formula:NanoFit_2 -> TSAL-AIL-rescue:NanoFit_2-Formula
- J3: renamed from J?; symbol Formula:MM_F_RA_06 -> TSAL-AIL-rescue:MM_F_RA_06-Formula
- Q1, Q2: renamed from Q?; symbol Formula:SSM3K333R -> TSAL-AIL-rescue:SSM3K333R-Formula
- R1, R4, R6, R7: renamed from R?; symbol Formula:R_270K -> TSAL-AIL-rescue:R_270K-Formula
- R10, R11, R2: renamed from R?; symbol Formula:R_1K -> TSAL-AIL-rescue:R_1K-Formula
- R12: renamed from R?; symbol Formula:R_499 -> TSAL-AIL-rescue:R_499-Formula
- R13, R14, R5: renamed from R?; symbol Formula:R_10K -> TSAL-AIL-rescue:R_10K-Formula
- R8: renamed from R?; symbol Formula:R_3K -> TSAL-AIL-rescue:R_3K-Formula
- R9: renamed from R?; symbol Formula:R_1.43K -> TSAL-AIL-rescue:R_1.43K-Formula
- U1: renamed from U?; symbol Formula:MCP6001 -> TSAL-AIL-rescue:MCP6001-Formula
- U2: renamed from U?; symbol Formula:LR8K4-G -> TSAL-AIL-rescue:LR8K4-G-Formula
- U3: renamed from U?; symbol Formula:CPC1025NTR -> TSAL-AIL-rescue:CPC1025NTR-Formula
- U4: renamed from U?; symbol Formula:BU4S11G2-TR -> TSAL-AIL-rescue:BU4S11G2-TR-Formula
- gave numbers to parts that had none: 1
Other:
- note added: "Is this a 137ohm resistor?\n"
