File: Boards/Steering/Steering.sch (KiCad schematic (older format))
At the start: 25 parts, among them J4 CONN_02X03, U1 MCP2561-E_SN, Y1 Crystal_SMD

Commit message: Sterring 1st passed layout
Parts:
- U2: renamed from U?; value ATMEGA16M1 -> MICROCONTROLLER
- gave numbers to parts that had none: 7
- renumbered C4 to C1, C1 to C2, C2 to C3, C6 to C4, C8 to C5, D5 to D1, D6 to D2, D4 to D3, R2 to R10, R7 to R2, R5 to R6, R6 to R7, R1 to R9
Connections:
- net B1_In: now also J1.1
- net CANH: now also R2.1
- net CANL: now also R2.2
- net RESET: no longer J4.5 (P5)
- net VCC: now also J1.2
- net +12V renamed +5V
- net Button_Readout2: no longer names the net of U2.17 ((PCINT12/ADC8/ACMPN3/AMP1-)PC4)
- net Button_Readout3: no longer names the net of U2.24 ((PCINT4/AMP0+)PB4)
- net Button_Readout4: no longer names the net of U2.25 ((PCINT15/D2A/AMP2+)PC7)
- no-connect marks 11 -> 14
Other:
- note removed: "MICROCONTROLLER"
- moved on the sheet: C1, D1, D2, D3, J1, J2, J3, J4, R1, R2, R3, R4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
