File: Boards/Throttle/throttle.sch (KiCad schematic (older format))
At the start: 68 parts, among them IC1 ATMEGA16M1, J1 micromatch_female_TOP_ENTRY_l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, J2 micromatch_female_TOP_ENTRY_l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, J3 CONN_02X03, Q1 SSM3K333R, Q2 SSM3K333R, Q3 SSM3K333R, U1 MCP6001, U2 MCP6001, U3 TPS560430YF, U4 CAN_Transceiver, Y1 Crystal_SMD

Commit message: throttle schematic complete
Connections:
- net Drive_Mode_Sense renamed DRIVE_MODE_SENSE
- net GND_DriveMode renamed GND_DRIVEMODE
- net ProgrammingLED1 renamed PROGRAMMINGLED1
- net ProgrammingLED2 renamed PROGRAMMINGLED2
- net ProgrammingLED3 renamed PROGRAMMINGLED3
- net SS_BOTS_Out_n renamed SS_BOTS_OUT
- net SS_Cockpit_EStop renamed SS_COCKPIT_ESTOP
- net SS_EStop_Out_n renamed SS_ESTOP_OUT
- net SS_Inertia_Out_n renamed SS_INERTIA_OUT
- net SS_Inertia_Switch renamed SS_INERTIA_SWITCH
- net Throttle1Sensing renamed THROTTLE1SENSING
- net Throttle1_Right_Sense renamed THROTTLE1_RIGHT_SENSE
- net Throttle2Sensing renamed THROTTLE2SENSING
- net Throttle2_Left_Sense renamed THROTTLE2_LEFT_SENSE

Commit message: edit layout
Other:
- moved on the sheet: C1, C2, D1, D2, D3, D4, D6, D8, Q1, Q2, Q3, R1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

Commit message: Begin Layout
Parts:
- renumbered C3 to C101, C4 to C102, C5 to C103, COUT1 to COUT101, COUT2 to COUT102, COUT3 to COUT103, D5 to D101, D7 to D102, D9 to D103, F1 to F101, L1 to L101, R18 to R101, R24 to R102, R25 to R103, R27 to R104, R28 to R105, U3 to U101

Commit message: Revert "Begin Layout"
This reverts commit f66e97611986f6cb10e89dffa2fa205961dd2a3d.
Parts:
- renumbered C101 to C3, C102 to C4, C103 to C5, COUT101 to COUT1, COUT102 to COUT2, COUT103 to COUT3, D101 to D5, D102 to D7, D103 to D9, F101 to F1, L101 to L1, R101 to R18, R102 to R24, R103 to R25, R104 to R27, R105 to R28, U101 to U3

Commit message: throttleboard files
Parts:
- renumbered C3 to C101, C4 to C102, C5 to C103, COUT1 to COUT101, COUT2 to COUT102, COUT3 to COUT103, D5 to D101, D7 to D102, D9 to D103, F1 to F101, L1 to L101, R18 to R101, R24 to R102, R25 to R103, R27 to R104, R28 to R105, U3 to U101
