File: Boards/Throttle/throttle_start3.kicad_pcb (KiCad board)
At the start: 4 copper layers, 58.4 x 40.3 mm, 70 parts, among them IC1 ATMEGA16M1, J1 micromatch_female_TOP_ENTRY_l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, J2 micromatch_female_TOP_ENTRY_l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, J3 CONN_02X03, Q1 SSM3K333R, Q2 SSM3K333R, Q3 SSM3K333R, U1 MCP6001, U101 TPS560430YF, U2 MCP6001, U4 CAN_Transceiver, Y1 Crystal_SMD

Commit message: throttleboard files
Parts:
- moved R104 65.1 mm to (157.3, 64.9)
- moved COUT102 65.1 mm to (163.0, 64.9)
- moved F101 64.0 mm to (152.1, 68.8)
- moved L101 64.0 mm to (159.6, 68.8)
- moved C101 64.0 mm to (151.9, 72.3)
- moved COUT101 64.0 mm to (164.1, 71.2)
- moved COUT103 64.0 mm to (164.1, 68.9)
- moved D101 64.0 mm to (147.1, 70.8)
- moved D103 64.0 mm to (155.8, 57.3)
- moved R102 64.0 mm to (155.6, 75.5)
- moved R103 64.0 mm to (159.5, 75.5)
- moved R105 64.0 mm to (155.8, 61.1)
- moved U101 64.0 mm to (156.8, 72.5)
- moved C102 64.0 mm to (153.7, 72.4)
- moved C103 64.0 mm to (160.1, 72.5)
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Routing:
- net Net-(D103-Pad2): track 25.5 -> 6.55 mm, vias 2 -> 0
- net /12V: track 3.87 -> 12.9 mm
- net VCC: track 167.6 -> 176.5 mm
- net GND: track 89.6 -> 94.9 mm, vias 44 -> 45
- net Net-(COUT101-Pad1): track 19.2 -> 17.3 mm
- net /SS_COCKPIT_ESTOP: vias 3 -> 2
