File: Boards/Throttle/throttle_start.kicad_pcb (KiCad board)
At the start: 2 copper layers, 109.3 x 58.3 mm, 54 parts, among them J1 CONN_02X03, J2 CONN_02X03, U1 LM3480, U101 TPS560430YF, U2 ATMEGA16M1, U3 TXB0104, U4 MCP2561-E_SN, U6 ATmega328P-AU, Y1 Crystal_SMD, Y2 Crystal_SMD

Commit message: Revert "Begin Layout"
This reverts commit f66e97611986f6cb10e89dffa2fa205961dd2a3d.
Parts:
- removed C11, C12: C_30pF, footprints:C_0805_OEM
- removed U6: ATmega328P-AU, Package_QFP:TQFP-32_7x7mm_P0.8mm
- removed Y2: Crystal_SMD, footprints:Crystal_SMD_FA238
- added COUT1: C_22uF, footprints:C_1206_OEM, F.Cu at (124.2, 130.8)
- added COUT2: C_33uF, footprints:Fuse_1812, F.Cu at (147.3, 121.9)
- added COUT3: C_47uF, footprints:C_0805_OEM, F.Cu at (116.8, 129.5)
- added D5: D_Zener_18V, footprints:DO-214AA, F.Cu at (109.2, 121.9)
- added D6: LED_0805, footprints:LED_0805_OEM, F.Cu at (173.4, 122.6)
- added D7: LED_0805, footprints:LED_0805_OEM, F.Cu at (131.0, 129.5)
- added D8: LED_0805, footprints:LED_0805_OEM, F.Cu at (162.6, 122.6)
- added D9: LED_0805, footprints:LED_0805_OEM, F.Cu at (105.6, 99.1)
- added F1: F_500mA_16V, footprints:Fuse_1210, F.Cu at (109.2, 129.5)
- added IC1: ATMEGA16M1, footprints:TQFP-32_7x7mm_Pitch0.8mm, F.Cu at (167.6, 99.1)
- added J3: CONN_02X03, footprints:Pin_Header_Straight_2x03, F.Cu at (167.6, 110.5)
- added Q1: SSM3K333R, footprints:SOT-23F, F.Cu at (187.3, 128.3)
- added Q2: SSM3K333R, footprints:SOT-23F, F.Cu at (176.5, 128.3)
- added Q3: SSM3K333R, footprints:SOT-23F, F.Cu at (165.7, 128.3)
- added R11: R_2.2k, footprints:R_0805_OEM, F.Cu at (194.9, 114.9)
- added R12: R_22K, footprints:R_0805_OEM, F.Cu at (203.2, 116.8)
- added R13: R_22K, footprints:R_0805_OEM, F.Cu at (198.8, 116.8)
- added R14: R_1k, footprints:R_0805_OEM, F.Cu at (187.3, 121.3)
- added R15: R_100k, footprints:R_0805_OEM, F.Cu at (187.3, 124.5)
- added R16: R_10k, footprints:R_0805_OEM, F.Cu at (191.1, 128.3)
- added R17: R_1k, footprints:R_0805_OEM, F.Cu at (176.5, 121.3)
- added R18: R_200, footprints:R_0805_OEM, F.Cu at (129.5, 126.4)
- added R19: R_100k, footprints:R_0805_OEM, F.Cu at (176.5, 124.5)
- added R20: R_10k, footprints:R_0805_OEM, F.Cu at (180.3, 128.3)
- added R21: R_1k, footprints:R_0805_OEM, F.Cu at (165.7, 121.3)
- added R22: R_100k, footprints:R_0805_OEM, F.Cu at (165.7, 124.5)
- added R23: R_10k, footprints:R_0805_OEM, F.Cu at (169.5, 128.3)
- added R24: R_25K, footprints:R_0805_OEM, F.Cu at (123.8, 122.6)
- added R25: R_100K, footprints:R_0805_OEM, F.Cu at (123.8, 126.4)
- added R26: R_100, footprints:R_0805_OEM, F.Cu at (160.0, 99.1)
- added R27: R_0_2512, footprints:R_2512_OEM, F.Cu at (116.8, 121.4)
- added R28: R_200, footprints:R_0805_OEM, F.Cu at (105.7, 104.1)
- added R29: R_10k, footprints:R_0805_OEM, F.Cu at (163.8, 91.4)
- added R30: R_120 DNP, footprints:R_0805_OEM, F.Cu at (173.4, 82.5)
- added R_1: R_200, footprints:R_0805_OEM, F.Cu at (175.9, 99.7)
- added R_2: R_200, footprints:R_0805_OEM, F.Cu at (175.9, 102.2)
- C101: footprint footprints:C_0805_OEM -> footprints:C_0603_1608Metric
- C102: footprint footprints:C_0603_1608Metric -> footprints:C_0805_OEM
- C4: value C_0.1uF -> C_2.2uF; footprint footprints:C_0805_OEM -> footprints:C_0603_1608Metric
- C5, C6: value C_30pF -> C_0.1uF
- C7: value C_0.1uF -> C_100pF
- C8, C9: value C_0.1uF -> C_30pF
- J1: value CONN_02X03 -> micromatch_female_TOP_ENTRY_locking_4; footprint footprints:Pin_Header_Straight_2x03 -> footprints:micromatch_female_vert_4; moved to B.Cu
- J2: value CONN_02X03 -> micromatch_female_TOP_ENTRY_locking_20; footprint footprints:Pin_Header_Straight_2x03 -> footprints:micromatch_female_vert_20; moved to B.Cu
- L101: footprint footprints:L_100uH_OEM -> footprints:L_100uH
- R1: value R_200 -> R_1M
- R10: value R_10K -> R_0-formula; footprint footprints:R_0805_OEM -> footprints:R_0603_1608Metric
- R2, R3: value R_200 -> R_0; footprint footprints:R_0805_OEM -> footprints:R_0603_1608Metric
- R4: value R_200 -> R_0-formula; footprint footprints:R_0805_OEM -> footprints:R_0603_1608Metric
- R5: value R_10K -> R_2.2k
- R6, R8: value R_4.7K -> R_200
- R7: value R_10K -> R_200
- R9: value R_120_DNP -> R_1M
- U1: value LM3480 -> MCP6001; footprint footprints:SOT-23-3_OEM -> footprints:SOT-23-5_OEM
- U2: value ATMEGA16M1 -> MCP6001; footprint footprints:TQFP-32_7x7mm_Pitch0.8mm -> footprints:SOT-23-5_OEM
- U3: value TXB0104 -> TPS560430YF; footprint Package_SO:TSSOP-14_4.4x5mm_P0.65mm -> footprints:SOT-23-6_OEM
- U4: value MCP2561-E_SN -> CAN_Transceiver
- moved G*** 63.2 mm to (242.6, 101.6)
- moved U1 60.9 mm to (178.4, 111.8), turned to 180 degrees
- moved U3 51.0 mm to (137.2, 128.6)
- moved R7 42.8 mm to (181.3, 91.4), turned to 180 degrees
- moved J2 39.1 mm to (203.2, 88.9), turned to 180 degrees
- moved C9 35.3 mm to (159.4, 109.2), turned to 180 degrees
- moved C7 34.4 mm to (157.5, 101.3), turned to 270 degrees
- moved U2 33.2 mm to (190.5, 111.8), turned to 180 degrees
- moved R5 31.6 mm to (182.9, 114.9)
- moved D3 30.8 mm to (186.1, 87.6), turned to 180 degrees
- moved R2 30.4 mm to (193.7, 92.7), turned to 180 degrees
- moved D1 29.9 mm to (186.1, 95.2), turned to 180 degrees
- moved C1 29.8 mm to (178.4, 115.6), turned to 180 degrees
- moved C10 22.7 mm to (167.6, 87.6)
- moved C5 21.9 mm to (137.2, 121.9), turned to 180 degrees
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Connections:
- C1 pad 1: VCC -> GND
- C1 pad 2: GND -> VCC
- C10 pad 1: /3.3V -> VCC
- C2 pad 1: /3.3V -> GND
- C2 pad 2: GND -> VCC
- C3 pad 1: VCC -> Net-(C3-Pad1)
- C4 pad 1: /3.3V -> Net-(C3-Pad1)
- C5 pad 2: GND -> Net-(C5-Pad2)
- C6 pad 1: Net-(C6-Pad1) -> VCC
- C7 pad 1: VCC -> Net-(C7-Pad1)
- C8 pad 1: VCC -> Net-(C8-Pad1)
- C9 pad 1: /3.3V -> Net-(C9-Pad1)
- D1 pad 1: GND -> Net-(D1-Pad1)
- D1 pad 2: Net-(D1-Pad2) -> /PROGRAMMINGLED1
- D2 pad 1: GND -> Net-(D2-Pad1)
- D2 pad 2: Net-(D2-Pad2) -> /PROGRAMMINGLED2
- D3 pad 1: GND -> Net-(D3-Pad1)
- D3 pad 2: Net-(D3-Pad2) -> /PROGRAMMINGLED3
- J1 pad 1: /MISO3.3V -> /SS_BOTS
- J1 pad 2: VCC -> /SS_INERTIA_SWITCH
- J1 pad 3: /SCK3.3V -> /SS_COCKPIT_ESTOP
- J1 pad 4: Net-(J1-Pad4) -> GND
- J1 pad 5: /RESET3.3V -> (no net)
- J2 pad 1: /MISO -> GND
- J2 pad 2: VCC -> +12V
- J2 pad 3: /SCK -> VCC
- J2 pad 4: /MOSI -> /MISO
- J2 pad 5: /RESET -> /MOSI
- J2 pad 6: GND -> /SCK
- L101 pad 1: Net-(C103-Pad2) -> Net-(C103-Pad1)
- R1 pad 1: /PROGRAMMINGLED1 -> VCC
- R1 pad 2: Net-(D1-Pad2) -> /THROTTLE1_RIGHT_SENSE
- R10 pad 1: /3.3V -> /THROTTLE1SENSING
- R10 pad 2: /RESET3.3V -> Net-(R10-Pad2)
- R2 pad 1: /PROGRAMMINGLED2 -> Net-(J2-Pad10)
- R2 pad 2: Net-(D2-Pad2) -> VCC
- R3 pad 1: /PROGRAMMINGLED3 -> VCC
- R3 pad 2: Net-(D3-Pad2) -> Net-(J2-Pad13)
- R4 pad 1: /PROGRAMMINGLED4 -> /THROTTLE2SENSING
- R4 pad 2: Net-(D4-Pad2) -> Net-(R4-Pad2)
- R5 pad 1: VCC -> Net-(R4-Pad2)
- R5 pad 2: /RESET -> GND
- R6 pad 1: /3.3V -> Net-(D1-Pad1)
- R6 pad 2: /SCL -> GND
- R7 pad 1: Net-(R7-Pad1) -> Net-(D2-Pad1)
- R7 pad 2: VCC -> GND
- R8 pad 1: /3.3V -> Net-(D3-Pad1)
- R8 pad 2: /SDA -> GND
- R9 pad 1: /CAN_H -> VCC
- R9 pad 2: /CAN_L -> /THROTTLE2_LEFT_SENSE
- U1 pad 1: /3.3V -> /THROTTLE2SENSING
- U1 pad 2: VCC -> GND
- U1 pad 3: GND -> /THROTTLE1_RIGHT_SENSE
- U101 pad 1: Net-(C103-Pad1) -> Net-(C103-Pad2)
- U101 pad 6: Net-(C103-Pad2) -> Net-(C103-Pad1)
- U2 pad 1: /MISO -> /THROTTLE1SENSING
- U2 pad 2: /MOSI -> GND
- U2 pad 3: /CS5V -> /THROTTLE2_LEFT_SENSE
- U2 pad 4: VCC -> Net-(R10-Pad2)
- U2 pad 5: GND -> VCC
- U3 pad 1: VCC -> Net-(C5-Pad2)
- U3 pad 2: /SCK5V -> GND
- U3 pad 3: /MISO5V -> Net-(R24-Pad1)
- U3 pad 4: /MOSI5V -> Net-(C3-Pad1)
- U3 pad 5: /CS5V -> Net-(C3-Pad1)
- U3 pad 6: Net-(U3-Pad6) -> Net-(C5-Pad1)
- U4 pad 1: /CAN_TX -> /TXCAN
- U4 pad 4: /CAN_RX -> /RXCAN
- U4 pad 6: /CAN_L -> /CANL
- U4 pad 7: /CAN_H -> /CANH
- Y1 pad 1: Net-(C5-Pad1) -> Net-(C8-Pad1)
- Y1 pad 3: Net-(C6-Pad1) -> Net-(C9-Pad1)
Routing:
- net VCC: track 3.93 -> 41.5 mm
- net GND: track 57.6 -> 79.2 mm
- net /SS_BOTS: track 0.00 -> 13.9 mm
- net /SS_INERTIA_SWITCH: track 0.00 -> 8.03 mm
- net /SS_COCKPIT_ESTOP: track 0.00 -> 8.03 mm
- net /SS_BOTS_OUT: track 0.00 -> 7.97 mm
- net Net-(D4-Pad2): track 0.00 -> 7.95 mm
- net /SS_ESTOP_OUT: track 0.00 -> 6.70 mm
- net Net-(D8-Pad2): track 0.00 -> 6.41 mm
- net Net-(D6-Pad2): track 0.00 -> 6.39 mm
- net /SS_INERTIA_OUT: track 0.00 -> 5.93 mm
- net Net-(C103-Pad1): track 2.39 -> 5.44 mm
- net Net-(C103-Pad2): track 5.44 -> 2.39 mm
Other:
- board text added: "5V"
