File: Boards/Tire_Temperature/_autosave-tire_temp.kicad_pcb (KiCad board)
At the start: 2 copper layers, 109.3 x 58.3 mm, 54 parts, among them J1 CONN_02X03, J2 CONN_02X03, U1 LM3480, U101 TPS560430YF, U2 ATMEGA16M1, U3 TXB0104, U4 MCP2561-E_SN, U6 ATmega328P-AU, Y1 Crystal_SMD, Y2 Crystal_SMD

Commit message: Revert "Begin Layout"
This reverts commit f66e97611986f6cb10e89dffa2fa205961dd2a3d.
Parts:
- added REF**: MLX90621ESF-BAB-000-TU, footprints:MLX90621ESF-BAB-000-TU, F.Cu at (181.0, 82.0)
- moved R7 11.3 mm to (187.3, 122.6)
- moved C3 10.4 mm to (116.2, 113.2)
- moved C4 10.4 mm to (121.4, 117.9)
- moved U1 10.4 mm to (120.4, 113.8)
- moved R6 10.2 mm to (190.0, 85.7)
- moved R8 6.82 mm to (189.8, 79.6)
- moved R9 3.07 mm to (187.1, 95.5)
- moved U4 3.07 mm to (180.8, 95.6)
- moved C8 2.72 mm to (174.6, 95.6)
- moved R10 0.31 mm to (191.6, 98.7)
Routing:
- net /12V: track 12.9 -> 3.87 mm
Changed lines of the file:
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@@
     (thickness 1.6)
     (drawings 6)
-    (tracks 100)
+    (tracks 99)
     (zones 0)
-    (modules 54)
+    (modules 55)
     (nets 77)
   )
@@
     (add_net VCC)
   )
+  (module footprints:MLX90621ESF-BAB-000-TU (layer F.Cu)
+    (at 180.975 82.042)
+    (fp_text reference REF** (at 0 0.5) (layer F.SilkS)
+      (effects (font (size 1 1) (thickness 0.15)))
+    )
+    (fp_text value MLX90621ESF-BAB-000-TU (at 0 -0.5) (layer F.Fab)
+      (effects (font (size 1 1) (thickness 0.15)))
+    )
+    (fp_circle (center 0 0) (end 2.54 0) (layer Dwgs.User) (width 0.12))
+    (fp_circle (center 0 0) (end 4.575 0) (layer F.SilkS) (width 0.12))
+    (pad 4 thru_hole circle (at -2.54 0) (size 1.524 1.524) (drill 0.762) (layers *.Cu *.Mask))
+    (pad 3 thru_hole circle (at 0 2.54) (size 1.524 1.524) (drill 0.762) (layers *.Cu *.Mask))
+    (pad 2 thru_hole circle (at 2.54 0) (size 1.524 1.524) (drill 0.762) (layers *.Cu *.Mask))
+    (pad 1 thru_hole circle (at 0 -2.54) (size 1.524 1.524) (drill 0.762) (layers *.Cu *.Mask))
+  )
   (module footprints:phoenix (layer B.Cu)
     (at 179.578 107.188 180)
@@
   )
   (module footprints:C_0805_OEM (layer F.Cu)
-    (at 114.554 123.444)
+    (at 116.205 113.157)
     (descr "Capacitor SMD 0805, reflow soldering, AVX (see smccp.pdf)")
     (tags "capacitor 0805")
@@
   )
   (module footprints:C_0805_OEM (layer F.Cu)
-    (at 119.777 128.143)
+    (at 121.428 117.856)
     (descr "Capacitor SMD 0805, reflow soldering, AVX (see smccp.pdf)")
     (tags "capacitor 0805")
@@
   )
   (module footprints:C_0805_OEM (layer F.Cu)
-    (at 176.784 93.98 90)
+    (at 174.625 95.631 90)
     (descr "Capacitor SMD 0805, reflow soldering, AVX (see smccp.pdf)")
     (tags "capacitor 0805")
@@
   )
   (module footprints:R_0805_OEM (layer F.Cu)
-    (at 200.152 85.09)
+    (at 189.992 85.725)
     (descr "Resistor SMD 0805, reflow soldering, Vishay (see dcrcw.pdf)")
     (tags "resistor 0805")
@@
   )
   (module footprints:R_0805_OEM (layer F.Cu)
-    (at 186.756 133.858)
+    (at 187.325 122.555)
     (descr "Resistor SMD 0805, reflow soldering, Vishay (see dcrcw.pdf)")
     (tags "resistor 0805")
@@
   )
   (module footprints:R_0805_OEM (layer F.Cu)
-    (at 195.072 83.947)
+    (at 189.799 79.629)
     (descr "Resistor SMD 0805, reflow soldering, Vishay (see dcrcw.pdf)")
     (tags "resistor 0805")
@@
   )
   (module footprints:R_0805_OEM (layer F.Cu)
-    (at 189.55 93.599 270)
+    (at 187.137 95.504 270)
     (descr "Resistor SMD 0805, reflow soldering, Vishay (see dcrcw.pdf)")
     (tags "resistor 0805")
@@
   )
   (module footprints:R_0805_OEM (layer F.Cu)
-    (at 191.643 99.06 270)
+    (at 191.643 98.745 270)
     (descr "Resistor SMD 0805, reflow soldering, Vishay (see dcrcw.pdf)")
     (tags "resistor 0805")
@@
   )
   (module footprints:SOT-23-3_OEM (layer F.Cu)
-    (at 118.745 124.079)
+    (at 120.396 113.792)
     (descr "5-pin SOT23 package")
     (tags SOT-23-5)
@@
   )
   (module footprints:SOIC-8_3.9x4.9mm_Pitch1.27mm_OEM (layer F.Cu)
-    (at 183.228 93.726)
+    (at 180.815 95.631)
     (descr "8-Lead Plastic Small Outline (SN) - Narrow, 3.90 mm Body [SOIC] (see Microchip Packaging Specification 00000049BS.pdf)")
     (tags "SOIC 1.27")
@@
   (segment (start 116.90666 105.77514) (end 116.9543 105.7275) (width 0.381) (layer F.Cu) (net 2))
   (segment (start 116.78666 105.89514) (end 116.9543 105.7275) (width 0.381) (layer F.Cu) (net 2))
-  (segment (start 107.7341 105.89514) (end 116.78666 105.89514) (width 0.381) (layer F.Cu) (net 2))
   (segment (start 116.9543 105.7275) (end 120.5208 105.7275) (width 0.381) (layer F.Cu) (net 2))
   (segment (start 125.7 110.52388) (end 125.7 111.796) (width 0.254) (layer F.Cu) (net 3))
