File: Boards/BMS_Core/BMS_core.sch (KiCad schematic (older format))
At the start: 72 parts, among them IC1 ATMEGA16M1, J1 CONN_02X03, J2 B5B-PH-K-S, J3 MM_F_VT_20, J4 MicroFit_V_2, J5 isoSPI-Cutout, K1 G5Q-1A4-DC5-5V, Q1 SSM3K333R, T1 T_LAN_7490100111A, U1 MCP2561-E_SN, U101 TPS561201, U2 SN74LVC1G17, U3 LTC6820HMS, U4 MCP6001, U5 MCP6001, U6 MCP6001, U7 SN74LVC1G32, Y1 Crystal_SMD

Commit message: update BMS Core schemtic)
Connections:
- no-connect marks 13 -> 11
Changed lines of the file:
@@
-$EndComp
-$Comp
-L formula:ATMEGA16M1 IC?
-U 1 1 5C6BBC18
-P 2650 3650
-AR Path="/5C6B723E/5C6BBC18" Ref="IC?"  Part="1"
-AR Path="/5C6BBC18" Ref="IC1"  Part="1"
-F 0 "IC1" H 1700 5480 50  0000 L BNN
-F 1 "ATMEGA16M1" H 3150 2250 50  0000 L BNN
-F 2 "footprints:TQFP-32_7x7mm_Pitch0.8mm" H 2650 3650 50  0001 C CIN
-F 3 "http://www.atmel.com/Images/Atmel-8209-8-bit%20AVR%20ATmega16M1-32M1-64M1_Datasheet.pdf" H 1700 5480 50  0001 C CNN
-F 4 "ATMEGA16M1-AU-ND" H 2650 3650 60  0001 C CNN "MPN"
-F 5 "Digi-Key" H 2650 3650 60  0001 C CNN "MFN"
-F 6 "Value" H 2650 3650 60  0001 C CNN "Package"
-F 7 "https://www.digikey.com/product-detail/en/atmel/ATMEGA16M1-AU/ATMEGA16M1-AU-ND/2271208" H 2100 5880 60  0001 C CNN "PurchasingLink"
-	1    2650 3650
-	1    0    0    -1
 $EndComp
 $Comp
@@
 	1350 1950 1550 1950
 Connection ~ 1350 2250
-Connection ~ 1550 4850
 Connection ~ 3750 4950
 Connection ~ 4050 4950
@@
 GND SHORT\nDETECTION
 NoConn ~ 3750 2450
-NoConn ~ 3750 3750
-NoConn ~ 3750 3850
 $Comp
 L formula:MicroFit_V_2 J4
@@
 Wire Wire Line
 	10550 2350 10550 2550
+Text Label 3750 3750 0    50   ~ 0
+Charge-Enable-1
+Connection ~ 1550 4850
+$Comp
+L formula:ATMEGA16M1 IC?
+U 1 1 5C6BBC18
+P 2650 3650
+AR Path="/5C6B723E/5C6BBC18" Ref="IC?"  Part="1"
+AR Path="/5C6BBC18" Ref="IC1"  Part="1"
+F 0 "IC1" H 1700 5480 50  0000 L BNN
+F 1 "ATMEGA16M1" H 3150 2250 50  0000 L BNN
+F 2 "footprints:TQFP-32_7x7mm_Pitch0.8mm" H 2650 3650 50  0001 C CIN
+F 3 "http://www.atmel.com/Images/Atmel-8209-8-bit%20AVR%20ATmega16M1-32M1-64M1_Datasheet.pdf" H 1700 5480 50  0001 C CNN
+F 4 "ATMEGA16M1-AU-ND" H 2650 3650 60  0001 C CNN "MPN"
+F 5 "Digi-Key" H 2650 3650 60  0001 C CNN "MFN"
+F 6 "Value" H 2650 3650 60  0001 C CNN "Package"
+F 7 "https://www.digikey.com/product-detail/en/atmel/ATMEGA16M1-AU/ATMEGA16M1-AU-ND/2271208" H 2100 5880 60  0001 C CNN "PurchasingLink"
+	1    2650 3650
+	1    0    0    -1
+$EndComp
+Text Label 3750 3850 0    50   ~ 0
+Charge-Enable-2
 $EndSCHEMATC

Commit message: Added bypass cap to Logic block; new core layout for ss layout
Parts:
- removed C101: C_22uF, footprints:C_1206_OEM, symbol formula:C_22uF
- removed C104: C_1uF, footprints:C_0805_OEM, symbol formula:C_1uF
- removed C105: C_0.1uF, footprints:C_0805_OEM, symbol formula:C_0.1uF
- removed L101: L_4.7uH, footprints:4.7uH_Inductor_OEM, symbol formula:L_4.7uH
- removed R102: R_10K, footprints:R_0805_OEM, symbol formula:R_10K
- removed U101: TPS561201, footprints:SOT-23-6_OEM, symbol formula:TPS561201
- added C101: C_2.2uF, footprints:C_0603_1608Metric, symbol footprints:C_2.2uF
- added C102: C_0.1uF, footprints:C_0805_OEM, symbol footprints:C_0.1uF
- added C12: C_0.1uF, footprints:C_0805_OEM, symbol formula:C_0.1uF
- added COUT102: C_22uF, footprints:C_1206_OEM, symbol footprints:C_22uF
- added COUT103: C_33uF, footprints:Fuse_1812, symbol footprints:C_33uF
- added L101: L_100uH, footprints:L_100uH_OEM, symbol formula:L_100uH
- added U8: TPS560430YF, footprints:SOT-23-6_OEM, symbol formula:TPS560430YF
- R102: renamed from R103; value R_10K -> R_25K
- R103: renamed from R104; value R_54.9K -> R_100K
- renumbered C102 to C103, C103 to COUT101, R105 to R104, R106 to R105
Connections:
- net labels removed: Charge-Enable-1, Charge-Enable-2
- wire segments 263 -> 267
- no-connect marks 11 -> 13
Other:
- note added: "Input Capacitors"
- note removed: "Input Capacitor"
- moved on the sheet: C103, D101, D102, F101, R101

Commit message: new transformer, mounting hole, moved I sensor
Parts:
- removed T1: T_LAN_7490100111A, footprints:T_LAN_7490100111A, symbol formula:T_LAN_7490100111A
- added T1: T_LAN_SM91501ALE, footprints:T_LAN_SM91501ALE, symbol footprints:T_LAN_SM91501ALE
Other:
- note removed: "Common-Mode Choke"
Changed lines of the file:
@@
 	3850 7050 4050 7050
-$Comp
-L formula:T_LAN_7490100111A T1
-U 1 1 5C6CFBB6
-P 10650 3100
-F 0 "T1" H 11150 4150 60  0000 C CNN
-F 1 "T_LAN_7490100111A" H 11600 2700 60  0000 C CNN
-F 2 "footprints:T_LAN_7490100111A" H 11050 4050 60  0001 C CNN
-F 3 "https://katalog.we-online.de/pbs/datasheet/7490100111A.pdf" H 10650 3100 60  0001 C CNN
-F 4 "DK" H 11000 3600 60  0001 C CNN "MFN"
-F 5 "732-5711-1-ND" H 10900 3500 60  0001 C CNN "MPN"
-F 6 "https://www.digikey.com/product-detail/en/wurth-electronics-inc/7490100111A/732-5711-1-ND/4969381" H 10800 3400 60  0001 C CNN "PurchasingLink"
-	1    10650 3100
-	-1   0    0    -1
-$EndComp
 $Comp
 L power:PWR_FLAG #FLG?
@@
 Text Notes 7450 1850 0    50   ~ 0
 120 Ohm Termination
-Text Notes 8800 2050 0    50   ~ 0
-Common-Mode Choke
 Text Notes 9750 1900 0    50   ~ 0
 Isolation Transformer
@@
 Text Label 12650 2750 0    50   ~ 0
 GND
+$Comp
+L footprints:T_LAN_SM91501ALE T1
+U 1 1 5EF8F2AF
+P 10650 3100
+F 0 "T1" H 11525 4297 60  0000 C CNN
+F 1 "T_LAN_SM91501ALE" H 11525 4191 60  0000 C CNN
+F 2 "footprints:T_LAN_SM91501ALE" H 11050 4050 60  0001 C CNN
+F 3 "https://www.mouser.com/datasheet/2/54/sm91501al-1488891.pdf" H 10650 3100 60  0001 C CNN
+F 4 "DK" H 11000 3600 60  0001 C CNN "MFN"
+F 5 "SM91501ALE" H 10900 3500 60  0001 C CNN "MPN"
+F 6 "https://www.digikey.si/product-detail/en/bourns-inc/SM91501ALE/SM91501ALETR-ND/9650127" H 10800 3400 60  0001 C CNN "PurchasingLink"
+	1    10650 3100
+	-1   0    0    -1
+$EndComp
 $EndSCHEMATC

Commit message: BMS core changes
Parts:
- removed K1: G5Q-1A4-DC5-5V, footprints:Relay_SPST_OMRON-G5Q-1A4_OEM, symbol formula:G5Q-1A4-DC5-5V
- added C13: C_0.1uF, footprints:C_0805_OEM, symbol formula:C_0.1uF
- added K?: G5Q-1A4-DC12, footprints:Relay_SPST_OMRON-G5Q-1A4_OEM, symbol footprints:G5Q-1A4-DC12
- added TP1, TP2, TP3, TP4, TP5: Test_Point_SMD, footprints:Test_Point_SMD, symbol formula:Test_Point_SMD
- R8: value R_3.01K -> R_1K
Connections:
- net labels added: CHARGE_ENABLE1, IM, IP
- wire segments 267 -> 270
- no-connect marks 13 -> 12
Other:
- note added: "GND\n12V\n5V_BMS\nMISO_BMS\nMOSI_BMS\nSCK_BMS\nRESET_BMS\nRJ45_LED_O_BMS\nRJ45_LED_G_BMS\nCAN HIGH\nCAN LOW\nBPSD CURRENT SENSE\nFAN PWM\nBMS SENSE\nGND\nGND\nGND\nGND\nCHARGE ENABLE 1\nGND"
- note removed: "GND\n12V\n5V_BMS\nMISO_BMS\nMOSI_BMS\nSCK_BMS\nRESET_BMS\nRJ45_LED_O_BMS\nRJ45_LED_G_BMS\nCAN HIGH\nCAN LOW\nBPSD CURRENT SENSE\nFAN PWM\nBMS SENSE\nCHARGE ENABLE 1\nCHARGE ENABLE 2\nGND\nGND\nGND\nGND"
Changed lines of the file:
@@
-$EndComp
-$Comp
-L formula:G5Q-1A4-DC5-5V K1
-U 1 1 5C831541
-P 8800 8800
-F 0 "K1" H 9150 8950 50  0000 L CNN
-F 1 "G5Q-1A4-DC5-5V" H 8400 8650 50  0000 L CNN
-F 2 "footprints:Relay_SPST_OMRON-G5Q-1A4_OEM" H 9250 8750 50  0001 L CNN
-F 3 "http://omronfs.omron.com/en_US/ecb/products/pdf/en-g5q.pdf" H 9250 8450 50  0001 L CNN
-F 4 "DK" H 9650 9350 60  0001 C CNN "MFN"
-F 5 "Z3632-ND" H 9550 9250 60  0001 C CNN "MPN"
-F 6 "https://www.digikey.com/product-detail/en/omron-electronics-inc-emc-div/G5Q-1A4-DC5/Z3632-ND/1815721" H 9750 9450 60  0001 C CNN "PurchasingLink"
-	1    8800 8800
-	1    0    0    -1
 $EndComp
 $Comp
@@
 L power:VCC #PWR020
 U 1 1 5C93825A
-P 5500 1900
-F 0 "#PWR020" H 5500 1750 50  0001 C CNN
-F 1 "VCC" H 5500 2050 50  0000 C CNN
-F 2 "" H 5500 1900 50  0001 C CNN
-F 3 "" H 5500 1900 50  0001 C CNN
-	1    5500 1900
+P 5500 1825
+F 0 "#PWR020" H 5500 1675 50  0001 C CNN
+F 1 "VCC" H 5500 1975 50  0000 C CNN
+F 2 "" H 5500 1825 50  0001 C CNN
+F 3 "" H 5500 1825 50  0001 C CNN
+	1    5500 1825
 	1    0    0    -1
 $EndComp
@@
 P 6700 2850
 F 0 "R8" V 6780 2850 50  0000 C CNN
-F 1 "R_3.01K" V 6600 2850 50  0000 C CNN
+F 1 "R_1K" V 6600 2850 50  0000 C CNN
 F 2 "footprints:R_0805_OEM" H 6630 2850 50  0001 C CNN
 F 3 "http://www.yageo.com.tw/exep/pages/download/literatures/PYu-R_INT-thick_7.pdf" H 6780 2850 50  0001 C CNN
@@
 $EndComp
 Text Notes 14500 3150 0    50   ~ 0
-GND\n12V\n5V_BMS\nMISO_BMS\nMOSI_BMS\nSCK_BMS\nRESET_BMS\nRJ45_LED_O_BMS\nRJ45_LED_G_BMS\nCAN HIGH\nCAN LOW\nBPSD CURRENT SENSE\nFAN PWM\nBMS SENSE\nCHARGE ENABLE 1\nCHARGE ENABLE 2\nGND\nGND\nGND\nGND
+GND\n12V\n5V_BMS\nMISO_BMS\nMOSI_BMS\nSCK_BMS\nRESET_BMS\nRJ45_LED_O_BMS\nRJ45_LED_G_BMS\nCAN HIGH\nCAN LOW\nBPSD CURRENT SENSE\nFAN PWM\nBMS SENSE\nGND\nGND\nGND\nGND\nCHARGE ENABLE 1\nGND
 Wire Notes Line
 	13950 800  11900 800
@@
 GND
 Text Label 12650 2950 0    50   ~ 0
-GND
-Text Label 12650 3050 0    50   ~ 0
 GND
 Text Label 12650 3150 0    50   ~ 0
@@
 Wire Wire Line
 	12000 4975 12000 5000
-NoConn ~ 3750 3750
 NoConn ~ 3750 3850
 Wire Wire Line
@@
 	-1   0    0    -1
 $EndComp
+Text Label 3750 3750 0    50   ~ 0
+CHARGE_ENABLE1
+Text Label 12650 3050 0    50   ~ 0
+CHARGE_ENABLE1
+$Comp
+L formula:C_0.1uF C13
+U 1 1 5E486BF9
+P 5350 1900
+F 0 "C13" V 5300 1700 50  0000 L CNN
+F 1 "C_0.1uF" V 5400 1550 50  0000 L CNN
+F 2 "footprints:C_0805_OEM" H 5388 1750 50  0001 C CNN
+F 3 "http://datasheets.avx.com/X7RDielectric.pdf" H 5375 2000 50  0001 C CNN
+F 4 "478-3352-1-ND" H 5350 1900 60  0001 C CNN "MPN"
+F 5 "Digi-Key" H 5350 1900 60  0001 C CNN "MFN"
+F 6 "Value" H 5350 1900 60  0001 C CNN "Package"
+F 7 "https://www.digikey.com/products/en?keywords=478-3352-1-ND" H 5775 2400 60  0001 C CNN "PurchasingLink"
+	1    5350 1900
+	0    1    -1   0
+$EndComp
+$Comp
+L power:GND #PWR052
+U 1 1 5E486BFF
+P 5100 1950
+F 0 "#PWR052" H 5100 1700 50  0001 C CNN
+F 1 "GND" H 5100 1800 50  0000 C CNN
+F 2 "" H 5100 1950 50  0001 C CNN
+F 3 "" H 5100 1950 50  0001 C CNN
+	1    5100 1950
+	-1   0    0    -1
+$EndComp
+Wire Wire Line
+	5200 1900 5100 1900
+Connection ~ 5500 1900
+Wire Wire Line
+	5100 1900 5100 1950
+Wire Wire Line
+	5500 1825 5500 1900
+$Comp
+L formula:Test_Point_SMD TP1
+U 1 1 5E4C6F2A
+P 13850 4175
+F 0 "TP1" V 13850 4450 50  0000 C CNN
+F 1 "Test_Point_SMD" H 13928 4172 50  0001 L CNN
+F 2 "footprints:Test_Point_SMD" H 13850 4025 50  0001 C CNN
+F 3 "" H 13850 4175 50  0001 C CNN
+	1    13850 4175
+	0    -1   -1   0
+$EndComp
+$Comp
+L formula:Test_Point_SMD TP2
+U 1 1 5E4DC281
+P 13850 4400
+F 0 "TP2" V 13850 4675 50  0000 C CNN
+F 1 "Test_Point_SMD" H 13928 4397 50  0001 L CNN
+F 2 "footprints:Test_Point_SMD" H 13850 4250 50  0001 C CNN
+F 3 "" H 13850 4400 50  0001 C CNN
+	1    13850 4400
+	0    -1   -1   0
+$EndComp
+$Comp
+L formula:Test_Point_SMD TP3
+U 1 1 5E4F03E3
+P 13850 4725
+F 0 "TP3" V 13850 4925 50  0000 L CNN
+F 1 "Test_Point_SMD" H 13928 4722 50  0001 L CNN
+F 2 "footprints:Test_Point_SMD" H 13850 4575 50  0001 C CNN
+F 3 "" H 13850 4725 50  0001 C CNN
+	1    13850 4725
+	0    -1   -1   0
+$EndComp
+Text Label 13900 4725 0    50   ~ 0
+BSPD_CURRENT
+$Comp
+L power:GND #PWR0116
+U 1 1 5E542E39
+P 13900 4400
+F 0 "#PWR0116" H 13900 4150 50  0001 C CNN
+F 1 "GND" H 13905 4227 50  0000 C CNN
+F 2 "" H 13900 4400 50  0001 C CNN
+F 3 "" H 13900 4400 50  0001 C CNN
+	1    13900 4400
+	1    0    0    -1
+$EndComp
+$Comp
+L power:+12V #PWR?
+U 1 1 5E54444B
+P 13900 4175
+AR Path="/5C6B723E/5E54444B" Ref="#PWR?"  Part="1"
+AR Path="/5E54444B" Ref="#PWR0117"  Part="1"
+AR Path="/5C702479/5E54444B" Ref="#PWR?"  Part="1"
+F 0 "#PWR0117" H 13900 4025 50  0001 C CNN
+F 1 "+12V" H 13900 4315 50  0000 C CNN
+F 2 "" H 13900 4175 50  0001 C CNN
+F 3 "" H 13900 4175 50  0001 C CNN
+	1    13900 4175
+	1    0    0    -1
+$EndComp
+$Comp
+L formula:Test_Point_SMD TP4
+U 1 1 5E5FD1CA
+P 13850 4950
+F 0 "TP4" V 13850 5225 50  0000 C CNN
+F 1 "Test_Point_SMD" H 13928 4947 50  0001 L CNN
+F 2 "footprints:Test_Point_SMD" H 13850 4800 50  0001 C CNN
+F 3 "" H 13850 4950 50  0001 C CNN
+	1    13850 4950
+	0    -1   -1   0
+$EndComp
+$Comp
+L formula:Test_Point_SMD TP5
+U 1 1 5E5FD1D0
+P 13850 5175
+F 0 "TP5" V 13850 5450 50  0000 C CNN
+F 1 "Test_Point_SMD" H 13928 5172 50  0001 L CNN
+F 2 "footprints:Test_Point_SMD" H 13850 5025 50  0001 C CNN
+F 3 "" H 13850 5175 50  0001 C CNN
+	1    13850 5175
+	0    -1   -1   0
+$EndComp
+Text Label 10550 2150 0    50   ~ 0
+IM
+Text Label 10550 2550 0    50   ~ 0
+IP
+Text Label 13900 4950 0    50   ~ 0
+IM
+Text Label 13900 5175 0    50   ~ 0
+IP
+$Comp
+L footprints:G5Q-1A4-DC12 K?
+U 1 1 5E4512AF
+P 8800 8800
+F 0 "K?" H 9130 8846 50  0000 L CNN
+F 1 "G5Q-1A4-DC12" H 9130 8755 50  0000 L CNN
+F 2 "footprints:Relay_SPST_OMRON-G5Q-1A4_OEM" H 8650 9200 50  0001 C CNN
+F 3 "https://omronfs.omron.com/en_US/ecb/products/pdf/en-g5q.pdf" H 8750 9300 50  0001 C CNN
+	1    8800 8800
+	1    0    0    -1
+$EndComp
 $EndSCHEMATC

Commit message: Final, and slight, changes to layout
Parts:
- added CANH, CANL: TP, footprints:tp_1.6mm, symbol formula:TP
- gave numbers to parts that had none: 1
- renumbered TP1 to 12V1, TP3 to BSPD1, TP2 to GND1, TP4 to IM1, TP5 to IP1, D1 to PD5, D2 to PD6, D3 to PD7
Connections:
- net CANH: now also CANH.1 (TP)
- net CANL: now also CANL.1 (TP)
Changed lines of the file:
@@
 	3850 2550 3750 2550
 $Comp
-L formula:LED_0805 D1
+L formula:LED_0805 PD5
 U 1 1 5C6F857F
 P 1000 6750
-F 0 "D1" H 1000 6650 50  0000 C CNN
+F 0 "PD5" H 1000 6650 50  0000 C CNN
 F 1 "LED_0805" H 1000 6850 50  0000 C CNN
 F 2 "footprints:LED_0805_OEM" H 900 6750 50  0001 C CNN
@@
 $EndComp
 $Comp
-L formula:LED_0805 D2
+L formula:LED_0805 PD6
 U 1 1 5C6F87B3
 P 1400 6750
-F 0 "D2" H 1400 6650 50  0000 C CNN
+F 0 "PD6" H 1400 6650 50  0000 C CNN
 F 1 "LED_0805" H 1400 6850 50  0000 C CNN
 F 2 "footprints:LED_0805_OEM" H 1300 6750 50  0001 C CNN
@@
 $EndComp
 $Comp
-L formula:LED_0805 D3
+L formula:LED_0805 PD7
 U 1 1 5C6F88AF
 P 1800 6750
-F 0 "D3" H 1800 6650 50  0000 C CNN
+F 0 "PD7" H 1800 6650 50  0000 C CNN
 F 1 "LED_0805" H 1800 6850 50  0000 C CNN
 F 2 "footprints:LED_0805_OEM" H 1700 6750 50  0001 C CNN
@@
 	5500 1825 5500 1900
 $Comp
-L formula:Test_Point_SMD TP1
+L formula:Test_Point_SMD 12V1
 U 1 1 5E4C6F2A
 P 13850 4175
-F 0 "TP1" V 13850 4450 50  0000 C CNN
+F 0 "12V1" V 13850 4450 50  0000 C CNN
 F 1 "Test_Point_SMD" H 13928 4172 50  0001 L CNN
 F 2 "footprints:Test_Point_SMD" H 13850 4025 50  0001 C CNN
@@
 $EndComp
 $Comp
-L formula:Test_Point_SMD TP2
+L formula:Test_Point_SMD GND1
 U 1 1 5E4DC281
 P 13850 4400
-F 0 "TP2" V 13850 4675 50  0000 C CNN
+F 0 "GND1" V 13850 4675 50  0000 C CNN
 F 1 "Test_Point_SMD" H 13928 4397 50  0001 L CNN
 F 2 "footprints:Test_Point_SMD" H 13850 4250 50  0001 C CNN
@@
 $EndComp
 $Comp
-L formula:Test_Point_SMD TP3
+L formula:Test_Point_SMD BSPD1
 U 1 1 5E4F03E3
 P 13850 4725
-F 0 "TP3" V 13850 4925 50  0000 L CNN
+F 0 "BSPD1" V 13850 4925 50  0000 L CNN
 F 1 "Test_Point_SMD" H 13928 4722 50  0001 L CNN
 F 2 "footprints:Test_Point_SMD" H 13850 4575 50  0001 C CNN
@@
 $EndComp
 $Comp
-L formula:Test_Point_SMD TP4
+L formula:Test_Point_SMD IM1
 U 1 1 5E5FD1CA
 P 13850 4950
-F 0 "TP4" V 13850 5225 50  0000 C CNN
+F 0 "IM1" V 13850 5225 50  0000 C CNN
 F 1 "Test_Point_SMD" H 13928 4947 50  0001 L CNN
 F 2 "footprints:Test_Point_SMD" H 13850 4800 50  0001 C CNN
@@
 $EndComp
 $Comp
-L formula:Test_Point_SMD TP5
+L formula:Test_Point_SMD IP1
 U 1 1 5E5FD1D0
 P 13850 5175
-F 0 "TP5" V 13850 5450 50  0000 C CNN
+F 0 "IP1" V 13850 5450 50  0000 C CNN
 F 1 "Test_Point_SMD" H 13928 5172 50  0001 L CNN
 F 2 "footprints:Test_Point_SMD" H 13850 5025 50  0001 C CNN
@@
 IP
 $Comp
-L footprints:G5Q-1A4-DC12 K?
+L footprints:G5Q-1A4-DC12 K1
 U 1 1 5E4512AF
 P 8800 8800
-F 0 "K?" H 9130 8846 50  0000 L CNN
+F 0 "K1" H 9130 8846 50  0000 L CNN
 F 1 "G5Q-1A4-DC12" H 9130 8755 50  0000 L CNN
 F 2 "footprints:Relay_SPST_OMRON-G5Q-1A4_OEM" H 8650 9200 50  0001 C CNN
@@
 	1    0    0    -1
 $EndComp
+Text Label 13900 5400 0    50   ~ 0
+CANH
+Text Label 13900 5600 0    50   ~ 0
+CANL
+$Comp
+L formula:TP CANH
+U 1 1 5E47CC53
+P 13700 5400
+F 0 "CANH" V 13700 5525 50  0000 C CNN
+F 1 "TP" V 13824 5292 50  0001 C CNN
+F 2 "footprints:tp_1.6mm" H 13600 5300 50  0001 C CNN
+F 3 "http://www.keyelco.com/product-pdf.cfm?p=1314" H 13700 5400 50  0001 C CNN
+F 4 "DK" H 13800 5500 50  0001 C CNN "MFN"
+F 5 "36-5006-ND" H 13900 5600 50  0001 C CNN "MPN"
+F 6 "https://www.digikey.com/product-detail/en/keystone-electronics/5006/36-5006-ND/255330" H 14000 5700 50  0001 C CNN "PurchasingLink"
+	1    13700 5400
+	0    -1   -1   0
+$EndComp
+$Comp
+L formula:TP CANL
+U 1 1 5E4B9979
+P 13700 5600
+F 0 "CANL" V 13700 5725 50  0000 C CNN
+F 1 "TP" V 13824 5492 50  0001 C CNN
+F 2 "footprints:tp_1.6mm" H 13600 5500 50  0001 C CNN
+F 3 "http://www.keyelco.com/product-pdf.cfm?p=1314" H 13700 5600 50  0001 C CNN
+F 4 "DK" H 13800 5700 50  0001 C CNN "MFN"
+F 5 "36-5006-ND" H 13900 5800 50  0001 C CNN "MPN"
+F 6 "https://www.digikey.com/product-detail/en/keystone-electronics/5006/36-5006-ND/255330" H 14000 5900 50  0001 C CNN "PurchasingLink"
+	1    13700 5600
+	0    -1   -1   0
+$EndComp
 $EndSCHEMATC

Commit message: BMS core rev1.0 for shipment
Parts:
- renumbered CANH to CANH1, CANL to CANL1
Changed lines of the file:
@@
 CANL
 $Comp
-L formula:TP CANH
+L formula:TP CANH1
 U 1 1 5E47CC53
 P 13700 5400
-F 0 "CANH" V 13700 5525 50  0000 C CNN
+F 0 "CANH1" V 13700 5525 50  0000 C CNN
 F 1 "TP" V 13824 5292 50  0001 C CNN
 F 2 "footprints:tp_1.6mm" H 13600 5300 50  0001 C CNN
@@
 $EndComp
 $Comp
-L formula:TP CANL
+L formula:TP CANL1
 U 1 1 5E4B9979
 P 13700 5600
-F 0 "CANL" V 13700 5725 50  0000 C CNN
+F 0 "CANL1" V 13700 5725 50  0000 C CNN
 F 1 "TP" V 13824 5492 50  0001 C CNN
 F 2 "footprints:tp_1.6mm" H 13600 5500 50  0001 C CNN

Commit message: modify Perhiperal and fix opamp volage divider on Core
Parts:
- removed R14: R_1K_0.1, footprints:R_0805_OEM, symbol formula:R_1K_0.1
- removed R21: R_14.3K, footprints:R_0805_OEM, symbol formula:R_17.8K
- added R?: R_475, footprints:R_0805_OEM, symbol formula:R_475
- added R?: R_10K, footprints:R_0805_OEM, symbol formula:R_10K
- C101: symbol footprints:C_2.2uF -> BMS_core-rescue:C_2.2uF-footprints
- C102: symbol footprints:C_0.1uF -> BMS_core-rescue:C_0.1uF-footprints
- COUT102: symbol footprints:C_22uF -> BMS_core-rescue:C_22uF-footprints
- COUT103: symbol footprints:C_33uF -> BMS_core-rescue:C_33uF-footprints
- K1: symbol footprints:G5Q-1A4-DC12 -> BMS_core-rescue:G5Q-1A4-DC12-footprints
- T1: symbol footprints:T_LAN_SM91501ALE -> BMS_core-rescue:T_LAN_SM91501ALE-footprints
- U7: symbol formula:SN74LVC1G32 -> BMS_core-rescue:SN74LVC1G32-formula
Connections:
- net GND: now also R?.1
- net VCC: now also R?.2
- net at U5.4 (-): now also R?.1, R?.2
Other:
- note added: "5kW/346V = 14.45A\n16 mV/A * 14.45A = 231mV\n"
- note removed: "5kW/240V = 20.83A\n16 mV/A * 20.83A = 333mV\n1K/14.3K * 5V = 333mV"
Changed lines of the file:
@@
 EESchema Schematic File Version 4
-LIBS:BMS_core-cache
 EELAYER 30 0
 EELAYER END
@@
 Unity-gain buffer vs. VREF
 Text Notes 9450 6550 0    50   ~ 0
-5kW/240V = 20.83A\n16 mV/A * 20.83A = 333mV\n1K/14.3K * 5V = 333mV
+5kW/346V = 14.45A\n16 mV/A * 14.45A = 231mV\n
 Text Label 6200 4600 0    50   ~ 0
 VOUT
-$Comp
-L formula:R_1K_0.1 R14
-U 1 1 5C9F0930
-P 10350 6100
-F 0 "R14" V 10430 6100 50  0000 C CNN
-F 1 "R_1K_0.1" V 10250 6100 50  0000 C CNN
-F 2 "footprints:R_0805_OEM" H 10280 6100 50  0001 C CNN
-F 3 "https://industrial.panasonic.com/cdbs/www-data/pdf/RDM0000/AOA0000C307.pdf" H 10430 6100 50  0001 C CNN
-F 4 "DK" H 10350 6100 60  0001 C CNN "MFN"
-F 5 "P1.0KDACT-ND" H 10350 6100 60  0001 C CNN "MPN"
-F 6 "https://www.digikey.com/product-detail/en/panasonic-electronic-components/ERA-6AEB102V/P1.0KDACT-ND/1465947" H 10830 6500 60  0001 C CNN "PurchasingLink"
-	1    10350 6100
-	0    -1   -1   0
-$EndComp
 Wire Wire Line
 	9600 6050 9600 6100
@@
 	9200 5750 10750 5750
 $Comp
-L formula:R_17.8K R21
-U 1 1 5CF2B53E
-P 9850 6100
-F 0 "R21" V 9643 6100 50  0000 C CNN
-F 1 "R_14.3K" V 9734 6100 50  0000 C CNN
-F 2 "footprints:R_0805_OEM" H 9850 6050 50  0001 C CNN
-F 3 "" H 9950 6150 50  0001 C CNN
-F 4 "DK" H 10050 6250 50  0001 C CNN "MFN"
-F 5 "" H 10150 6350 50  0001 C CNN "MPN"
-F 6 "" H 10350 6550 50  0001 C CNN "PurchasingLink"
-	1    9850 6100
-	0    1    1    0
-$EndComp
-$Comp
 L formula:MCP6001 U6
 U 1 1 5CF2C95C
@@
 0.45V
 $Comp
-L formula:SN74LVC1G32 U7
+L BMS_core-rescue:SN74LVC1G32-formula U7
 U 1 1 5CFD6270
 P 12000 5350
@@
 $EndComp
 $Comp
-L footprints:C_22uF COUT102
+L BMS_core-rescue:C_22uF-footprints COUT102
 U 1 1 5E5C89C8
 P 5350 9000
@@
 $EndComp
 $Comp
-L footprints:C_33uF COUT103
+L BMS_core-rescue:C_33uF-footprints COUT103
 U 1 1 5E5CA0AF
 P 5700 9000
@@
 	1000 8650 1075 8650
 $Comp
-L footprints:C_0.1uF C102
+L BMS_core-rescue:C_0.1uF-footprints C102
 U 1 1 5E6C94BB
 P 2650 8875
@@
 $EndComp
 $Comp
-L footprints:C_2.2uF C101
+L BMS_core-rescue:C_2.2uF-footprints C101
 U 1 1 5E6CA759
 P 2425 8875
@@
 GND
 $Comp
-L footprints:T_LAN_SM91501ALE T1
+L BMS_core-rescue:T_LAN_SM91501ALE-footprints T1
 U 1 1 5EF8F2AF
 P 10650 3100
@@
 IP
 $Comp
-L footprints:G5Q-1A4-DC12 K1
+L BMS_core-rescue:G5Q-1A4-DC12-footprints K1
 U 1 1 5E4512AF
 P 8800 8800
@@
 	0    -1   -1   0
 $EndComp
+$Comp
+L formula:R_475 R?
+U 1 1 5E4B64F1
+P 9850 6100
+F 0 "R?" V 9643 6100 50  0000 C CNN
+F 1 "R_475" V 9734 6100 50  0000 C CNN
+F 2 "footprints:R_0805_OEM" H 9780 6100 50  0001 C CNN
+F 3 "http://www.yageo.com.tw/exep/pages/download/literatures/PYu-R_INT-thick_7.pdf" H 9930 6100 50  0001 C CNN
+F 4 "DK" H 9850 6100 60  0001 C CNN "MFN"
+F 5 "311-475CRCT-ND" H 9850 6100 60  0001 C CNN "MPN"
+F 6 "https://www.digikey.com/products/en?keywords=311-475CRCT-ND" H 10330 6500 60  0001 C CNN "PurchasingLink"
+	1    9850 6100
+	0    1    1    0
+$EndComp
+$Comp
+L formula:R_10K R?
+U 1 1 5E4CC23B
+P 10350 6100
+F 0 "R?" V 10143 6100 50  0000 C CNN
+F 1 "R_10K" V 10234 6100 50  0000 C CNN
+F 2 "footprints:R_0805_OEM" H 10280 6100 50  0001 C CNN
+F 3 "http://www.bourns.com/data/global/pdfs/CRS.pdf" H 10430 6100 50  0001 C CNN
+F 4 "DK" H 10350 6100 60  0001 C CNN "MFN"
+F 5 "CRS0805-FX-1002ELFCT-ND" H 10350 6100 60  0001 C CNN "MPN"
+F 6 "https://www.digikey.com/products/en?keywords=CRS0805-FX-1002ELFCT-ND" H 10830 6500 60  0001 C CNN "PurchasingLink"
+	1    10350 6100
+	0    1    1    0
+$EndComp
 $EndSCHEMATC
