File: Boards/BMS_Peripheral/BMS_peripheral_v2.kicad_pcb (KiCad board)
At the start: 4 copper layers, 50 x 236.2 mm, 134 parts, among them J1 MM_F_VT_12, J2 MM_F_VT_10, J3 MM_F_VT_16, J4 MM_F_VT_12, J5 MM_M_VT_12, J6 MicroFit_RA_V_2_SMD, J7 MicroFit_RA_V_2_SMD, Q1 NSS1C201MZ4, Q2 NSS1C201MZ4, T1 T_LAN_7490100111A, T2 T_LAN_7490100111A, U1 LTC6811-1, U2 LTC6811-1, U3 24AA01, U4 MCP6001T-I-LT, U5 LTC1380IGN, U6 LTC1380IGN, U7 LTC1380IGN, U8 MCP6001T-I-LT

Commit message: modify Perhiperal and fix opamp volage divider on Core
Parts:
- added J1: MM_F_VT_12, footprints:micromatch_female_vt_12, B.Cu at (429.6, 262.5)
- added J2: MM_F_VT_10, footprints:micromatch_female_vert_10, B.Cu at (428.5, 237.9)
- added J3: MM_F_VT_16, footprints:micromatch_female_vert_16, B.Cu at (429.8, 203.8)
- added J4: MM_F_VT_12, footprints:micromatch_female_vt_12, B.Cu at (430.0, 179.9)
- added J5: MM_M_VT_12, footprints:micromatch_female_vt_12, B.Cu at (430.0, 155.0)
- T1, T2: value T_LAN_7490100111A -> T_LAN_SM91501ALE; footprint footprints:T_LAN_7490100111A -> footprints:T_LAN_SM91501ALE
- moved T1 6.69 mm to (207.8, 295.4), turned to 180 degrees
- moved T2 6.45 mm to (193.4, 295.4)
- moved C33 3.15 mm to (183.9, 287.6)
- moved C28 0.82 mm to (180.2, 299.6)
- moved C29 0.82 mm to (180.2, 293.2)
- moved C32 0.82 mm to (184.8, 304.9)
- moved R61 0.82 mm to (184.8, 301.3)
- moved R62 0.82 mm to (184.8, 297.8)
- moved R63 0.82 mm to (184.8, 294.2)
- moved R64 0.82 mm to (184.8, 290.7)
- moved C30 0.71 mm to (216.0, 286.4)
- moved C31 0.71 mm to (216.0, 305.2)
- moved R58 0.71 mm to (216.0, 293.7)
- moved R59 0.71 mm to (216.0, 297.5)
- moved R57 0.71 mm to (216.0, 290.2)
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Connections:
- C17 pad 2: /GND1 -> /GND2
- C18 pad 2: /GND2 -> /GND1
- C19 pad 2: /GND1 -> /GND2
- C20 pad 2: /GND1 -> /GND2
- C21 pad 2: /GND2 -> /GND1
- C22 pad 2: /GND1 -> /GND2
- C23 pad 2: /GND2 -> /GND1
- C24 pad 2: /GND1 -> /GND2
- C25 pad 2: /GND2 -> /GND1
- C26 pad 2: /GND1 -> /GND2
- C27 pad 2: /GND1 -> /GND2
- C28 pad 2: /GND2 -> /GND1
- C29 pad 2: /GND2 -> /GND1
- C30 pad 2: /GND1 -> /GND2
- C31 pad 2: /GND1 -> /GND2
- C32 pad 2: /GND2 -> /GND1
- C33 pad 2: /GND2 -> /GND1
- C34 pad 2: /GND1 -> /GND2
- C35 pad 2: /GND1 -> /GND2
- C36 pad 2: /GND1 -> /GND2
- C37 pad 2: /GND1 -> /GND2
- R35 pad 1: /V+1 -> /V+2
- R36 pad 1: /V+2 -> /V+1
- R40 pad 2: /GND1 -> /GND2
- R41 pad 2: /GND2 -> /GND1
- R43 pad 1: /V+1 -> /V+2
- R44 pad 1: /V+2 -> /V+1
- R57 pad 1: /IPA1 -> /IPA2
- R58 pad 2: /IMA1 -> /IMA2
- R59 pad 1: /IPB1 -> /IPB2
- R60 pad 2: /IMB1 -> /IMB2
- R61 pad 1: /IPA2 -> /IPA1
- R62 pad 2: /IMA2 -> /IMA1
- R63 pad 1: /IPB2 -> /IPB1
- R64 pad 2: /IMB2 -> /IMB1
- T1 pad 1: Net-(J6-Pad1) -> /IPA2
- T1 pad 10: Net-(C31-Pad1) -> Net-(J6-Pad2)
- T1 pad 11: /IPB1 -> Net-(T1-Pad11)
- T1 pad 12: (no net) -> Net-(J6-Pad1)
- T1 pad 2: Net-(T1-Pad2) -> Net-(C30-Pad1)
- T1 pad 3: Net-(J6-Pad2) -> /IMA2
- T1 pad 4: (no net) -> /IPB2
- T1 pad 5: (no net) -> Net-(C31-Pad1)
- T1 pad 6: Net-(T1-Pad6) -> /IMB2
- T1 pad 9: /IMB1 -> Net-(T1-Pad9)
- T2 pad 1: Net-(T1-Pad6) -> /IPA1
- T2 pad 10: Net-(C33-Pad1) -> Net-(T1-Pad7)
- T2 pad 11: /IPB2 -> Net-(T2-Pad11)
- T2 pad 12: (no net) -> Net-(T1-Pad9)
- T2 pad 2: Net-(T2-Pad2) -> Net-(C32-Pad1)
- T2 pad 3: Net-(T1-Pad8) -> /IMA1
- T2 pad 4: (no net) -> /IPB1
- T2 pad 5: (no net) -> Net-(C33-Pad1)
- T2 pad 6: Net-(J7-Pad1) -> /IMB1
- T2 pad 7: Net-(T2-Pad7) -> Net-(J7-Pad2)
- T2 pad 8: Net-(J7-Pad2) -> Net-(T2-Pad8)
- T2 pad 9: /IMB2 -> Net-(J7-Pad1)
- U1 pad 30: /GND1 -> /GND2
- U1 pad 31: /GND1 -> /GND2
- U1 pad 36: /GND1 -> /GND2
- U1 pad 41: /IMA1 -> /IMA2
- U1 pad 42: /IPA1 -> /IPA2
- U1 pad 47: /IMB1 -> /IMB2
- U1 pad 48: /IPB1 -> /IPB2
- U2 pad 30: /GND2 -> /GND1
- U2 pad 31: /GND2 -> /GND1
- U2 pad 36: /GND2 -> /GND1
- U2 pad 41: /IMA2 -> /IMA1
- U2 pad 42: /IPA2 -> /IPA1
- U2 pad 47: /IMB2 -> /IMB1
- U2 pad 48: /IPB2 -> /IPB1
- U3 pad 2: /GND1 -> /GND2
- U3 pad 5: /GND1 -> /GND2
- U4 pad 2: /GND1 -> /GND2
- U5 pad 10: /GND1 -> /GND2
- U5 pad 11: /GND1 -> /GND2
- U5 pad 12: /GND1 -> /GND2
- U5 pad 13: /GND1 -> /GND2
- U6 pad 10: /GND1 -> /GND2
- U6 pad 11: /GND1 -> /GND2
- U6 pad 12: /GND1 -> /GND2
- U7 pad 10: /GND1 -> /GND2
- U7 pad 11: /GND1 -> /GND2
- U7 pad 13: /GND1 -> /GND2
- U8 pad 2: /GND1 -> /GND2
Routing:
- net /V+1: track 240.9 -> 0.00 mm, vias 2 -> 0
- net /GND1: track 262.0 -> 33.3 mm, vias 18 -> 8
- net /V+2: track 180.7 -> 221.1 mm
- net Net-(J6-Pad1): track 36.8 -> 0.82 mm
- net Net-(J6-Pad2): track 33.0 -> 3.34 mm
- net Net-(J7-Pad2): track 50.8 -> 26.7 mm
- net Net-(J7-Pad1): track 53.3 -> 31.0 mm
- net /IPB2: track 91.5 -> 69.6 mm
- net /IMB2: track 98.5 -> 85.0 mm
- net /IPA2: track 86.6 -> 74.2 mm
- net /IPB1: track 71.6 -> 59.6 mm
- net /IMA2: track 92.3 -> 80.5 mm
- net /IPA1: track 77.2 -> 66.4 mm
- net Net-(T1-Pad8): track 10.3 -> 0.00 mm
- net Net-(C31-Pad1): track 9.50 -> 0.00 mm
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- added copper zone on In2.Cu, net /GND1
- removed copper zone on In1.Cu, net /GND1
- removed copper zone on In1.Cu, net /VREF2
Other:
- board size 50 x 236.2 mm -> 294 x 237.6 mm

Commit message: setup DA Board 1 for layout
Parts:
- added J8: MM_F_VT_04, footprints:micromatch_female_vert_4, B.Cu at (436.0, 371.6)
- added J8: MM_F_VT_04, footprints:micromatch_female_vert_4, B.Cu at (213.6, 373.0)
- moved J3 21.7 mm to (408.4, 201.0)
- moved J4 21.7 mm to (408.5, 177.1)
- moved J5 21.7 mm to (408.5, 152.2)
- moved J2 21.7 mm to (407.0, 235.1)
- moved J1 21.7 mm to (408.1, 259.6)
Routing:
- net /IMA1: track 63.3 -> 56.4 mm
- net /IMA2: track 80.5 -> 79.7 mm
Other:
- board size 294 x 237.6 mm -> 272.5 x 237.7 mm

Commit message: First draft of BMS Periph V2
Parts:
- removed the J1 at (408.1, 259.6)
- removed the J2 at (407.0, 235.1)
- removed the J3 at (408.4, 201.0)
- removed the J4 at (408.5, 177.1)
- removed the J5 at (408.5, 152.2)
- removed the J8 at (436.0, 371.6)
- moved C29 75.9 mm to (209.8, 363.1)
- moved Q1 75.8 mm to (186.8, 293.5), turned to 180 degrees
- moved C28 75.2 mm to (217.1, 365.1), turned to 180 degrees
- moved R64 75.0 mm to (211.8, 360.6), turned to 0 degrees
- moved R62 71.5 mm to (218.9, 360.6), turned to 0 degrees
- moved R43 70.5 mm to (188.1, 299.6), turned to 180 degrees
- moved R63 70.4 mm to (208.2, 360.6), turned to 0 degrees
- moved C24 69.1 mm to (188.1, 302.6), turned to 0 degrees
- moved C33 68.9 mm to (222.6, 344.7), turned to 0 degrees
- moved C32 67.2 mm to (222.4, 360.6), turned to 0 degrees
- moved R61 66.7 mm to (215.4, 360.6), turned to 0 degrees
- moved R35 64.6 mm to (193.5, 297.8), turned to 0 degrees
- moved C17 63.4 mm to (193.5, 299.8), turned to 180 degrees
- moved T2 59.6 mm to (212.7, 351.8), turned to 90 degrees
- moved C30 56.6 mm to (222.6, 342.6), turned to 0 degrees
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Routing:
- net /VREF2: track 73.0 -> 457.9 mm, vias 26 -> 10
- net /V+1: track 0.00 -> 205.4 mm, vias 0 -> 1
- net /V+2: track 221.1 -> 125.5 mm, vias 2 -> 1
- net /IMB2: track 85.0 -> 25.3 mm
- net /IMA2: track 79.7 -> 35.7 mm, vias 2 -> 0
- net /IPB2: track 69.6 -> 30.7 mm
- net /IPA1: track 66.4 -> 32.9 mm
- net Net-(R1-Pad1): track 167.8 -> 134.5 mm
- net /C7_T3: track 179.3 -> 146.4 mm
- net /C15_T2: track 204.9 -> 172.2 mm
- net /C9_T2: track 78.1 -> 45.4 mm
- net Net-(C3-Pad2): track 115.1 -> 82.4 mm
- net Net-(C5-Pad2): track 106.8 -> 74.2 mm
- net Net-(C1-Pad2): track 128.4 -> 95.8 mm
- net Net-(C2-Pad2): track 225.6 -> 193.1 mm
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- removed copper zone on F.Cu, net /VREF2
Other:
- board size 272.5 x 237.7 mm -> 50 x 236.2 mm

Commit message: almost final rev periph v2
Parts:
- added TP1: Test_Point_SMD, footprints:Test_Point_SMD, F.Cu at (198.6, 351.9)
- added TP10: Test_Point_SMD, footprints:Test_Point_SMD, F.Cu at (198.7, 319.1)
- added TP11: Test_Point_SMD, footprints:Test_Point_SMD, F.Cu at (198.6, 347.8)
- added TP12: Test_Point_SMD, footprints:Test_Point_SMD, F.Cu at (198.6, 340.9)
- added TP13: Test_Point_SMD, footprints:Test_Point_SMD, F.Cu at (198.6, 332.9)
- added TP14: Test_Point_SMD, footprints:Test_Point_SMD, F.Cu at (198.6, 327.2)
- added TP2: Test_Point_SMD, footprints:Test_Point_SMD, F.Cu at (192.6, 287.1)
- added TP3: Test_Point_SMD, footprints:Test_Point_SMD, F.Cu at (193.7, 292.0)
- added TP4: Test_Point_SMD, footprints:Test_Point_SMD, F.Cu at (198.6, 355.7)
- added TP5: Test_Point_SMD, footprints:Test_Point_SMD, F.Cu at (221.8, 324.5)
- added TP6: Test_Point_SMD, footprints:Test_Point_SMD, F.Cu at (198.6, 359.3)
- added TP7: Test_Point_SMD, footprints:Test_Point_SMD, F.Cu at (206.2, 365.3)
- added TP8: Test_Point_SMD, footprints:Test_Point_SMD, F.Cu at (212.1, 321.3)
- added TP9: Test_Point_SMD, footprints:Test_Point_SMD, F.Cu at (198.7, 322.5)
- moved C29 0.44 mm to (209.8, 363.6)
- moved C27 0.14 mm to (206.1, 323.1)
- moved C31 0.13 mm to (208.7, 320.5)
Routing:
- net /IMB2: track 25.3 -> 37.0 mm, vias 0 -> 2
- net /IPB2: track 30.7 -> 36.3 mm
- net Net-(C23-Pad1): track 19.8 -> 24.9 mm
- net /IMA2: track 35.7 -> 40.1 mm
- net /IMB1: track 41.8 -> 45.1 mm
- net /GND2: track 50.4 -> 53.5 mm, vias 17 -> 18
- net /GND1: track 33.1 -> 35.9 mm, vias 8 -> 9
- net /IPB1: track 29.7 -> 32.4 mm
- net Net-(C8-Pad2): track 159.7 -> 161.0 mm
- net Net-(J6-Pad2): track 32.4 -> 33.7 mm
- net Net-(J7-Pad2): track 27.1 -> 28.4 mm
- net Net-(J7-Pad1): track 27.5 -> 28.8 mm
- net /IPA2: track 45.4 -> 46.6 mm
- net Net-(J6-Pad1): track 32.6 -> 33.6 mm
- net /C15_T2: track 172.2 -> 173.0 mm
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Other:
- board text added: "GND1"
- board text added: "GND2"
- board text added: "IMA2"
- board text added: "IMB1"
- board text added: "IPA2"
- board text added: "IPB1"
- board text added: "VREG"
