File: Boards/Suspension_Strain/Suspension_Strain.sch (KiCad schematic (older format))
At the start: 37 parts, among them J1 CONN_02X03, J101 MM_F_RA_20, J102 MM_F_RA_08, U1 MCP2561-E_SN, U101 TPS560430YF, U102 74HC4051, U2 ATMEGA16M1, Y1 Crystal_SMD

Commit message: Rename rename Chassis_Strain to Suspension_Strain
Parts:
- C1, C101, C103, C2: symbol Chassis_Strain-rescue:C_0.1uF-formula -> Suspension_Strain-rescue:C_0.1uF-formula-Suspension_Strain-rescue
- C102: symbol Chassis_Strain-rescue:C_2.2uF-formula -> Suspension_Strain-rescue:C_2.2uF-formula-Suspension_Strain-rescue
- C3: symbol Chassis_Strain-rescue:C_100pF-formula -> Suspension_Strain-rescue:C_100pF-formula-Suspension_Strain-rescue
- C4, C5: symbol Chassis_Strain-rescue:C_30pF-formula -> Suspension_Strain-rescue:C_30pF-formula-Suspension_Strain-rescue
- COUT101: symbol Chassis_Strain-rescue:C_22uF-formula -> Suspension_Strain-rescue:C_22uF-formula-Suspension_Strain-rescue
- COUT102: symbol Chassis_Strain-rescue:C_33uF-formula -> Suspension_Strain-rescue:C_33uF-formula-Suspension_Strain-rescue
- COUT103: symbol Chassis_Strain-rescue:C_47uF-formula -> Suspension_Strain-rescue:C_47uF-formula-Suspension_Strain-rescue
- D101: symbol Chassis_Strain-rescue:D_Zener_18V-formula -> Suspension_Strain-rescue:D_Zener_18V-formula-Suspension_Strain-rescue
- D102, D103: symbol Chassis_Strain-rescue:LED_0805-formula -> Suspension_Strain-rescue:LED_0805-formula-Suspension_Strain-rescue
- F101: symbol Chassis_Strain-rescue:F_500mA_16V-formula -> Suspension_Strain-rescue:F_500mA_16V-formula-Suspension_Strain-rescue
- J1: symbol Chassis_Strain-rescue:CONN_02X03-formula -> Suspension_Strain-rescue:CONN_02X03-formula-Suspension_Strain-rescue
- L101: symbol Chassis_Strain-rescue:L_100uH-formula -> Suspension_Strain-rescue:L_100uH-formula-Suspension_Strain-rescue
- R1: symbol Chassis_Strain-rescue:R_100-formula -> Suspension_Strain-rescue:R_100-formula-Suspension_Strain-rescue
- R102: symbol Chassis_Strain-rescue:R_25K-formula -> Suspension_Strain-rescue:R_25K-formula-Suspension_Strain-rescue
- R103: symbol Chassis_Strain-rescue:R_100K-formula -> Suspension_Strain-rescue:R_100K-formula-Suspension_Strain-rescue
- R104: symbol Chassis_Strain-rescue:R_0_2512-formula -> Suspension_Strain-rescue:R_0_2512-formula-Suspension_Strain-rescue
- R105: symbol Chassis_Strain-rescue:R_200-formula -> Suspension_Strain-rescue:R_200-formula-Suspension_Strain-rescue
- R3: symbol Chassis_Strain-rescue:R_10K-formula -> Suspension_Strain-rescue:R_10K-formula-Suspension_Strain-rescue
- U1: symbol Chassis_Strain-rescue:MCP2561-E_SN-formula -> Suspension_Strain-rescue:MCP2561-E_SN-formula-Suspension_Strain-rescue
- U101: symbol Chassis_Strain-rescue:TPS560430YF-formula -> Suspension_Strain-rescue:TPS560430YF-formula-Suspension_Strain-rescue
- U2: symbol Chassis_Strain-rescue:ATMEGA16M1-formula -> Suspension_Strain-rescue:ATMEGA16M1-formula-Suspension_Strain-rescue
- Y1: symbol Chassis_Strain-rescue:Crystal_SMD-formula -> Suspension_Strain-rescue:Crystal_SMD-formula-Suspension_Strain-rescue
Changed lines of the file:
@@
 $EndComp
 $Comp
-L Chassis_Strain-rescue:C_2.2uF-formula C102
+L Suspension_Strain-rescue:C_2.2uF-formula-Suspension_Strain-rescue C102
 U 1 1 5BEE2647
 P 2250 6250
@@
 $EndComp
 $Comp
-L Chassis_Strain-rescue:C_0.1uF-formula C101
+L Suspension_Strain-rescue:C_0.1uF-formula-Suspension_Strain-rescue C101
 U 1 1 5BEE2923
 P 1950 6250
@@
 $EndComp
 $Comp
-L Chassis_Strain-rescue:R_100K-formula R103
+L Suspension_Strain-rescue:R_100K-formula-Suspension_Strain-rescue R103
 U 1 1 5BEE2A52
 P 3850 6900
@@
 $EndComp
 $Comp
-L Chassis_Strain-rescue:C_0.1uF-formula C103
+L Suspension_Strain-rescue:C_0.1uF-formula-Suspension_Strain-rescue C103
 U 1 1 5BEE239B
 P 3850 6050
@@
 12V
 $Comp
-L Chassis_Strain-rescue:C_22uF-formula COUT101
+L Suspension_Strain-rescue:C_22uF-formula-Suspension_Strain-rescue COUT101
 U 1 1 5C061BB4
 P 4650 6350
@@
 $EndComp
 $Comp
-L Chassis_Strain-rescue:C_47uF-formula COUT103
+L Suspension_Strain-rescue:C_47uF-formula-Suspension_Strain-rescue COUT103
 U 1 1 5C062E7A
 P 5450 6350
@@
 $EndComp
 $Comp
-L Chassis_Strain-rescue:C_33uF-formula COUT102
+L Suspension_Strain-rescue:C_33uF-formula-Suspension_Strain-rescue COUT102
 U 1 1 5C08921B
 P 5050 6350
@@
 $EndComp
 $Comp
-L Chassis_Strain-rescue:R_25K-formula R102
+L Suspension_Strain-rescue:R_25K-formula-Suspension_Strain-rescue R102
 U 1 1 5C0B315C
 P 3350 6900
@@
 $EndComp
 $Comp
-L Chassis_Strain-rescue:F_500mA_16V-formula F101
+L Suspension_Strain-rescue:F_500mA_16V-formula-Suspension_Strain-rescue F101
 U 1 1 5C0BFA29
 P 1150 6100
@@
 $EndComp
 $Comp
-L Chassis_Strain-rescue:R_0_2512-formula R104
+L Suspension_Strain-rescue:R_0_2512-formula-Suspension_Strain-rescue R104
 U 1 1 5C0C29A9
 P 6000 6200
@@
 $EndComp
 $Comp
-L Chassis_Strain-rescue:LED_0805-formula D103
+L Suspension_Strain-rescue:LED_0805-formula-Suspension_Strain-rescue D103
 U 1 1 5C0C344A
 P 6400 7050
@@
 $EndComp
 $Comp
-L Chassis_Strain-rescue:R_200-formula R105
+L Suspension_Strain-rescue:R_200-formula-Suspension_Strain-rescue R105
 U 1 1 5C0C44F9
 P 6400 6450
@@
 $EndComp
 $Comp
-L Chassis_Strain-rescue:D_Zener_18V-formula D101
+L Suspension_Strain-rescue:D_Zener_18V-formula-Suspension_Strain-rescue D101
 U 1 1 5C623D49
 P 800 6400
@@
 12V
 $Comp
-L Chassis_Strain-rescue:LED_0805-formula D102
+L Suspension_Strain-rescue:LED_0805-formula-Suspension_Strain-rescue D102
 U 1 1 5C754D7D
 P 1550 6650
@@
 Bootstrap Capacitor\n
 $Comp
-L Chassis_Strain-rescue:L_100uH-formula L101
+L Suspension_Strain-rescue:L_100uH-formula-Suspension_Strain-rescue L101
 U 1 1 5BEE27A2
 P 4250 6200
@@
 RESET
 $Comp
-L Chassis_Strain-rescue:R_100-formula R1
+L Suspension_Strain-rescue:R_100-formula-Suspension_Strain-rescue R1
 U 1 1 5D58E16F
 P 1150 1150
@@
 $EndComp
 $Comp
-L Chassis_Strain-rescue:C_100pF-formula C3
+L Suspension_Strain-rescue:C_100pF-formula-Suspension_Strain-rescue C3
 U 1 1 5D58E505
 P 1150 1450
@@
 $EndComp
 $Comp
-L Chassis_Strain-rescue:Crystal_SMD-formula Y1
+L Suspension_Strain-rescue:Crystal_SMD-formula-Suspension_Strain-rescue Y1
 U 1 1 5D5EB332
 P 4550 4100
@@
 $EndComp
 $Comp
-L Chassis_Strain-rescue:C_30pF-formula C4
+L Suspension_Strain-rescue:C_30pF-formula-Suspension_Strain-rescue C4
 U 1 1 5D5EB5B2
 P 4350 4350
@@
 $EndComp
 $Comp
-L Chassis_Strain-rescue:C_30pF-formula C5
+L Suspension_Strain-rescue:C_30pF-formula-Suspension_Strain-rescue C5
 U 1 1 5D5EB694
 P 4750 4350
@@
 $EndComp
 $Comp
-L Chassis_Strain-rescue:R_10K-formula R3
+L Suspension_Strain-rescue:R_10K-formula-Suspension_Strain-rescue R3
 U 1 1 5D5EB7F3
 P 4600 3500
@@
 $EndComp
 $Comp
-L Chassis_Strain-rescue:MCP2561-E_SN-formula U1
+L Suspension_Strain-rescue:MCP2561-E_SN-formula-Suspension_Strain-rescue U1
 U 1 1 5D5FAEDE
 P 9900 1750
@@
 $EndComp
 $Comp
-L Chassis_Strain-rescue:C_0.1uF-formula C1
+L Suspension_Strain-rescue:C_0.1uF-formula-Suspension_Strain-rescue C1
 U 1 1 5D5FB603
 P 9750 1150
@@
 GND
 $Comp
-L Chassis_Strain-rescue:CONN_02X03-formula J1
+L Suspension_Strain-rescue:CONN_02X03-formula-Suspension_Strain-rescue J1
 U 1 1 5D628C9D
 P 9950 3450
@@
 Connection ~ 1150 1300
 $Comp
-L Chassis_Strain-rescue:C_0.1uF-formula C2
+L Suspension_Strain-rescue:C_0.1uF-formula-Suspension_Strain-rescue C2
 U 1 1 5D58E34B
 P 800 1150
@@
 	10900 6000 10900 6150
 $Comp
-L Chassis_Strain-rescue:TPS560430YF-formula U101
+L Suspension_Strain-rescue:TPS560430YF-formula-Suspension_Strain-rescue U101
 U 1 1 5C75D405
 P 2950 6250
@@
 CAN_TX
 $Comp
-L Chassis_Strain-rescue:ATMEGA16M1-formula U2
+L Suspension_Strain-rescue:ATMEGA16M1-formula-Suspension_Strain-rescue U2
 U 1 1 5D58A7A6
 P 2550 2700
