File: Boards/TSAL_AIL/TSAL_AIL/TSAL-AIL.kicad_pcb (KiCad board)
At the start: 2 copper layers, 83.4 x 40.6 mm, 29 parts, among them J1 Ultrafit_4_RA, J2 NanoFit_2, J3 MM_F_RA_06, Q1 SSM3K333R, Q2 SSM3K333R, U1 MCP6001, U2 LR8K4-G, U3 CPC1025NTR, U4 BU4S11G2-TR

Commit message: minor TSAL updates
Parts:
- F1: footprint Formula:F_21mA_420V -> footprints:F_21mA_420V
- J1: footprint Formula:Ultrafit_4_RA -> footprints:Ultrafit_4_RA
- J3: moved to B.Cu
- U3: footprint Formula:4-pin_SOP -> Package_DIP:DIP-5-6_W7.62mm
- moved C4 22.4 mm to (205.1, 91.9), turned to 0 degrees
- moved R13 21.3 mm to (206.0, 98.5), turned to 180 degrees
- moved R14 21.2 mm to (206.0, 109.4), turned to 0 degrees
- moved C3 20.7 mm to (165.5, 95.8), turned to 270 degrees
- moved U4 20.6 mm to (206.0, 95.3), turned to 90 degrees
- moved R1 16.5 mm to (153.2, 109.1), turned to 270 degrees
- moved R5 15.9 mm to (161.1, 97.1), turned to 270 degrees
- moved Q1 15.5 mm to (206.0, 101.8), turned to 270 degrees
- moved Q2 15.1 mm to (206.0, 105.8), turned to 90 degrees
- moved R3 12.1 mm to (163.3, 97.1)
- moved R4 11.1 mm to (153.2, 105.3), turned to 270 degrees
- moved J1 9.24 mm to (145.1, 90.8)
- moved R2 9.04 mm to (155.2, 90.1)
- moved J3 8.21 mm to (199.6, 103.5)
- moved R11 7.87 mm to (161.2, 101.0), turned to 0 degrees
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Routing:
- net /AIL-: track 154.9 -> 67.8 mm
- net /TSAL_FLAG: track 19.4 -> 57.7 mm
- net GND: track 3.13 -> 31.1 mm
- net /TSAL_GREEN-: track 28.5 -> 3.87 mm
- net /TSAL_RED-: track 20.1 -> 4.11 mm
- net /GLV+: track 51.6 -> 64.7 mm
- net /TS+: track 26.1 -> 38.1 mm
- net /5V: track 47.4 -> 36.2 mm
- net /AIL+: track 12.4 -> 19.0 mm
- net Net-(D1-Pad2): track 17.5 -> 13.8 mm, vias 2 -> 0
- net Net-(R10-Pad2): track 9.87 -> 6.75 mm
- net Net-(F1-Pad1): track 3.93 -> 5.74 mm
- net Net-(R12-Pad1): track 10.8 -> 12.6 mm
- net Net-(R5-Pad1): track 11.2 -> 9.44 mm
- net /NAND_Out: track 3.91 -> 2.53 mm
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- removed copper zone on F.Cu, net /5V
- removed copper zone on B.Cu, net GND
- removed copper zone on F.Cu, net GND

Commit message: TSAL First Pass
Parts:
- removed F1: F_21mA_420V, footprints:F_21mA_420V
- added C5: C_2.2uF, footprints:C_0805_OEM, B.Cu at (167.3, 80.8)
- added C6: C_470pF, footprints:C_0805_OEM, B.Cu at (167.3, 82.7)
- added C7: C_.22uF, footprints:C_0805_OEM, B.Cu at (170.3, 79.8)
- added C8: C_100uF+, footprints:C_100uF+, F.Cu at (177.2, 100.9)
- added C9: C_1uF, footprints:C_0805_OEM, F.Cu at (183.7, 104.8)
- added L1: L_1.2mH, footprints:L_1.2mH, F.Cu at (172.2, 91.5)
- added R15: R_6.2K, footprints:R_0805_OEM, B.Cu at (167.3, 84.5)
- added R16: R_3K, footprints:R_0805_OEM, F.Cu at (189.8, 104.8)
- added U5: Diode_600V_1A_SM, footprints:Diode_600V_1A_SM, B.Cu at (168.2, 76.7)
- added U6: Diode_600V_1A_SM, footprints:Diode_600V_1A_SM, F.Cu at (169.9, 110.3)
- added U7: Diode_600V_1A_SM, footprints:Diode_600V_1A_SM, F.Cu at (177.2, 82.6)
- C1, C2: footprint Formula:C_0805_OEM -> footprints:C_0805_OEM
- C3: value C_1uF -> C_10uF_450V; footprint Formula:C_0805_OEM -> footprints:C_10uF_450V
- D1: footprint Formula:LED_0805_OEM -> footprints:LED_0805_OEM
- R1, R11, R12, R2, R3, R4, R5, R6, R7, R9: footprint Formula:R_0805_OEM -> footprints:R_0805_OEM
- R10: value R_1K -> R_6.04K; footprint Formula:R_0805_OEM -> footprints:R_0805_OEM; moved to B.Cu
- R8: value R_3K -> R_10K; footprint Formula:R_0805_OEM -> footprints:R_0805_OEM; moved to B.Cu
- U2: value LR8K4-G -> Buck_Converter_450V_300mA; footprint Package_TO_SOT_SMD:TO-252-2 -> footprints:Converter_DCDC_MPS_MP9488; moved to B.Cu
- moved R1 51.5 mm to (193.1, 76.4), turned to 0 degrees
- moved R4 46.5 mm to (189.6, 76.4), turned to 0 degrees
- moved R6 41.4 mm to (186.2, 76.4), turned to 0 degrees
- moved C2 38.7 mm to (187.6, 104.8), turned to 90 degrees
- moved C1 37.8 mm to (185.6, 104.8), turned to 90 degrees
- moved R9 37.1 mm to (183.8, 81.3)
- moved D1 37.1 mm to (184.9, 78.6), turned to 180 degrees
- moved R7 36.5 mm to (182.8, 76.4), turned to 0 degrees
- moved R11 31.5 mm to (185.8, 81.3), turned to 270 degrees
- moved R12 29.9 mm to (181.7, 81.3), turned to 90 degrees
- moved R5 27.8 mm to (179.6, 76.4), turned to 180 degrees
- moved U1 27.0 mm to (178.3, 79.4), turned to 180 degrees
- moved R3 24.4 mm to (176.2, 76.4), turned to 0 degrees
- moved R2 22.7 mm to (175.3, 79.4), turned to 270 degrees
- moved U3 16.9 mm to (183.5, 87.5), turned to 0 degrees
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Connections:
- C1 pad 1: /AIL- -> GND
- C1 pad 2: /5V -> /15V+
- C2 pad 1: /AIL- -> GND
- C2 pad 2: /5V -> /15V+
- C3 pad 1: /5V -> GND
- C3 pad 2: /AIL- -> /TS+
- J1 pad 2: /AIL- -> GND
- J1 pad 4: /AIL- -> GND
- J2 pad 2: /AIL- -> GND
- R10 pad 1: /5V -> Net-(C7-Pad1)
- R10 pad 2: Net-(R10-Pad2) -> /FB
- R11 pad 2: /AIL- -> GND
- R2 pad 2: /5V -> /15V+
- R3 pad 2: /AIL- -> GND
- R5 pad 2: /AIL- -> GND
- R8 pad 1: /AIL- -> Net-(R8-Pad1)
- R8 pad 2: Net-(R10-Pad2) -> /VCC
- U1 pad 2: /AIL- -> GND
- U1 pad 5: /5V -> /15V+
- U2 pad 1: Net-(F1-Pad1) -> /VCC
- U2 pad 2: /5V -> /FB
- U2 pad 3: Net-(R10-Pad2) -> /SW
- U3 pad 2: /AIL- -> GND
Routing:
- net GND: track 31.1 -> 159.0 mm
- net /AIL-: track 67.8 -> 0.00 mm, vias 3 -> 0
- net /TS+: track 38.1 -> 79.0 mm, vias 0 -> 2
- net /AIL+: track 19.0 -> 58.7 mm, vias 0 -> 1
- net /15V+: track 0.00 -> 37.1 mm
- net /5V: track 36.2 -> 0.00 mm
- net /GLV+: track 64.7 -> 38.8 mm
- net /TSAL_FLAG: track 57.7 -> 37.8 mm
- net /SW: track 0.00 -> 17.0 mm
- net /FB: track 0.00 -> 9.80 mm
- net Net-(C7-Pad1): track 0.00 -> 9.64 mm, vias 0 -> 1
- net Net-(R2-Pad1): track 12.3 -> 3.90 mm
- net /VCC: track 0.00 -> 7.94 mm
- net Net-(D1-Pad2): track 13.8 -> 6.21 mm
- net Net-(R10-Pad2): track 6.75 -> 0.00 mm
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- added copper zone on B.Cu, net /SW
- added copper zone on B.Cu, net /TS+

Commit message: Final SS Boards Rev 2
Parts:
- C1, C8, C9, R16: moved to B.Cu
- D3: renamed from U6; moved to B.Cu
- R2: value R_1K -> R_1.91K
- R3: value R_137 -> R_51.1K
- U3: footprint Package_DIP:DIP-5-6_W7.62mm -> footprints:DIP-5-6_W7.62mm
- moved C2 55.3 mm to (137.2, 82.0), turned to 180 degrees
- moved R1 40.6 mm to (152.5, 78.7)
- moved R2 37.2 mm to (138.1, 79.5)
- moved R3 37.2 mm to (139.1, 76.6)
- moved R11 37.1 mm to (148.7, 81.5)
- moved R4 37.1 mm to (152.5, 76.6)
- moved R5 37.1 mm to (142.5, 76.6)
- moved R6 37.1 mm to (149.1, 76.6)
- moved R7 37.1 mm to (145.7, 76.6)
- moved R9 37.1 mm to (146.7, 81.5)
- moved U1 37.1 mm to (141.2, 79.6)
- moved D1 37.1 mm to (147.8, 78.8)
- moved R12 37.1 mm to (144.6, 81.5)
- moved R16 26.6 mm to (163.9, 111.0), turned to 0 degrees
- moved D3 25.6 mm to (161.8, 86.1), turned to 180 degrees
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- renumbered U5 to D2, U7 to D4
Connections:
- R10 pad 2: /FB -> Net-(R10-Pad2)
- R15 pad 1: /FB -> Net-(R10-Pad2)
- U4 pad 4: Net-(U4-Pad4) -> /NAND_Out
Routing:
- net /15V+: track 37.1 -> 84.7 mm, vias 0 -> 3
- net GND: track 159.0 -> 202.6 mm
- net Net-(R12-Pad1): track 6.03 -> 48.6 mm, vias 0 -> 1
- net /AIL+: track 58.7 -> 26.9 mm, vias 1 -> 0
- net /TS+: track 79.0 -> 55.2 mm, vias 2 -> 0
- net /SW: track 17.0 -> 1.32 mm
- net /NAND_Out: track 2.53 -> 16.4 mm, vias 0 -> 2
- net /TSAL_FLAG: track 37.8 -> 46.0 mm
- net Net-(R10-Pad2): track 0.00 -> 7.09 mm
- net /GLV+: track 38.8 -> 44.2 mm
- net /FB: track 9.80 -> 4.76 mm
- net Net-(C7-Pad1): track 9.64 -> 11.7 mm
- net Net-(R1-Pad1): track 1.54 -> 2.89 mm
