File: Boards/BSPD_Brakelight/BSPD_Brakelight.sch (KiCad schematic (older format))
At the start: 89 parts, among them IC1 ATMEGA16M1, J2 MM_F_RA_20, J3 CONN_02X03, Q1 SSM3K333R, Q2 SSM3K333R, Q3 SSM3K333R, Q6 SSM3K333R, U1 SN74LVC1G08, U101 TPS560430YF, U2 MCP6001, U3 CAN_Transceiver, U4 MCP6001, U5 SN74LVC1G02, U6 SN74LVC1G02, U7 MCP6001, U8 SN74LVC1G32, Y1 Crystal_SMD

Commit message: Updated BSPD/Brakelight with Adi's changes
Also deleted old files from rev 1 and renamed files to keep with naming
convention
Parts:
- added C15, C16, C17: C_0.1uF, footprints:C_0805_OEM, symbol formula:C_0.1uF
- C10, C11, C7: symbol Brakelight_Shutdown_BSPD-rescue:C_1uF-formula -> formula:C_1uF
- C102: symbol Brakelight_Shutdown_BSPD-rescue:C_2.2uF-formula -> formula:C_2.2uF
- C5: symbol Brakelight_Shutdown_BSPD-rescue:C_10uF-formula -> formula:C_10uF
Connections:
- net GND: now also C15.2, C16.2, C17.2
- net VCC: now also C15.1, C16.1, C17.1
Other:
- note added: "BSPD circuit is tripped when the motor controller is still providing power \nto the motor while the brake is being pressed. This means the brake \nis not behaving correctly and this is a very dangerous situation, so the\nBSPD relay is tripped and the shutdown circuit is opened (car shuts \ndown).\n\nThere is a BSPD test switch included for testing to make sure the\ncircuit works, and also because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"
- note added: "Break Pressure Sensor\nhttps://www.digikey.com/product-detail/en/honeywell-sensing-and\n-productivity-solutions/MLH02KPSB06A/480-2534-ND/1248869\n\nVoltage range of .5-4.5V\nThis circuit uses the following ranges with corresponding behaivors:\n\n0-.45V (open circuit): Since the voltage is too low, we treat this as \nan open circuit, so we keep the brakelight on.\n\n.45-.92V: Brake isn't being pre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"
- note added: "Timer Calculations"
- note added: "VCC = 5V"
- note added: "V_cap = .5V because that is the \nvalue we compare to using the\nop amp (U2)."
- note added: "V_cap = V_source * (1 - e ^ (-t / RC))\nt = -RC * ln(1 - (V_cap / V_source))\nt = -(71500 * .00001 * ln(2.5 / 5))\n = .5 s"
- note added: "V_out = VCC * R16 / (R15 + R16)\n5 * 1000 / (10000 + 1000) = .45"
- note added: "V_out = VCC * R19 / (R19 + R12)\n5 * 499 / (499 + 2200) = .92"
