File: Boards/lv_bms/bms.kicad_pcb (KiCad board)
At the start: 4 copper layers, 109.3 x 58.3 mm, 99 parts, among them J1 CONN_02X03, J2 Screw_Terminal_01x05, J3 NanoFit_RA_TH_04, SW1 SW_Push_SPST_NO, U1 MCP2561-E_SN, U101 TPS560430YF, U14 LR8K4-G, U2 ATMEGA16M1, U3 BQ79606A-Q1, Y1 Crystal_SMD

Commit message: changes to lv bms
Parts:
- removed TP1, TP2, TP3, TP4, TP5, TP6, TP7, TP8: Test_Point_SMD, footprints:Test_Point_SMD
- added C30: C_1uF, formula:C_0805_OEM, F.Cu at (145.6, 131.8)
- added C31: C_1uF, formula:C_0805_OEM, F.Cu at (144.8, 128.2)
- added J4: NanoFit_RA_TH_06, formula:NanoFit_RA_TH_6, F.Cu at (104.4, 117.8)
- added J5: NanoFit_RA_TH_06, formula:NanoFit_RA_TH_6, F.Cu at (157.2, 79.2)
- added J6: NanoFit_RA_TH_06, formula:NanoFit_RA_TH_6, F.Cu at (158.2, 126.8)
- added Q1: MMBF170, formula:SOT-23-3_OEM, F.Cu at (198.4, 100.3)
- added R34: R_1K_0.1, formula:C_0805_OEM, F.Cu at (150.2, 131.8)
- added R35: R_1K, formula:C_0805_OEM, F.Cu at (147.6, 128.2)
- added R36: R_1K_0.1, formula:C_0805_OEM, F.Cu at (154.7, 131.8)
- added R37: R_1K, formula:C_0805_OEM, F.Cu at (150.5, 128.2)
- C1, C10, C101, C11, C12, C13, C14, C16, C2, C20, C21, C22, C23, C24, C25, C27, C28, C3, C4, C5, C6, C7, C8, C9: footprint footprints:C_0805_OEM -> formula:C_0805_OEM
- J2: value Screw_Terminal_01x05 -> NanoFit_RA_TH_06; footprint TerminalBlock_TE-Connectivity:TerminalBlock_TE_282834-5_1x05_P2.54mm_Horizontal -> formula:NanoFit_RA_TH_6
- J3: footprint footprints:NanoFit_RA_4 -> TerminalBlock_TE-Connectivity:TerminalBlock_TE_282834-5_1x05_P2.54mm_Horizontal
- L101: footprint footprints:L_100uH_OEM -> formula:L_100uH_OEM
- R10, R101, R102, R103, R11, R12, R13, R14, R15, R16, R17, R18, R19, R20, R21, R22, R23, R24, R25, R26, R27, R28, R29, R30, R31, R32, R33, R8, R9: footprint footprints:R_0805_OEM -> formula:C_0805_OEM
- moved J2 88.1 mm to (193.5, 105.0), turned to 0 degrees
- moved J3 81.3 mm to (201.3, 117.7), turned to 270 degrees
- moved J1 30.1 mm to (120.2, 90.7)
- moved C12 2.95 mm to (121.3, 107.3)
- moved C13 2.95 mm to (121.3, 121.3)
- moved C6 2.95 mm to (121.3, 111.2)
- moved C8 2.95 mm to (121.3, 103.8)
- moved C9 2.95 mm to (121.3, 117.8)
- moved R25 2.95 mm to (117.1, 124.9)
- moved C10 2.95 mm to (121.3, 114.2)
- moved C11 2.95 mm to (121.1, 124.9)
- moved C14 2.95 mm to (121.1, 128.2)
- moved C20 2.95 mm to (127.9, 130.5)
- moved C7 2.95 mm to (121.1, 132.2)
- moved R22 2.95 mm to (117.2, 103.8)
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Connections:
- C17 pad 2: VCC -> /TSREF
- J2 pad 1: /BattConn0 -> VCC
- J2 pad 2: /BattConn1 -> VCC
- J2 pad 3: /BattConn2 -> /CURRENT_SENSE_IN
- J2 pad 4: /BattConn3 -> /RELAY_GND
- J2 pad 5: /BattConn4 -> Net-(J2-Pad5)
- U2 pad 17: Net-(U2-Pad17) -> /CURRENT_SENSE_IN
- U2 pad 30: Net-(U2-Pad30) -> /RELAY
- U3 pad 43: VCC -> /TSREF
Routing:
- net VCC: track 172.7 -> 125.6 mm
- net /BattConn1: track 12.9 -> 0.00 mm
- net /BattConn3: track 10.9 -> 23.9 mm
- net /-Therm2SMD: track 15.2 -> 7.64 mm
- net /-Therm4SMD: track 14.9 -> 7.39 mm
- net /-Therm3SMD: track 15.0 -> 7.69 mm
- net /CAN_HI: track 18.3 -> 23.4 mm
- net /CAN_LO: track 8.99 -> 3.92 mm
- net /VC0: track 35.7 -> 36.7 mm, vias 2 -> 3
- net GNDA: track 91.2 -> 90.2 mm, vias 18 -> 17
Other:
- board size 109.3 x 58.3 mm -> 119.4 x 58.3 mm
- board text added: "BATT_SENSE"
- board text added: "CAN"
- board text added: "RELAY CURRENT_SENSE"
- board text added: "THERM"
