File: repackaged/service_section_controller/air_control_carryover.sch (KiCad schematic (older format))
At the start: 0 parts

Commit message: added ss carryover boards
Parts:
- added C1, C2: CP_1mF, footprints:C_Radial_D10_L13_P5_OEM, symbol formula:CP_1mF
- added C101, C103, C4, C7: C_0.1uF, footprints:C_0805_OEM, symbol formula:C_0.1uF
- added C102: C_2.2uF, footprints:C_0603_1608Metric, symbol AIR_control-rescue:C_2.2uF-formula
- added C11, C13: C_30pF, footprints:C_0805_OEM, symbol formula:C_30pF
- added C6: C_100pF, footprints:C_0805_OEM, symbol formula:C_100pF
- added COUT101: C_22uF, footprints:C_1206_OEM, symbol formula:C_22uF
- added COUT102: C_33uF, footprints:C_1812_OEM, symbol formula:C_33uF
- added COUT103: C_47uF, footprints:C_0805_OEM, symbol formula:C_47uF
- added D1, D10, D102, D103, D12, D13, D15, D16, D2, D3, D4, D5, D6, D7, D8, D9: LED_0805, footprints:LED_0805_OEM, symbol formula:LED_0805
- added D101: D_Zener_18V, footprints:DO-214AA, symbol formula:D_Zener_18V
- added F101: F_500mA_16V, footprints:Fuse_1210, symbol formula:F_500mA_16V
- added J1: MicroFit_VT_12, footprints:MicroFit_VT_12, symbol formula:MicroFit_VT_12
- added J2: MicroFit_V_2, footprints:MicroFit_V_2, symbol formula:MicroFit_V_2
- added J3: CONN_02X03, footprints:Pin_Header_Straight_2x03, symbol formula:CONN_02X03
- added J4: MM_F_VT_20, footprints:micromatch_female_vert_20, symbol formula:MM_F_VT_20
- added L101: L_100uH, footprints:L_100uH, symbol formula:L_100uH
- added Q1, Q2, Q3, Q4, Q5, Q6, Q7, Q8: SSM3K333R, footprints:SOT-23F, symbol formula:SSM3K333R
- added R1, R105, R2, R28, R29, R3, R36, R5, R7, R9: R_200, footprints:R_0805_OEM, symbol formula:R_200
- added R10, R15, R16, R22, R23, R27, R30, R35, R4, R6, R8: R_10K, footprints:R_0805_OEM, symbol formula:R_10K
- added R101, R11, R12, R17, R18, R19, R24, R33: R_1K, footprints:R_0805_OEM, symbol formula:R_1K
- added R102: R_25K, footprints:R_0805_OEM, symbol formula:R_25K
- added R103, R13, R14, R20, R21, R25, R26, R34: R_100K, footprints:R_0805_OEM, symbol formula:R_100K
- added R104: R_0_2512, footprints:R_2512_OEM, symbol formula:R_0_2512
- added R_DNP1: R_120_DNP, footprints:R_0805_OEM, symbol formula:R_120_DNP
- added U1: MCP2561-E_SN, footprints:SOIC-8_3.9x4.9mm_Pitch1.27mm_OEM, symbol formula:MCP2561-E_SN
- added U101: TPS560430YF, Package_TO_SOT_SMD:SOT-23-6_Handsoldering, symbol formula:TPS560430YF
- added U3: ATMEGA16M1, footprints:TQFP-32_7x7mm_Pitch0.8mm, symbol formula:ATMEGA16M1
- added Y1: Crystal_SMD, footprints:Crystal_SMD_FA238, symbol formula:Crystal_SMD
Connections:
- net labels added: +12V, AIR+Weld_Detect, AIR-LSD, AIR-Weld_Detect, Air+Aux+, Air+Aux-, Air+Coil+, Air+Coil-, Air-Aux+, Air-Aux-, Air-Coil+, Air-Coil-, BMS_Sense, CANRX, CANTX, CAN_H, CAN_L, Final_Shutdown, GND, IMD_Sense, MISO, MOSI, P_LED_1, P_LED_2, P_LED_3, PrechargeCTL, Precharge_LSD, RESET, RJ45_LED1, RJ45_LED2, SCK, SS_BMS, SS_HVD, SS_HVDConn, SS_IMD, SS_MainTSConn, SS_TSMS, ShutdownSense_BMS, ShutdownSense_HVD, ShutdownSense_HVDConn, ShutdownSense_IMD, ShutdownSense_TSConn, ShutdownSense_TSMS, Shutdown_In, VCC
- wire segments 0 -> 158
- no-connect marks 0 -> 4
Other:
- note added: "(5V)"
- note added: "5V Indicator"
- note added: "AIR + Circuit"
- note added: "AIR - Circuit"
- note added: "Air+ Weld Detection"
- note added: "Air- Weld Detection"
- note added: "BUCK CONVERTER\n"
- note added: "CAN Transceiver"
- note added: "Connectors"
- note added: "MICROCONTROLLER"
- note added: "Power Flags"
- note added: "Precharge Circuit"
- note added: "Programming LEDs"
- note added: "Relay Circuits"
- note added: "Shutdown Sensing"
