File: repackaged/service_section_controller/imd_carryover.sch (KiCad schematic (older format))
At the start: 0 parts

Commit message: added ss carryover boards
Parts:
- added C1: C_2.2uF, footprints:C_0603_1608Metric, symbol IMD_LATCH-rescue:C_2.2uF-formula
- added C2: C_10uF_16V, footprints:C_0805_OEM, symbol IMD_LATCH-rescue:C_10uF_16V-Formula
- added C3, C4: C_0.1uF, footprints:C_0805_OEM, symbol IMD_LATCH-rescue:C_0.1uF-footprints
- added C5: C_0.1uF, footprints:C_0805_OEM, symbol IMD_LATCH-rescue:C_0.1uF-Formula
- added D1: D_Zener_18V, footprints:DO-214AA, symbol IMD_LATCH-rescue:D_Zener_18V-Formula
- added D2, D4: LED_0805, footprints:LED_0805_OEM, symbol IMD_LATCH-rescue:LED_0805-Formula
- added D3: D_Schottky_Small, footprints:D_0805_OEM, symbol Device:D_Schottky_Small
- added F1: F_500mA_16V, footprints:Fuse_1210, symbol IMD_LATCH-rescue:F_500mA_16V-Formula
- added J1: UF_5_VT, footprints:Ultrafit_5, symbol IMD_LATCH-rescue:UF_5_VT-formula
- added J2: MM_F_RA_04, footprints:micromatch_female_ra_4, symbol IMD_LATCH-rescue:MM_F_RA_04-Formula
- added J3: MicroFit_V_2, footprints:MicroFit_V_2, symbol IMD_LATCH-rescue:MicroFit_V_2-Formula
- added K1: G5Q-1A4-DC5-5V, footprints:Relay_SPST_OMRON-G5Q-1A4_OEM, symbol IMD_LATCH-rescue:G5Q-1A4-DC5-5V-Formula
- added Q1, Q2: SSM3K333R, footprints:SOT-23F, symbol IMD_LATCH-rescue:SSM3K333R-Formula
- added R1, R11: R_2.2K, footprints:R_0805_OEM, symbol IMD_LATCH-rescue:R_2.2K-Formula
- added R10: R_2.2K, footprints:R_0805_OEM, symbol IMD_LATCH-rescue:R_2.2K-formula
- added R12, R2: R_300K, footprints:R_0805_OEM, symbol IMD_LATCH-rescue:R_300K-Formula
- added R13, R3, R8: R_604K, footprints:R_0805_OEM, symbol IMD_LATCH-rescue:R_604K-Formula
- added R4, R5, R9: R_1K, footprints:R_0805_OEM, symbol IMD_LATCH-rescue:R_1K-Formula
- added R6: R_120K, footprints:R_0805_OEM, symbol IMD_LATCH-rescue:R_120K-Formula
- added R7: R_1.82M, footprints:R_0805_OEM, symbol IMD_LATCH-rescue:R_1.82M-formula
- added U1, U3: TLV3701QDBVRG4Q1, footprints:SOT-23-5_OEM, symbol IMD_LATCH-rescue:TLV3701QDBVRG4Q1-Formula
- added U2: CD4043BPWR, footprints:TSSOP-16-OEM, symbol IMD_LATCH-rescue:CD4043BPWR-formula
Connections:
- net labels added: +12V, 12V_Fused, GND, IMD_Output, IMD_Status_Output
- wire segments 0 -> 104
- no-connect marks 0 -> 4
Other:
- note added: "10V Output in 4.2 Sec delay\n"
- note added: "DELAY SIDE:\ntimer gives the IMD time to power up"
- note added: "I _lim: 20mA\n"
- note added: "IMD Output Status LED\n"
- note added: "IMD SIDE\nMakes analog imd signal digital\n"
- note added: "INPUT CONNECTOR\n\n"
- note added: "Latch outputs 12V when the IMD Output is “Healthy”"
- note added: "NAND LATCH\n"
- note added: "POWER MANAGEMENT / FUSING\n\n"
- note added: "Power Relay\n"
- note added: "SIGNAL LIGHT\nON = GOOD\n"
- note added: "This is IMD\n\n"
- note added: "t= -ln((10-x)/10)*2.662\n\n"
- note added: "“GOOD” Output is Logical High in a range of 0V-12V; Threshold set to +8V\n"
