File: repackaged/service_section_controller/tsal_carryover.sch (KiCad schematic (older format))
At the start: 0 parts

Commit message: added ss carryover boards
Parts:
- added C1: C_10uF, footprints:C_0805_OEM, symbol TSAL-AIL-rescue:C_10uF-Formula-TSAL-AIL-rescue
- added C2: C_0.1uF, footprints:C_0805_OEM, symbol TSAL-AIL-rescue:C_0.1uF-Formula-TSAL-AIL-rescue
- added C3: C_10uF_450V, footprints:C_10uF_450V, symbol Formula:C_10uF_450V
- added C4: C_1uF, Formula:C_0805_OEM, symbol TSAL-AIL-rescue:C_1uF-Formula-TSAL-AIL-rescue
- added C5: C_2.2uF, footprints:C_0805_OEM, symbol Formula:C_2.2uF
- added C6: C_470pF, footprints:C_0805_OEM, symbol Formula:C_470pF
- added C7: C_.22uF, footprints:C_0805_OEM, symbol Formula:C_.22uF
- added C8: C_100uF+, footprints:C_100uF+, symbol Formula:C_100uF+
- added C9: C_1uF, footprints:C_0805_OEM, symbol Formula:C_1uF
- added D1: LED_0805, footprints:LED_0805_OEM, symbol TSAL-AIL-rescue:LED_0805-Formula-TSAL-AIL-rescue
- added D2, D3, D4: Diode_600V_1A_SM, footprints:Diode_600V_1A_SM, symbol Formula:Diode_600V_1A_SM
- added J1: Ultrafit_4_RA, footprints:Ultrafit_4_RA, symbol Formula:Ultrafit_4_RA
- added J2: NanoFit_2, Formula:NanoFit_Molex_1x02x2.50mm_Angled_OEM, symbol TSAL-AIL-rescue:NanoFit_2-Formula-TSAL-AIL-rescue
- added J3: MM_F_RA_06, Formula:micromatch_female_ra_6, symbol TSAL-AIL-rescue:MM_F_RA_06-Formula-TSAL-AIL-rescue
- added L1: L_1.2mH, footprints:L_1.2mH, symbol Formula:L_1.2mH
- added Q1, Q2: SSM3K333R, Formula:SOT-23F, symbol TSAL-AIL-rescue:SSM3K333R-Formula-TSAL-AIL-rescue
- added R1: R_270K, footprints:R_0805_OEM, symbol Formula:R_270K
- added R10: R_6.04K, footprints:R_0805_OEM, symbol Formula:R_6.04K
- added R11: R_1K, footprints:R_0805_OEM, symbol TSAL-AIL-rescue:R_1K-Formula-TSAL-AIL-rescue
- added R12: R_499, footprints:R_0805_OEM, symbol TSAL-AIL-rescue:R_499-Formula-TSAL-AIL-rescue
- added R13, R14: R_10K, Formula:R_0805_OEM, symbol TSAL-AIL-rescue:R_10K-Formula-TSAL-AIL-rescue
- added R15: R_6.2K, footprints:R_0805_OEM, symbol Formula:R_6.2K
- added R16: R_3K, footprints:R_0805_OEM, symbol Formula:R_3K
- added R2: R_1.91K, footprints:R_0805_OEM, symbol Formula:R_1.91K
- added R3: R_51.1K, footprints:R_0805_OEM, symbol Formula:R_51.1K
- added R4, R6, R7: R_270K, footprints:R_0805_OEM, symbol TSAL-AIL-rescue:R_270K-Formula-TSAL-AIL-rescue
- added R5: R_10K, footprints:R_0805_OEM, symbol TSAL-AIL-rescue:R_10K-Formula-TSAL-AIL-rescue
- added R8: R_10K, footprints:R_0805_OEM, symbol Formula:R_10K
- added R9: R_1.43K, footprints:R_0805_OEM, symbol TSAL-AIL-rescue:R_1.43K-Formula-TSAL-AIL-rescue
- added U1: MCP6001, Package_TO_SOT_SMD:SOT-23-5, symbol Formula:MCP6001
- added U2: Buck_Converter_450V_300mA, footprints:Converter_DCDC_MPS_MP9488, symbol Formula:Buck_Converter_450V_300mA
- added U3: CPC1025NTR, footprints:DIP-5-6_W7.62mm, symbol Formula:CPC1025NTR
- added U4: BU4S11G2-TR, Formula:SSOP5, symbol Formula:BU4S11G2-TR
Connections:
- net labels added: 15V+, 15V-, AIL+, AIL-, FB, GLV+, GND, NAND_Out, SW, TS+, TS-, TSAL_FLAG, TSAL_GREEN+, TSAL_GREEN-, TSAL_RED+, TSAL_RED-, VCC
- wire segments 0 -> 116
Other:
- note added: "GREEN TSAL\n"
- note added: "HV"
- note added: "LV\n\n"
- note added: "RED TSAL"
