File: repackaged/service_section_controller/service_section_controller.kicad_pcb (KiCad board)
At the start: 2 copper layers, 211 parts, among them IC1001 ATMEGA16M1, J1001 CONN_02X03, J1002 CONN_02X03, J301 UF_5_VT, J401 MM_F_VT_16, J402 MM_F_VT_16, J403 MicroFit_VT_12, J404 Ultrafit_4_RA, J405 Ultrafit_4_RA, J801 B5B-PH-K-S, J802 isoSPI-Cutout, K301 G5Q-1A4-DC5-5V, K801 G5Q-1A4-DC12, Q301 SSM3K333R, Q302 SSM3K333R, Q501 SSM3K333R, Q502 SSM3K333R, Q503 SSM3K333R, Q504 SSM3K333R, Q505 SSM3K333R, Q506 SSM3K333R, Q801 SSM3K333R, Q901 SSM3K333R, Q902 SSM3K333R, T801 T_LAN_SM91501ALE, U1001 MCP2561-E_SN, U1002 MCP2561-E_SN, U1003 ATMEGA16M1, U201 TPS560430YF, U301 TLV3701QDBVRG4Q1, U302 TLV3701QDBVRG4Q1, U303 CD4043BPWR, U601 MCP6001, U602 CPC1025NTR, U701 MP9488, U702 LR8K4-G, U801 SN74LVC1G17, U802 LTC6820HMS, U803 MCP6001, U804 MCP6001, U805 MCP6001, U806 SN74LVC1G32DBVR, Y1001 Crystal_SMD, Y1002 Crystal_SMD

Commit message: updated layout and schematic
Parts:
- removed IC1001: ATMEGA16M1, footprints:TQFP-32_7x7mm_Pitch0.8mm
- added J1101: MicroFit_VT_12, footprints:MicroFit_VT_12, F.Cu at (139.6, 84.3)
- added J601: NanoFit_2, footprints:NanoFit_Molex_1x02x2.50mm_Angled_OEM, F.Cu at (275.7, 176.0)
- added Q601: SSM3K333R, footprints:SOT-23F, F.Cu at (315.8, 72.7)
- added Q602: SSM3K333R, footprints:SOT-23F, F.Cu at (314.2, 28.1)
- added R313: R_2.2K, footprints:R_0805_OEM, F.Cu at (119.3, 126.4)
- added R314: R_1K, footprints:R_0805_OEM, F.Cu at (115.3, 126.4)
- added R315: R_1.13K, footprints:R_0805_OEM, F.Cu at (115.6, 122.4)
- added R611: R_10K, footprints:R_0805_OEM, F.Cu at (315.5, 37.0)
- added R612: R_10K, footprints:R_0805_OEM, F.Cu at (310.6, 76.2)
- added R707: R_23.7K, footprints:R_0805_OEM, F.Cu at (346.9, 121.4)
- added U1004: ATMEGA64M1, footprints:TQFP-32_7x7mm_Pitch0.8mm, F.Cu at (165.1, 117.8)
- added U603: BU4S11G2-TR, footprints:SSOP5, F.Cu at (311.0, 72.6)
- C701, L701: moved to B.Cu
- D301: value D_Schottky_Small -> BAS40-00; footprint footprints:D_0805_OEM -> Package_TO_SOT_SMD:SOT-23
- J402: value MM_F_VT_16 -> MM_F_VT_18; footprint footprints:micromatch_female_vert_16 -> footprints:micromatch_female_vert_18
- K301: value G5Q-1A4-DC5-5V -> G5Q-1A4-DC12
- R1011: value R_100K -> R_100
- R702: value R_3K -> R_43k
- R703: value R_6.04K -> R_23.7K
- R704: value R_6.2K -> R_4.99K
- R705: value R_1K -> R_6.04K
- U303: value CD4043BPWR -> CD4044BDR; footprint footprints:TSSOP-16-OEM -> footprints:SOIC127P600X175-16N
- moved C701 542.8 mm to (384.9, 148.7)
- moved R603 535.3 mm to (387.6, 85.6), turned to 90 degrees
- moved R606 535.1 mm to (386.5, 77.7)
- moved R602 532.3 mm to (379.8, 87.8)
- moved R601 532.1 mm to (390.7, 74.8)
- moved R604 532.1 mm to (390.7, 77.7)
- moved R607 530.1 mm to (386.5, 74.5)
- moved R605 524.0 mm to (386.7, 81.2)
- moved C706 523.2 mm to (400.8, 109.7)
- moved C602 516.2 mm to (363.5, 62.7)
- moved U601 515.9 mm to (369.8, 68.5)
- moved D601 513.0 mm to (356.0, 69.5)
- moved C601 510.4 mm to (363.6, 58.7)
- moved F702 509.7 mm to (382.8, 118.3)
- moved D703 507.7 mm to (365.5, 117.4), turned to 180 degrees
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Connections:
- net Net-(C201-Pad1) renamed /power_main/12v_BUCK
- D301 pad 1: 12V_SHUTDOWN -> Net-(D301-Pad1)
- D301 pad 2: Net-(D301-Pad2) -> (no net)
- J402 pad 17: (no net) -> Net-(J402-Pad17)
- K301 pad 1: Net-(D301-Pad2) -> Net-(D301-Pad1)
- Q301 pad 1: IMD_STATUS_OUTPUT -> /imd_latch/LATCH_OUTPUT
- Q301 pad 3: Net-(D301-Pad2) -> Net-(D301-Pad1)
- Q302 pad 1: IMD_STATUS_OUTPUT -> /imd_latch/LATCH_OUTPUT
- R205 pad 1: +5V -> Net-(COUT201-Pad1)
- R311 pad 1: IMD_STATUS_OUTPUT -> /imd_latch/LATCH_OUTPUT
- R702 pad 2: 15V- -> Net-(R702-Pad2)
- R703 pad 1: Net-(C704-Pad1) -> Net-(R702-Pad2)
- R703 pad 2: Net-(R703-Pad2) -> 15V-
- R704 pad 1: Net-(R703-Pad2) -> /power_secondary.sch/FB
- T801 pad 1: Net-(R809-Pad1) -> IM
- T801 pad 10: IP -> Net-(R810-Pad2)
- T801 pad 11: Net-(T801-Pad11) -> Net-(C805-Pad1)
- T801 pad 12: IM -> Net-(R809-Pad1)
- T801 pad 2: Net-(C805-Pad1) -> Net-(T801-Pad2)
- T801 pad 3: Net-(R810-Pad2) -> IP
- U303 pad 13: Net-(U303-Pad13) -> /imd_latch/LATCH_OUTPUT
- U303 pad 2: IMD_STATUS_OUTPUT -> Net-(U303-Pad2)
Routing:
- net +AIR_COIL-: track 0.00 -> 244.5 mm, vias 0 -> 80
- net 12V_IMD: track 0.00 -> 215.3 mm, vias 0 -> 2
- net IMD_STATUS_OUTPUT: track 0.00 -> 191.0 mm, vias 0 -> 4
- net +AIR_COIL+: track 0.00 -> 131.3 mm
- net Net-(R809-Pad1): track 0.00 -> 125.1 mm
- net Net-(R810-Pad2): track 0.00 -> 109.6 mm
- net Net-(C805-Pad1): track 0.00 -> 99.0 mm
- net PM_SCK: track 0.00 -> 92.9 mm, vias 0 -> 6
- net 12V_SHUTDOWN: track 0.00 -> 90.4 mm
- net PM_RESET: track 0.00 -> 89.0 mm, vias 0 -> 4
- net BSPD_CURRENT_SENSE: track 0.00 -> 88.9 mm, vias 0 -> 4
- net PM_MOSI: track 0.00 -> 80.7 mm, vias 0 -> 4
- net PM_MISO: track 0.00 -> 78.2 mm, vias 0 -> 6
- net CHARGE_ENABLE1: track 0.00 -> 76.9 mm, vias 0 -> 6
- net CHARGE_ENABLE2: track 0.00 -> 73.9 mm, vias 0 -> 6
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- added copper zone on F.Cu, net +AIR_COIL-
- added copper zone on F.Cu, net 15V-
- added copper zone on F.Cu, net Net-(C203-Pad1)
- added copper zone on F.Cu, net Net-(C203-Pad2)
- added copper zone on F.Cu, net Net-(COUT201-Pad1)
- added copper zone on F.Cu, net TS+
Other:
- copper layers 2 -> 4
- board text added: "400V - 15V Lin Reg (DNP)"
- board text added: "AIR CONTROL RELAY CIRCUITS"
- board text added: "AIR+"
- board text added: "AIR+ WELD"
- board text added: "AIR-"
- board text added: "AIR- WELD"
- board text added: "BMS"
- board text added: "GLV"
- board text added: "HV"
- board text added: "HVD"
- board text added: "HVD CONN"
- board text added: "IMD LATCH"
- board text added: "IMD LED"
- board text added: "IMD Shutdown Relay"
- board text added: "MPC"
- board text added: "PRECHARGE"
- board text added: "Primary CAN Tranceiver"
- board text added: "Primary Micro"
- board text added: "Primary Micro LEDs"
- board text added: "Programming Headers"
- board text added: "Secondary CAN Tranceiver"
- board text added: "Secondary Micro"
- board text added: "Secondary Micro LEDs"
- board text added: "Shutdown Sense"
- board text added: "TSMS"
- board text added: "i need help with the buck please"

Commit message: removed all traces and planes from layout. started adding test points
Parts:
- added REF**: TestPoint_Pad_D1.5mm, TestPoint:TestPoint_Pad_D1.5mm, F.Cu at (196.1, 68.6)
- added REF**: TestPoint_Pad_D1.5mm, TestPoint:TestPoint_Pad_D1.5mm, F.Cu at (196.1, 65.8)
- added REF**: TestPoint_Pad_D1.5mm, TestPoint:TestPoint_Pad_D1.5mm, F.Cu at (196.1, 63.0)
- added REF**: TestPoint_Pad_D1.5mm, TestPoint:TestPoint_Pad_D1.5mm, F.Cu at (196.1, 60.2)
- C701, L701: moved to F.Cu
- C702, C703, C704, D701, R701, R704, R707, U701: moved to B.Cu
- moved C201 138.4 mm to (36.3, 120.7)
- moved C202 138.4 mm to (34.4, 120.7)
- moved C203 138.4 mm to (28.1, 120.8)
- moved COUT201 138.4 mm to (23.6, 119.9)
- moved COUT202 138.4 mm to (23.1, 117.5)
- moved COUT203 138.4 mm to (24.8, 113.0)
- moved D201 138.4 mm to (40.4, 119.9)
- moved D202 138.4 mm to (47.1, 121.8)
- moved D203 138.4 mm to (29.1, 107.2)
- moved F201 138.4 mm to (40.1, 107.2)
- moved F202 138.4 mm to (40.1, 111.9)
- moved F203 138.4 mm to (36.0, 116.6)
- moved F204 138.4 mm to (63.6, 124.8)
- moved F205 138.4 mm to (58.4, 124.8)
- moved F206 138.4 mm to (52.8, 124.8)
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Routing:
- net +AIR_COIL-: track 244.5 -> 0.00 mm, vias 80 -> 0
- net 12V_IMD: track 215.3 -> 0.00 mm, vias 2 -> 0
- net IMD_STATUS_OUTPUT: track 191.0 -> 0.00 mm, vias 4 -> 0
- net +AIR_COIL+: track 131.3 -> 0.14 mm
- net Net-(R809-Pad1): track 125.1 -> 0.00 mm
- net Net-(R810-Pad2): track 109.6 -> 0.00 mm
- net Net-(C805-Pad1): track 99.0 -> 0.00 mm
- net PM_SCK: track 92.9 -> 0.07 mm, vias 6 -> 0
- net 12V_SHUTDOWN: track 90.4 -> 0.00 mm
- net PM_RESET: track 89.0 -> 0.00 mm, vias 4 -> 0
- net BSPD_CURRENT_SENSE: track 88.9 -> 0.00 mm, vias 4 -> 0
- net PM_MOSI: track 80.7 -> 0.00 mm, vias 4 -> 0
- net PM_MISO: track 78.2 -> 0.00 mm, vias 6 -> 0
- net CHARGE_ENABLE1: track 76.9 -> 0.00 mm, vias 6 -> 0
- net CHARGE_ENABLE2: track 73.9 -> 0.00 mm, vias 6 -> 0
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- removed copper zone on F.Cu, net 15V-
- removed copper zone on F.Cu, net TS+
Other:
- rule trace_min: 0.2 -> 0.01
- board text removed: "i need help with the buck please"

Commit message: added test points and re-did schematic with new traces.
Parts:
- removed REF** (x4): TestPoint_Pad_D1.5mm, TestPoint:TestPoint_Pad_D1.5mm
- added TP201: 5V_BMS, TestPoint:TestPoint_Pad_D1.0mm, F.Cu at (175.9, 182.7)
- added TP202: 5V_AIR_CONTROL, TestPoint:TestPoint_Pad_D1.0mm, F.Cu at (189.4, 172.8)
- added TP203: FB, TestPoint:TestPoint_Pad_D1.0mm, F.Cu at (175.8, 135.0)
- added TP204: 12V_TSAL, TestPoint:TestPoint_Pad_D1.0mm, F.Cu at (212.2, 101.3)
- added TP205: 12V_IMD, TestPoint:TestPoint_Pad_D1.0mm, F.Cu at (162.0, 114.1)
- added TP206: 12V_SHUTDOWN, TestPoint:TestPoint_Pad_D1.0mm, F.Cu at (163.2, 127.6)
- added TP207: 12V_BUCK, TestPoint:TestPoint_Pad_D1.0mm, F.Cu at (178.1, 149.7)
- added TP208: BUCK_OUTPUT, TestPoint:TestPoint_Pad_D1.0mm, F.Cu at (177.5, 129.4)
- added TP301: IMD_OUTPUT, TestPoint:TestPoint_Pad_D1.0mm, F.Cu at (146.3, 101.9)
- added TP302: Test_Point_SMD, TestPoint:TestPoint_Pad_D1.0mm, F.Cu at (146.3, 108.7)
- added TP303: Test_Point_SMD, TestPoint:TestPoint_Pad_D1.0mm, F.Cu at (146.3, 111.0)
- added TP304: 8V_OPAMP, TestPoint:TestPoint_Pad_D1.0mm, F.Cu at (146.3, 104.1)
- added TP305: OPAMP_OUTPUT, TestPoint:TestPoint_Pad_D1.0mm, F.Cu at (146.3, 106.4)
- added TP306: Test_Point_SMD, TestPoint:TestPoint_Pad_D1.0mm, F.Cu at (146.3, 113.4)
- added TP307: Test_Point_SMD, TestPoint:TestPoint_Pad_D1.0mm, F.Cu at (146.3, 115.8)
- added TP308: IMD_STATUS_OUTPUT, TestPoint:TestPoint_Pad_D1.0mm, F.Cu at (148.1, 120.7)
- added TP501: DETECT_MPC, TestPoint:TestPoint_Pad_D1.0mm, F.Cu at (215.9, 106.6)
- added TP502: DETECT_HVD_CONN, TestPoint:TestPoint_Pad_D1.0mm, F.Cu at (213.6, 106.6)
- added TP503: DETECT_HVD, TestPoint:TestPoint_Pad_D1.0mm, F.Cu at (204.4, 106.6)
- added TP504: SS_HVD_CONN, TestPoint:TestPoint_Pad_D1.0mm, F.Cu at (211.3, 106.6)
- added TP505: SS_HVD, TestPoint:TestPoint_Pad_D1.0mm, F.Cu at (206.5, 138.6)
- added TP506: SS_MPC, TestPoint:TestPoint_Pad_D1.0mm, F.Cu at (214.1, 138.6)
- added TP507: DETECT_IMD_LATCH, TestPoint:TestPoint_Pad_D1.0mm, F.Cu at (206.7, 106.6)
- added TP508: DETECT_BMS, TestPoint:TestPoint_Pad_D1.0mm, F.Cu at (209.0, 106.6)
- added TP509: DETECT_TSMS, TestPoint:TestPoint_Pad_D1.0mm, F.Cu at (211.5, 138.6)
- added TP510: SS_BMS, TestPoint:TestPoint_Pad_D1.0mm, F.Cu at (216.6, 138.6)
- added TP511: SS_IMD_LATCH, TestPoint:TestPoint_Pad_D1.0mm, F.Cu at (204.2, 138.6)
- added TP512: SS_TSMS, TestPoint:TestPoint_Pad_D1.0mm, F.Cu at (209.0, 138.6)
- added TP601: 15V+, TestPoint:TestPoint_Pad_D1.0mm, F.Cu at (264.0, 99.1)
- added TP602: VIN, TestPoint:TestPoint_Pad_D1.0mm, F.Cu at (251.8, 104.9)
- added TP603: 15V+, TestPoint:TestPoint_Pad_D1.0mm, F.Cu at (256.3, 102.6)
- added TP604: VREF, TestPoint:TestPoint_Pad_D1.0mm, F.Cu at (251.8, 90.6)
- added TP605: OPAMP_OUTPUT, TestPoint:TestPoint_Pad_D1.0mm, F.Cu at (264.0, 96.5)
- added TP606: TSAL_FLAG, TestPoint:TestPoint_Pad_D1.0mm, F.Cu at (201.6, 105.2)
- added TP701: 15V+_OUTPUT, TestPoint:TestPoint_Pad_D1.0mm, F.Cu at (255.5, 173.1)
- added TP702: FB, TestPoint:TestPoint_Pad_D1.0mm, F.Cu at (249.2, 151.3)
- added TP703: 15V+_OUTPUT, TestPoint:TestPoint_Pad_D1.0mm, F.Cu at (233.2, 136.3)
- added TP704: 15V_RETURN, TestPoint:TestPoint_Pad_D1.0mm, F.Cu at (281.2, 142.9)
- added TP801: Test_Point_SMD, TestPoint:TestPoint_Pad_D1.0mm, F.Cu at (165.1, 178.8)
- added TP802: VOUT, TestPoint:TestPoint_Pad_D1.0mm, F.Cu at (157.2, 178.8)
- added TP803: VREF, TestPoint:TestPoint_Pad_D1.0mm, F.Cu at (160.0, 178.8)
- added TP804: Test_Point_SMD, TestPoint:TestPoint_Pad_D1.0mm, F.Cu at (165.6, 159.7)
- added TP805: Test_Point_SMD, TestPoint:TestPoint_Pad_D1.0mm, F.Cu at (170.1, 178.8)
- added TP806: Test_Point_SMD, TestPoint:TestPoint_Pad_D1.0mm, F.Cu at (172.7, 178.8)
- added TP807: Test_Point_SMD, TestPoint:TestPoint_Pad_D1.0mm, F.Cu at (162.8, 178.8)
- added TP808: Test_Point_SMD, TestPoint:TestPoint_Pad_D1.0mm, F.Cu at (159.2, 164.3)
- added TP809: Test_Point_SMD, TestPoint:TestPoint_Pad_D1.0mm, F.Cu at (167.6, 178.8)
- added TP901: PRECHARGE_CTL, TestPoint:TestPoint_Pad_D1.0mm, F.Cu at (205.1, 146.5)
- added TP902: PRECHARGE_LSD, TestPoint:TestPoint_Pad_D1.0mm, F.Cu at (207.4, 146.5)
- added TP903: -AIR_WELD_DETECT, TestPoint:TestPoint_Pad_D1.0mm, F.Cu at (212.0, 146.5)
- added TP904: -AIR_LSD, TestPoint:TestPoint_Pad_D1.0mm, F.Cu at (214.3, 146.5)
- added TP905: +AIR_WELD_DETECT, TestPoint:TestPoint_Pad_D1.0mm, F.Cu at (209.7, 146.5)
- added TP906: -AIR_COIL-, TestPoint:TestPoint_Pad_D1.0mm, F.Cu at (216.6, 146.5)
- added TP907: +AIR_COIL+, TestPoint:TestPoint_Pad_D1.0mm, F.Cu at (202.9, 146.5)
- BSPD801, IM801, IP801: footprint footprints:Test_Point_SMD -> TestPoint:TestPoint_Pad_D1.0mm
- moved F702 209.3 mm to (231.4, 130.9), turned to 270 degrees
- moved D703 197.2 mm to (236.5, 129.4), turned to 270 degrees
- moved R706 190.9 mm to (265.7, 105.0), turned to 0 degrees
- moved C707 186.2 mm to (265.7, 108.8), turned to 0 degrees
- moved L701 182.1 mm to (250.2, 127.9), turned to 270 degrees
- moved C706 180.7 mm to (261.9, 115.8), turned to 90 degrees
- moved D701 174.6 mm to (236.5, 144.4), turned to 270 degrees
- moved C704 170.0 mm to (244.7, 140.0), turned to 0 degrees
- moved D203 169.5 mm to (196.8, 131.6), turned to 180 degrees
- moved R707 169.4 mm to (239.6, 146.3), turned to 270 degrees
- moved COUT203 166.8 mm to (191.0, 127.3), turned to 90 degrees
- moved R701 166.2 mm to (239.0, 150.7), turned to 0 degrees
- moved R205 164.5 mm to (195.7, 136.1), turned to 90 degrees
- moved C702 164.1 mm to (243.5, 147.6), turned to 90 degrees
- moved COUT202 163.6 mm to (186.5, 125.7), turned to 90 degrees
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Connections:
- net /power_main/12v_BUCK renamed /power_main/12V_BUCK
- net 15V- renamed 15V_RETURN
- J801 pad 3: VOUT -> +AIR_COIL-
- J801 pad 4: VREF -> +AIR_COIL-
- J801 pad 5: nOCD -> +AIR_COIL-
- R801 pad 2: nOCD -> +AIR_COIL-
- R802 pad 1: VOUT -> +AIR_COIL-
- R803 pad 1: VOUT -> +AIR_COIL-
- R804 pad 1: VREF -> +AIR_COIL-
- R808 pad 2: Net-(R808-Pad2) -> +AIR_COIL-
- U1004 pad 16: nOCD -> +AIR_COIL-
- U1004 pad 17: VREF -> +AIR_COIL-
- U1004 pad 18: VOUT -> +AIR_COIL-
- U803 pad 1: Net-(R808-Pad2) -> +AIR_COIL-
- U804 pad 4: VOUT -> +AIR_COIL-
- U805 pad 3: Net-(R808-Pad2) -> +AIR_COIL-
Routing:
- net +AIR_COIL-: track 0.00 -> 333.9 mm, vias 0 -> 52
- net Net-(R810-Pad2): track 0.00 -> 190.9 mm, vias 0 -> 2
- net 15V_RETURN: track 0.00 -> 187.1 mm, vias 2 -> 9
- net Net-(R809-Pad1): track 0.00 -> 185.7 mm, vias 0 -> 2
- net IMD_STATUS_OUTPUT: track 0.00 -> 159.4 mm, vias 0 -> 2
- net TS+: track 0.00 -> 114.6 mm, vias 1 -> 4
- net 5V_BMS: track 0.00 -> 113.3 mm, vias 0 -> 10
- net SS_HVD: track 0.00 -> 110.6 mm, vias 0 -> 5
- net PM_MOSI: track 0.00 -> 99.9 mm, vias 0 -> 4
- net SM_MOSI: track 0.00 -> 99.8 mm, vias 0 -> 2
- net TSAL_GREEN-: track 0.00 -> 95.0 mm, vias 0 -> 2
- net PM_MISO: track 0.00 -> 86.4 mm, vias 0 -> 2
- net SS_MPC: track 0.00 -> 83.3 mm, vias 0 -> 3
- net SS_BMS: track 0.00 -> 81.5 mm, vias 0 -> 3
- net PM_RESET: track 0.00 -> 77.9 mm, vias 0 -> 6
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- added copper zone on In2.Cu_PWR, net +AIR_AUX+
- added copper zone on In1.Cu_GND, net +AIR_COIL-
- added copper zone on B.Cu, net /power_secondary.sch/SW
- added copper zone on In2.Cu_PWR, net 12V_IMD
- added copper zone on B.Cu, net 15V_RETURN
- added copper zone on F.Cu, net 15V_RETURN
- added copper zone on In2.Cu_PWR, net 5V_BMS
- added copper zone on B.Cu, net Net-(C704-Pad1)
- added copper zone on B.Cu, net Net-(C706-Pad1)
- added copper zone on B.Cu, net TS+
- added copper zone on F.Cu, net TS+
Other:
- board text added: "LV"
- board text added: "should I remove these?"
- board text removed: "AIR CONTROL RELAY CIRCUITS"
