File: repackaged/sensing_controller/wheel_speed.sch (KiCad schematic (older format))
At the start: 0 parts

Commit message: Copy over wheel speed carryover schematic.
Parts:
- added C1, C101, C103, C2, C6: C_0.1uF, footprints:C_0805_OEM, symbol formula:C_0.1uF
- added C102: C_2.2uF, footprints:C_0603_1608Metric, symbol formula:C_2.2uF
- added C3: C_100pF, footprints:C_0805_OEM, symbol formula:C_100pF
- added C4, C5: C_30pF, footprints:C_0805_OEM, symbol formula:C_30pF
- added COUT101: C_22uF, footprints:C_1206_OEM, symbol formula:C_22uF
- added COUT102: C_33uF, footprints:C_1812_OEM, symbol formula:C_33uF
- added COUT103: C_47uF, footprints:C_0805_OEM, symbol formula:C_47uF
- added D1, D102, D103, D2, D3: LED_0805, footprints:LED_0805_OEM, symbol formula:LED_0805
- added D101: D_Zener_18V, footprints:DO-214AA, symbol formula:D_Zener_18V
- added F101: F_500mA_16V, footprints:Fuse_1210, symbol formula:F_500mA_16V
- added J1: CONN_02X03, footprints:Pin_Header_Straight_2x03, symbol formula:CONN_02X03
- added J2: MM_F_RA_08, footprints:micromatch_female_ra_8, symbol formula:MM_F_RA_08
- added JP1: FRONT_BACK, Jumper:SolderJumper-2_P1.3mm_Open_RoundedPad1.0x1.5mm, symbol Device:Jumper_NO_Small
- added JP2: LEFT_RIGHT, Jumper:SolderJumper-2_P1.3mm_Open_RoundedPad1.0x1.5mm, symbol Device:Jumper_NO_Small
- added L101: L_100uH, formula:L_100uH, symbol formula:L_100uH
- added R1: R_100, footprints:R_0805_OEM, symbol formula:R_100
- added R101, R105, R6, R7, R8: R_200, footprints:R_0805_OEM, symbol formula:R_200
- added R102: R_25K, footprints:R_0805_OEM, symbol formula:R_25K
- added R103: R_100K, footprints:R_0805_OEM, symbol formula:R_100K
- added R104: R_0_2512, footprints:R_2512_OEM, symbol formula:R_0_2512
- added R2: R_120_DNP, footprints:R_0805_OEM, symbol formula:R_120_DNP
- added R3, R4, R5: R_10K, footprints:R_0805_OEM, symbol formula:R_10K
- added U1: MCP2561-E_SN, footprints:SOIC-8_3.9x4.9mm_Pitch1.27mm_OEM, symbol formula:MCP2561-E_SN
- added U101: TPS560430YF, Package_TO_SOT_SMD:SOT-23-6_Handsoldering, symbol formula:TPS560430YF
- added U2: ATMEGA16M1, footprints:TQFP-32_7x7mm_Pitch0.8mm, symbol formula:ATMEGA16M1
- added Y1: Crystal_SMD, footprints:Crystal_SMD_FA238, symbol formula:Crystal_SMD
Connections:
- net labels added: 12V, 5V, CAN_HI, CAN_LO, CAN_RX, CAN_TX, DEBUG, FRONT_SENSE, GND, LEFT_SENSE, MISO, MOSI, RESET, SCK, SENSE_IN, VCC
- wire segments 0 -> 109
- no-connect marks 0 -> 17
Other:
- note added: "12V Indicator"
- note added: "16 MHz CRYSTAL\n"
- note added: "16M1 PROGRAMMING HEADER\n"
- note added: "5V"
- note added: "5V Indicator"
- note added: "ATMEGA 16M1\n"
- note added: "BUCK CONVERTER\n"
- note added: "Bootstrap Capacitor\n"
- note added: "CAN TRANSCEIVER\n"
- note added: "CONFIG"
- note added: "CONNECTOR\nPOWER, GND, CAN, SENSOR"
- note added: "DEBUG"
- note added: "Feedback Divider\n"
- note added: "Inductor\n"
- note added: "Input Capacitors\n\n"
- note added: "Output Capacitors\n"
- note added: "POWER FLAGS\n"
- note added: "Protection\n"
- note added: "VCC Jumper\n"
