File: Boards/lv_bms_2/lv_bms_2/lv_bms_2.sch (KiCad schematic (older format))
At the start: 44 parts, among them J1 CONN_02X03, U1 MCP2561-E_SN, U101 TPS560430YF, U2 ATMEGA16M1, Y1 Crystal_SMD

Commit message: lv_bms_2 schematic first pass
Parts:
- added C10, C6, C7, C8, C9: C_10nF, footprints:C_1206_OEM, symbol formula:C_10nF
- added C11, C12: C_1uF, footprints:C_0805_OEM, symbol formula:C_1uF
- added C13: C_0.1uF, footprints:C_0805_OEM, symbol formula:C_0.1uF
- added D? (x2): LED_0805_Red, footprints:LED_0805_OEM, symbol formula:LED_0805_Red
- added D? (x2): LED_0805, footprints:LED_0805_OEM, symbol formula:LED_0805
- added J3: NanoFit_RA_TH_06, footprints:NanoFit_RA_6, symbol formula:NanoFit_RA_TH_06
- added Q1: NSS1C201MZ4, footprints:SOT-223, symbol formula:NSS1C201MZ4
- added Q2: MMBF170, TO_SOT_Packages_SMD:SOT-23, symbol formula:MMBF170
- added R10, R11, R12, R13, R14, R9: R_100, footprints:R_0805_OEM, symbol formula:R_100
- added R18, R28: R_25K, footprints:R_0805_OEM, symbol formula:R_25K
- added R19, R20, R21, R25, R26, R29: R_1K, footprints:R_0805_OEM, symbol formula:R_1K
- added R22, R27: R_22K, footprints:R_0805_OEM, symbol formula:R_22K
- added R4, R5, R6, R7, R8: 356030RFT, formula:356030RFT, symbol formula:356030RFT
- added R? (x4): R_200, footprints:R_0805_OEM, symbol formula:R_200
- added R?: R_100K, footprints:R_0805_OEM, symbol formula:R_100K
- added R?: R_5K, footprints:R_0805_OEM, symbol formula:R_10K
- added TP1, TP2, TP3, TP4, TP5, TP6: Test_Point_SMD, footprints:Test_Point_SMD, symbol formula:Test_Point_SMD
- added U4: MCP6001T-I-LT, Package_TO_SOT_SMD:SOT-353_SC-70-5, symbol formula:MCP6001T-I-LT
- added U6, U7: TLV3701QDBVRG4Q1, footprints:SOT-23-5_OEM, symbol formula:TLV3701QDBVRG4Q1
- gave numbers to parts that had none: 15
Connections:
- net labels added: +5V-power, 2A_in, 2A_out, CAN_STBY, CSB, CURRENT_SENSE_IN, LED_0, LED_1, LED_2, LED_3, RELAY, RELAY_GND, batt_0, batt_1, batt_2, batt_3, batt_4
- wire segments 108 -> 199
- no-connect marks 4 -> 25
Other:
- note added: "LTC6810-1"
- note added: "Programming LEDs"
- note added: "analog I2C mux with current buffer"
- note added: "compartors @ > 2.6V | < 2.4V +- 2A\nfor powering BMS system on"
- note added: "connectors"
- note added: "current measurement thermistors"
- note added: "level triggered external interrupt \nto wake uC from sleep"
- note added: "thermistor mux"
- moved on the sheet: C14, C15, J2, J4, J5, R15, R16, R17, R23, R24, R30, R31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

Commit message: added .pdf for rev1 lv_bms_2
Parts:
- gave numbers to parts that had none: 10
Changed lines of the file:
@@
 RELAY
 $Comp
-L formula:LED_0805_Red D?
+L formula:LED_0805_Red D1
 U 1 1 617D5575
 P 5925 2075
-F 0 "D?" V 5925 2000 50  0000 R CNN
+F 0 "D1" V 5925 2000 50  0000 R CNN
 F 1 "LED_0805_Red" H 6175 2200 50  0000 R CNN
 F 2 "footprints:LED_0805_OEM" H 5825 2075 50  0001 C CNN
@@
 $EndComp
 $Comp
-L formula:LED_0805_Red D?
+L formula:LED_0805_Red D2
 U 1 1 617D947A
 P 6275 2075
-F 0 "D?" V 6275 2000 50  0000 R CNN
+F 0 "D2" V 6275 2000 50  0000 R CNN
 F 1 "LED_0805_Red" H 6525 2175 50  0000 R CNN
 F 2 "footprints:LED_0805_OEM" H 6175 2075 50  0001 C CNN
@@
 $EndComp
 $Comp
-L formula:LED_0805 D?
+L formula:LED_0805 D3
 U 1 1 617DB227
 P 6600 2075
-F 0 "D?" V 6600 2000 50  0000 R CNN
+F 0 "D3" V 6600 2000 50  0000 R CNN
 F 1 "LED_0805" H 6750 2175 50  0000 R CNN
 F 2 "footprints:LED_0805_OEM" H 6500 2075 50  0001 C CNN
@@
 $EndComp
 $Comp
-L formula:LED_0805 D?
+L formula:LED_0805 D4
 U 1 1 617DC0FC
 P 6925 2075
-F 0 "D?" V 6925 2000 50  0000 R CNN
+F 0 "D4" V 6925 2000 50  0000 R CNN
 F 1 "LED_0805" H 7075 2150 50  0000 R CNN
 F 2 "footprints:LED_0805_OEM" H 6825 2075 50  0001 C CNN
@@
 $EndComp
 $Comp
-L lv_bms_2-rescue:GND-power #PWR?
+L lv_bms_2-rescue:GND-power #PWR0136
 U 1 1 617EF401
 P 5925 2225
-F 0 "#PWR?" H 5925 1975 50  0001 C CNN
+F 0 "#PWR0136" H 5925 1975 50  0001 C CNN
 F 1 "GND" H 5930 2052 50  0000 C CNN
 F 2 "" H 5925 2225 50  0001 C CNN
@@
 $EndComp
 $Comp
-L lv_bms_2-rescue:GND-power #PWR?
+L lv_bms_2-rescue:GND-power #PWR0137
 U 1 1 617FB1B0
 P 6275 2225
-F 0 "#PWR?" H 6275 1975 50  0001 C CNN
+F 0 "#PWR0137" H 6275 1975 50  0001 C CNN
 F 1 "GND" H 6280 2052 50  0000 C CNN
 F 2 "" H 6275 2225 50  0001 C CNN
@@
 $EndComp
 $Comp
-L lv_bms_2-rescue:GND-power #PWR?
+L lv_bms_2-rescue:GND-power #PWR0138
 U 1 1 6180742F
 P 6600 2225
-F 0 "#PWR?" H 6600 1975 50  0001 C CNN
+F 0 "#PWR0138" H 6600 1975 50  0001 C CNN
 F 1 "GND" H 6605 2052 50  0000 C CNN
 F 2 "" H 6600 2225 50  0001 C CNN
@@
 $EndComp
 $Comp
-L lv_bms_2-rescue:GND-power #PWR?
+L lv_bms_2-rescue:GND-power #PWR0139
 U 1 1 61813340
 P 6925 2225
-F 0 "#PWR?" H 6925 1975 50  0001 C CNN
+F 0 "#PWR0139" H 6925 1975 50  0001 C CNN
 F 1 "GND" H 6930 2052 50  0000 C CNN
 F 2 "" H 6925 2225 50  0001 C CNN
@@
 $EndComp
 $Comp
-L formula:R_200 R?
+L formula:R_200 R35
 U 1 1 6186CE56
 P 6600 1775
-F 0 "R?" H 6670 1821 50  0000 L CNN
+F 0 "R35" H 6670 1821 50  0000 L CNN
 F 1 "R_200" V 6500 1675 50  0000 L CNN
 F 2 "footprints:R_0805_OEM" H 6530 1775 50  0001 C CNN
@@
 $EndComp
 $Comp
-L formula:R_200 R?
+L formula:R_200 R36
 U 1 1 6186D9F0
 P 6925 1775
-F 0 "R?" H 6995 1821 50  0000 L CNN
+F 0 "R36" H 6995 1821 50  0000 L CNN
 F 1 "R_200" V 6825 1675 50  0000 L CNN
 F 2 "footprints:R_0805_OEM" H 6855 1775 50  0001 C CNN
@@
 LED_3
 $Comp
-L formula:R_200 R?
+L formula:R_200 R32
 U 1 1 6187746D
 P 5925 1775
-F 0 "R?" H 5995 1821 50  0000 L CNN
+F 0 "R32" H 5995 1821 50  0000 L CNN
 F 1 "R_200" V 5800 1750 50  0000 L CNN
 F 2 "footprints:R_0805_OEM" H 5855 1775 50  0001 C CNN
@@
 $EndComp
 $Comp
-L formula:R_200 R?
+L formula:R_200 R33
 U 1 1 61877C41
 P 6275 1775
-F 0 "R?" H 6345 1821 50  0000 L CNN
+F 0 "R33" H 6345 1821 50  0000 L CNN
 F 1 "R_200" V 6175 1750 50  0000 L CNN
 F 2 "footprints:R_0805_OEM" H 6205 1775 50  0001 C CNN
@@
 NoConn ~ 3650 3500
 $Comp
-L formula:R_100K R?
+L formula:R_100K R37
 U 1 1 61A93FF9
 P 13925 2100
-F 0 "R?" H 13800 2100 50  0000 L CNN
+F 0 "R37" H 13800 2100 50  0000 L CNN
 F 1 "R_100K" H 13995 2055 50  0000 L CNN
 F 2 "footprints:R_0805_OEM" H 13855 2100 50  0001 C CNN
@@
 $EndComp
 $Comp
-L lv_bms_2-rescue:+5V-power #PWR?
+L lv_bms_2-rescue:+5V-power #PWR0140
 U 1 1 61AA95E1
 P 13925 1950
-F 0 "#PWR?" H 13925 1800 50  0001 C CNN
+F 0 "#PWR0140" H 13925 1800 50  0001 C CNN
 F 1 "+5V-power" V 13850 2100 50  0000 C CNN
 F 2 "" H 13925 1950 50  0001 C CNN
@@
 MISO
 $Comp
-L lv_bms_2-rescue:+5V-power #PWR?
+L lv_bms_2-rescue:+5V-power #PWR0141
 U 1 1 61AE1812
 P 6375 5825
-F 0 "#PWR?" H 6375 5675 50  0001 C CNN
+F 0 "#PWR0141" H 6375 5675 50  0001 C CNN
 F 1 "+5V-power" H 6390 5998 50  0000 C CNN
 F 2 "" H 6375 5825 50  0001 C CNN
@@
 $EndComp
 $Comp
-L formula:R_10K R?
+L formula:R_10K R34
 U 1 1 61AE2DAA
 P 6375 5975
-F 0 "R?" H 6275 6125 50  0000 L CNN
+F 0 "R34" H 6275 6125 50  0000 L CNN
 F 1 "R_5K" V 6450 5875 50  0000 L CNN
 F 2 "footprints:R_0805_OEM" H 6305 5975 50  0001 C CNN

Commit message: lv bms updates
Parts:
- removed C103, C14, C15: C_0.1uF, footprints:C_0805_OEM, symbol formula:C_0.1uF
- removed COUT101: C_22uF, footprints:C_1206_OEM, symbol formula:C_22uF
- removed COUT102: C_33uF, footprints:Fuse_1812, symbol formula:C_33uF
- removed COUT103: C_47uF, footprints:C_0805_OEM, symbol formula:C_47uF
- removed J3, J4, J5: NanoFit_RA_TH_06, footprints:NanoFit_RA_6, symbol formula:NanoFit_RA_TH_06
- removed L101: L_100uH, formula:L_100uH, symbol formula:L_100uH
- removed Q2: MMBF170, TO_SOT_Packages_SMD:SOT-23, symbol formula:MMBF170
- removed R102, R18, R28: R_25K, footprints:R_0805_OEM, symbol formula:R_25K
- removed R103: R_100K, footprints:R_0805_OEM, symbol formula:R_100K
- removed R19, R20, R21, R25, R26, R29: R_1K, footprints:R_0805_OEM, symbol formula:R_1K
- removed R22, R27: R_22K, footprints:R_0805_OEM, symbol formula:R_22K
- removed R31: R_100, footprints:R_0805_OEM, symbol formula:R_100
- removed R4, R5, R6, R7, R8: 356030RFT, formula:356030RFT, symbol formula:356030RFT
- removed U101: TPS560430YF, footprints:SOT-23-6_OEM, symbol formula:TPS560430YF
- removed U4, U8: MCP6001T-I-LT, Package_TO_SOT_SMD:SOT-353_SC-70-5, symbol formula:MCP6001T-I-LT
- removed U5: LTC1380IGN, Package_SO:SSOP-16_3.9x4.9mm_P0.635mm, symbol formula:LTC1380IGN
- removed U6, U7: TLV3701QDBVRG4Q1, footprints:SOT-23-5_OEM, symbol formula:TLV3701QDBVRG4Q1
- added C14: C_470pF, footprints:C_0805_OEM, symbol formula:C_470pF
- added C15: C_10nF, footprints:C_1206_OEM, symbol formula:C_10nF
- added C16: C_10uF, footprints:C_0805_OEM, symbol formula:C_10uF
- added C17, C21: C_1uF, footprints:C_0805_OEM, symbol formula:C_1uF
- added C18, C19: C_0.1uF, footprints:C_0805_OEM, symbol formula:C_0.1uF
- added C20: C_1nf, formula:C_0805_OEM, symbol formula:C_1nf
- added J10: NanoFit_RA_TH_04, footprints:NanoFit_RA_4, symbol formula:NanoFit_RA_TH_04
- added J4, J5, J6, J7, J8, J9: NanoFit_RA_TH_02, footprints:NanoFit_Molex_1x02x2.50mm_Angled_OEM, symbol formula:NanoFit_RA_TH_02
- added Q2, Q5: SQM110P06, formula:TO-263-2-Heatsink, symbol formula:SQM110P06
- added Q3, Q4: MMBF170, TO_SOT_Packages_SMD:SOT-23, symbol formula:MMBF170
- added R18, R21, R26, R38, R39: R_100K, footprints:R_0805_OEM, symbol formula:R_100K
- added R19: R_1.5k, footprints:R_2010_Vishay, symbol formula:R_1.5k
- added R20, R28, R40: R_10K, footprints:R_0805_OEM, symbol formula:R_10K
- added R22, R27: R_1M, footprints:R_0805_OEM, symbol formula:R_1M
- added R25: R_402K, footprints:R_0805_OEM, symbol formula:R_402K
- added R29, R31: R_0_2512, footprints:R_2512_OEM, symbol formula:R_0_2512
- added R4, R5, R6, R7, R8: R_30_6W_1%, formula:356030RFT, symbol formula:R_30_6W_1%
- added R41: R_10, footprints:R_0805_OEM, symbol formula:R_10
- added TP10, TP11, TP12, TP13, TP7, TP8, TP9: Test_Point_SMD, footprints:Test_Point_SMD, symbol formula:Test_Point_SMD
- added U10: ACHS-7124, formula:OPTO_HCPL-070A-000E, symbol formula:ACHS-7124
- added U11, U9: redcube-7461057, formula:redcube_pressfit_6pin, symbol formula:redcube-7461057
- added U4: LT3066IMSE-5, formula:MSOP-8, symbol formula:LT3066IMSE-5
- added U5: LT1017IS8, formula:SO-8_S, symbol formula:LT1017IS8
- added U6, U7, U8: R_500, footprints:R_0805_OEM, symbol formula:R_500
- C102: footprint footprints:C_0603_1608Metric -> footprints:C_0805_OEM; PurchasingLink https://www.digikey.com/product-detail/en/yageo/CC0603KRX5R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 -> https://www.digikey.com/product-detail/en/tdk-corporation/C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
- R34: value R_5K -> R_10K
Connections:
- net labels added: BATTERY_SIDE_DIV_SIG, BATT_0, BATT_1, BATT_2, BATT_3, BATT_4, BATT_SIDE_DIV_SIG, CAN+, CAN-, COMP_1_OUT, COMP_2_OUT, CURRENT_SENSE_SIGNAL, GND-power, LED_0_+, LED_1_+, LED_2_+, LOAD_SIDE_CURRENT_PATH, LOAD_SIDE_DIV_SIG, LOAD_SWITCH_FET_DRIVE, MISO_LIM, MOSI_LIM, ON_STATE_CMPNTS_-, ON_STATE_CMPNTS_FET_DRIVE, PACK_SIDE_CURRENT_PATH, SCK_LIM, SHIELD, SHUNT_LOAD_SIDE, THERM_0_+, THERM_0_-, THERM_1_+, THERM_1_-, THERM_2_+, THERM_2_-, THERM_3_+, THERM_3_-, THERM_4_+, THERM_4_-, THERM_5_+, THERM_5_-
- net labels removed: +5V, 12V, 2A_in, 2A_out, CAN_+, CAN_-, CURRENT_SENSE_IN, GND, LED_0, LED_1, LED_2, LED_3, RELAY, RELAY_GND, SCL, SDA, T0, T1, T2, T3, T4, T5, TEMP_SENSE, VREF2, batt_0, batt_1, batt_2, batt_3, batt_4
- wire segments 199 -> 261
- no-connect marks 25 -> 20
Other:
- note added: "10K thermistor \nresistor dividers, \nonly powered on \nafter Wakeup"
- note added: "500mA micropower reg for simplicity features 70uA \nquiescent current draw during system off state"
- note added: "5V Jumper\n"
- note added: "6 individual nanofit connectors for thermistors \nto be distributed around the edges of the PCB\nhttps://www.digikey.com/en/products/detail\n/epcos-tdk/B57861S0103F040/739889"
- note added: "BATT_4 Jumper\n"
- note added: "Battery (+) Side"
- note added: "Battery (-) Side"
- note added: "Bidirectional Discrete \nDual-PMOS Load switch"
- note added: "Bidirectional Hall Effect Isolated \nRatiometric current sensor \nGLV system - ACHS-7121 | 10A 185mV/A\nCooling Pack system - ACHS-7124 | 40A 50mV/A"
- note added: "Both packs will see single digits of total discharge cycles --> where\ncells and segments can't get that imbalanced --> balancing is lower\npriority --> we'll use LTC's internal balancing FET's that can limit us \nto 150mA of balancing current, instead of more capable external FET's. \nExpecting 4.2V/30Ohms = 140mA of balancing current thru resistors\n& 4.2V*.140A = .588W of power dissipated thru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"
- note added: "CAN connector"
- note added: "CONNECTORS\n"
- note added: "Comparator logic chart \n+--------+------+-----+---------+\n| | No Load | Charging | Discharging |\n+--------+------+-----+---------+\n| COMP_1_OUT | 1 | 1 | 0 |\n+--------+------+-----+---------+\n| COMP_2_OUT | 1 | 0 | 1 |\n+--------+------+-----+---------+\n\nThe outputs of both comparators are fed into \nLOW Level Triggered External interrupts on the Atemga\nwhere C1 LOW indicates Discharge s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"
- note added: "Drive pin used to drive NPN linear \nregulator to supply LTC chip 5V \nregulated power. Features low pass \nfilter on input."
- note added: "Entire system pulls 170uA of \ncurrent in STANDBY state\nEntire system pulls ~~250mA of \ncurrent in ON state"
- note added: "FET"
- note added: "HIGH CURRENT PATH\n"
- note added: "LEDS"
- note added: "LINEAR REGULATOR\n"
- note added: "LTC6810 BMS CHIP"
- note added: "Low side driven FET to enable \nand disable load switch"
- note added: "Low side driven FET to toggle \nthermistors & current sensor that\nonly need power after system state wakeup"
- note added: "MOSI, MISO, and SCK must\nstay connected to the _A pins\nfor programming.\n\nBecause ISP uses same SPI bus \nas LTC chip comms, we place \nresistors to limit current"
- note added: "Resistor divider on ~SHDN~ to pull net below 1.1V \nwhen battery voltage falls lower than 10.6V. Disables \nLinreg\n"
- note added: "Resistor dividers set at ~~90% to \nact as inputs for comparators"
- note added: "SENSE pin must be connected directly \nto load according to datasheet"
- note added: "THERMISTORS"
- note added: "WAKEUP SHUNT & LOGIC"
- note added: "Wakeup Dual Comparator chosen for\nHV-capable inputs & low quiescent current of 30uA"
- note added: "Wakeup shunt resistor between top \ncell in pack and top of system load. \nRuns in parallel to load switch &\ncurrent sensor. Used to determine\nstate of BMS system - Charging, \nDischarging, or No Load."
- note added: "level triggered external interrupt on \nPB2 & PB5 from comparator outputs\nto wake uC from standby mode\n"
- note added: "~I will get shafted on this design review.~ -Adi R."
- note removed: "BUCK CONVERTER\n"
- note removed: "Bootstrap Capacitor\n"
- note removed: "Feedback Divider\n"
- note removed: "Inductor\n"
- note removed: "LTC6810-1"
- note removed: "MOSI, MISO, and SCK must\nstay connected to the _A pins\nfor programming."
- note removed: "Output Capacitors\n"
- note removed: "POWER FLAGS\n"
- note removed: "Programming LEDs"
- note removed: "VCC Jumper\n"
- note removed: "analog I2C mux with current buffer"
- note removed: "compartors @ > 2.6V | < 2.4V +- 2A\nfor powering BMS system on"
- note removed: "connectors"
- note removed: "current measurement thermistors"
- note removed: "level triggered external interrupt \nto wake uC from sleep"
- note removed: "thermistor + side"
- note removed: "thermistor - side"
- note removed: "thermistor mux"
- moved on the sheet: C101, C102, C11, C13, D1, D101, D102, D103, D2, D3, D4, F101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
